File: kicad/BUTTON-LEDs .kicad_sch (KiCad schematic)
At the start: 15 parts, among them K2 kEY-4, K3 kEY-4, Q22 2N3904, Q23 2N3904

Commit message: Changed MCU to STM32G473VCT6
Parts:
- R120, R121, R122, R123, R124, R125, R126: footprint oomwoo_altium:RES-0402 -> Resistor_SMD:R_0603_1608Metric
Changed lines of the file:
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@@
 			)
 		)
-		(property "Footprint" "oomwoo_altium:RES-0402"
+		(property "Footprint" "Resistor_SMD:R_0603_1608Metric"
 			(at 349.885 158.75 0)
 			(hide yes)
@@
 			)
 		)
-		(property "Footprint" "oomwoo_altium:RES-0402"
+		(property "Footprint" "Resistor_SMD:R_0603_1608Metric"
 			(at 230.505 265.43 0)
 			(hide yes)
@@
 			)
 		)
-		(property "Footprint" "oomwoo_altium:RES-0402"
+		(property "Footprint" "Resistor_SMD:R_0603_1608Metric"
 			(at 230.505 252.73 0)
 			(hide yes)
@@
 			)
 		)
-		(property "Footprint" "oomwoo_altium:RES-0402"
+		(property "Footprint" "Resistor_SMD:R_0603_1608Metric"
 			(at 250.825 173.99 0)
 			(hide yes)
@@
 			)
 		)
-		(property "Footprint" "oomwoo_altium:RES-0402"
+		(property "Footprint" "Resistor_SMD:R_0603_1608Metric"
 			(at 230.505 186.69 0)
 			(hide yes)
@@
 			)
 		)
-		(property "Footprint" "oomwoo_altium:RES-0402"
+		(property "Footprint" "Resistor_SMD:R_0603_1608Metric"
 			(at 250.825 252.73 0)
 			(hide yes)
@@
 			)
 		)
-		(property "Footprint" "oomwoo_altium:RES-0402"
+		(property "Footprint" "Resistor_SMD:R_0603_1608Metric"
 			(at 230.505 173.99 0)
 			(hide yes)

Commit message: STM32G473VCT6
Parts:
- removed Q22, Q23: 2N3904, oomwoo_altium:SOT23-3D, symbol DesignLibrary:BUTTON-LED_0_NPN-SOT23_DesignLibrary.SchLib
- removed R123, R126: 1K, Resistor_SMD:R_0603_1608Metric, symbol DesignLibrary:BUTTON-LED_2_Resistor-1_DesignLibrary.SchLib
- added Q10, Q12: IRLML6344TRPBF, JLCImport:IRLML6344TRPBF, symbol JLCImport:IRLML6344TRPBF
- added R71, R72: 10, Resistor_SMD:R_0603_1608Metric_Pad0.98x0.95mm_HandSolder, symbol Device:R_US
Connections:
- net GND: now also Q10.2 (S), Q12.2 (S)
- net LED-HOME: now also R71.2
- net LED-PWR: now also R72.2
- net at R121.1, R122.1: now also Q10.3 (D)
- net at R124.1, R125.1: now also Q12.3 (D)
- new net: Q10.1 (G), R71.1
- new net: Q12.1 (G), R72.1
