File: kicad/Battery-Charger.kicad_sch (KiCad schematic)
At the start: 67 parts, among them IC5 TPS25730DREFR, IC6 TVS2200DRVR, IC7 TVS2200DRVR, J1 BATTERY, Q26 CSD17581Q3A, Q27 CSD17581Q3A, Q28 CSD17581Q3A, Q29 CSD17581Q3A, U7 BQ25792RQMR

Commit message: Added Pi CM4/CM5
Parts:
- added CN1: EV2400, JLCImport:22053041_C5271241, symbol JLCImport:22053041_C5271241
- added D4: SMCJ18A-13-F, JLCImport:SMCJ18A-13-F, symbol JLCImport:SMCJ18A-13-F
Connections:
- net GND: now also CN1.1, D4.2 (A)
- net SCL: now also CN1.2
- net SDA: now also CN1.3
- net +3.3V renamed VCC3V3_SYS
- net VCC-BAT-IN renamed BAT-VCC
- net BAT-VCC: now also D4.1 (K)
- net ~{FAULT_IN}: no longer names the net of IC5.18 (~{FAULT_IN}), R128.2
- no-connect marks 13 -> 14
Other:
- note added: "OPTIONAL"
- note added: "Put the MCU into RESET mode if use EV2400 to debug the charger"
- moved on the sheet: BAT2

Commit message: Changed MCU to STM32G473VCT6
Parts:
- C60, C69, C75, C77, C78, C79, C83: footprint (none) -> Capacitor_SMD:C_0603_1608Metric
- C62, C63, C70: footprint JLCImport:CL05A475MP5NRNC -> Capacitor_SMD:C_0603_1608Metric
- C80: footprint Capacitor_SMD:C_0603_1608Metric -> Capacitor_SMD:C_0805_2012Metric
- R100, R127, R132, R58, R59, R60: footprint (none) -> Resistor_SMD:R_0603_1608Metric
- R115: footprint JLCImport:FRC0402F1003TS -> Resistor_SMD:R_0603_1608Metric
- R37: footprint oomwoo_altium:RES-0402 -> Resistor_SMD:R_0603_1608Metric
Changed lines of the file:
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@@
 			)
 		)
-		(property "Footprint" ""
+		(property "Footprint" "Capacitor_SMD:C_0603_1608Metric"
 			(at 308.9148 358.14 0)
 			(hide yes)
@@
 			)
 		)
-		(property "Footprint" ""
+		(property "Footprint" "Capacitor_SMD:C_0603_1608Metric"
 			(at 192.7352 359.41 0)
 			(hide yes)
@@
 			)
 		)
-		(property "Footprint" "JLCImport:CL05A475MP5NRNC"
+		(property "Footprint" "Capacitor_SMD:C_0603_1608Metric"
 			(at 132.3848 300.99 0)
 			(hide yes)
@@
 			)
 		)
-		(property "Footprint" ""
+		(property "Footprint" "Resistor_SMD:R_0603_1608Metric"
 			(at 260.604 325.374 90)
 			(hide yes)
@@
 			)
 		)
-		(property "Footprint" ""
+		(property "Footprint" "Resistor_SMD:R_0603_1608Metric"
 			(at 260.096 332.486 90)
 			(hide yes)
@@
 			)
 		)
-		(property "Footprint" "JLCImport:FRC0402F1003TS"
+		(property "Footprint" "Resistor_SMD:R_0603_1608Metric"
 			(at 260.604 327.914 90)
 			(hide yes)
@@
 			)
 		)
-		(property "Footprint" ""
+		(property "Footprint" "Capacitor_SMD:C_0603_1608Metric"
 			(at 262.5852 350.52 0)
 			(hide yes)
@@
 			)
 		)
-		(property "Footprint" ""
+		(property "Footprint" "Capacitor_SMD:C_0603_1608Metric"
 			(at 232.41 280.9748 0)
 			(hide yes)
@@
 			)
 		)
-		(property "Footprint" ""
+		(property "Footprint" "Capacitor_SMD:C_0603_1608Metric"
 			(at 119.0752 359.41 0)
 			(hide yes)
@@
 			)
 		)
-		(property "Footprint" ""
+		(property "Footprint" "Capacitor_SMD:C_0603_1608Metric"
 			(at 277.1648 358.14 0)
 			(hide yes)
@@
 			)
 		)
-		(property "Footprint" ""
+		(property "Footprint" "Resistor_SMD:R_0603_1608Metric"
 			(at 153.924 310.134 90)
 			(hide yes)
@@
 			)
 		)
-		(property "Footprint" "JLCImport:CL05A475MP5NRNC"
+		(property "Footprint" "Capacitor_SMD:C_0603_1608Metric"
 			(at 132.3848 323.85 0)
 			(hide yes)
@@
 			)
 		)
-		(property "Footprint" "oomwoo_altium:RES-0402"
+		(property "Footprint" "Resistor_SMD:R_0603_1608Metric"
 			(at 208.28 274.32 0)
 			(hide yes)
@@
 			)
 		)
-		(property "Footprint" ""
+		(property "Footprint" "Resistor_SMD:R_0603_1608Metric"
 			(at 153.924 332.994 90)
 			(hide yes)
@@
 			)
 		)
-		(property "Footprint" ""
+		(property "Footprint" "Resistor_SMD:R_0603_1608Metric"
 			(at 247.904 352.806 90)
 			(hide yes)
@@
 			)
 		)
-		(property "Footprint" "JLCImport:CL05A475MP5NRNC"
+		(property "Footprint" "Capacitor_SMD:C_0603_1608Metric"
 			(at 203.5048 351.79 0)
 			(hide yes)
@@
 			)
 		)
-		(property "Footprint" "Capacitor_SMD:C_0603_1608Metric"
+		(property "Footprint" "Capacitor_SMD:C_0805_2012Metric"
 			(at 285.4198 350.52 0)
 			(hide yes)
@@
 			)
 		)
-		(property "Footprint" ""
+		(property "Footprint" "Capacitor_SMD:C_0603_1608Metric"
 			(at 282.2448 309.88 0)
 			(hide yes)
@@
 			)
 		)
-		(property "Footprint" ""
+		(property "Footprint" "Resistor_SMD:R_0603_1608Metric"
 			(at 294.894 291.846 90)
 			(hide yes)

Commit message: STM32G473VCT6
Connections:
- net VCC3V3_SYS is gone; now on net VCC-3V3-P: C59.2, IC5.38 (VIN_3V3)
Changed lines of the file:
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@@
 	)
 	(symbol
-		(lib_id "oomwoo-kicad-altium-import:VCC3V3_SYS_BAR")
-		(at 78.74 72.39 180)
-		(unit 1)
-		(body_style 1)
-		(exclude_from_sim no)
-		(in_bom yes)
-		(on_board yes)
-		(in_pos_files yes)
-		(dnp no)
-		(property "Reference" "#PWR065"
-			(at 78.74 72.39 0)
-			(hide yes)
-			(show_name no)
-			(do_not_autoplace no)
-			(effects
-				(font
-					(size 1.27 1.27)
-				)
-			)
-		)
-		(property "Value" "VCC3V3_SYS"
-			(at 78.74 68.58 0)
-			(show_name no)
-			(do_not_autoplace no)
-			(effects
-				(font
-					(size 1.27 1.27)
-				)
-			)
-		)
-		(property "Footprint" ""
-			(at 78.74 72.39 0)
-			(show_name no)
-			(do_not_autoplace no)
-			(effects
-				(font
-					(size 1.27 1.27)
-				)
-			)
-		)
-		(property "Datasheet" ""
-			(at 78.74 72.39 0)
-			(show_name no)
-			(do_not_autoplace no)
-			(effects
-				(font
-					(size 1.27 1.27)
-				)
-			)
-		)
-		(property "Description" ""
-			(at 78.74 72.39 0)
-			(show_name no)
-			(do_not_autoplace no)
-			(effects
-				(font
-					(size 1.27 1.27)
-				)
-			)
-		)
-		(pin ""
-		)
-		(instances
-			(project "oomwoo-kicad"
-				(path "/dbcfb655-8d45-4808-9a74-2a0eb03372e8/ef1147df-ce85-4822-98ae-5614ce438d97"
-					(reference "#PWR065")
-					(unit 1)
-				)
-			)
-		)
-	)
-	(symbol
 		(lib_id "DesignLibrary:POWER_0_LED-SMD_DesignLibrary.SchLib")
 		(at 208.28 248.92 0)
@@
 					(unit 1)
 				)
+			)
+		)
+	)
+	(symbol
+		(lib_id "oomwoo-kicad-altium-import:VCC-3V3-P_BAR")
+		(at 78.74 72.39 180)
+		(unit 1)
+		(body_style 1)
+		(exclude_from_sim no)
+		(in_bom yes)
+		(on_board yes)
+		(in_pos_files yes)
+		(dnp no)
+		(property "Reference" "#PWR065"
+			(at 78.74 72.39 0)
+			(hide yes)
+			(show_name no)
+			(do_not_autoplace no)
+			(effects
+				(font
+					(size 1.27 1.27)
+				)
+			)
+		)
+		(property "Value" "VCC-3V3-P"
+			(at 78.74 68.58 0)
+			(show_name no)
+			(do_not_autoplace no)
+			(effects
+				(font
+					(size 1.27 1.27)
+				)
+			)
+		)
+		(property "Footprint" ""
+			(at 78.74 72.39 0)
+			(show_name no)
+			(do_not_autoplace no)
+			(effects
+				(font
+					(size 1.27 1.27)
+				)
+			)
+		)
+		(property "Datasheet" ""
+			(at 78.74 72.39 0)
+			(show_name no)
+			(do_not_autoplace no)
+			(effects
+				(font
+					(size 1.27 1.27)
+				)
+			)
+		)
+		(property "Description" ""
+			(at 78.74 72.39 0)
+			(show_name no)
+			(do_not_autoplace no)
+			(effects
+				(font
+					(size 1.27 1.27)
+				)
+			)
+		)
+		(pin ""
+		)
+		(instances
+			(project "oomwoo-kicad"
+				(path "/dbcfb655-8d45-4808-9a74-2a0eb03372e8/ef1147df-ce85-4822-98ae-5614ce438d97"
+					(reference "#PWR065")
+					(unit 1)
+				)
