File: kicad/IMU-ICM-4267-P .kicad_sch (KiCad schematic)
At the start: 7 parts, among them U19 ICM-42607-P

Commit message: Changed MCU to STM32G473VCT6
Parts:
- C108: footprint oomwoo_altium:CAP-0603 -> Capacitor_SMD:C_0603_1608Metric
- C109, C110: footprint oomwoo_altium:CAP-0402 -> Capacitor_SMD:C_0603_1608Metric
- R18, R92, R93: footprint oomwoo_altium:RES-0402 -> Resistor_SMD:R_0603_1608Metric
Changed lines of the file:
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@@
 			)
 		)
-		(property "Footprint" "oomwoo_altium:RES-0402"
+		(property "Footprint" "Resistor_SMD:R_0603_1608Metric"
 			(at 249.555 179.705 0)
 			(hide yes)
@@
 			)
 		)
-		(property "Footprint" "oomwoo_altium:CAP-0402"
+		(property "Footprint" "Capacitor_SMD:C_0603_1608Metric"
 			(at 389.255 205.105 0)
 			(hide yes)
@@
 			)
 		)
-		(property "Footprint" "oomwoo_altium:CAP-0603"
+		(property "Footprint" "Capacitor_SMD:C_0603_1608Metric"
 			(at 368.935 205.105 0)
 			(hide yes)
@@
 			)
 		)
-		(property "Footprint" "oomwoo_altium:RES-0402"
+		(property "Footprint" "Resistor_SMD:R_0603_1608Metric"
 			(at 257.175 179.705 0)
 			(hide yes)
@@
 			)
 		)
-		(property "Footprint" "oomwoo_altium:RES-0402"
+		(property "Footprint" "Resistor_SMD:R_0603_1608Metric"
 			(at 241.935 179.705 0)
 			(hide yes)
@@
 			)
 		)
-		(property "Footprint" "oomwoo_altium:CAP-0402"
+		(property "Footprint" "Capacitor_SMD:C_0603_1608Metric"
 			(at 379.095 205.105 0)
 			(hide yes)

Commit message: STM32G473VCT6
Connections:
- net VCC3V3_SYS renamed VCC-3V3-P
Changed lines of the file:
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@@
+	)
+	(symbol
+		(lib_id "oomwoo-kicad-altium-import:VCC-3V3-P_BAR")
+		(at 361.315 187.325 180)
+		(unit 1)
+		(body_style 1)
+		(exclude_from_sim no)
+		(in_bom yes)
+		(on_board yes)
+		(in_pos_files yes)
+		(dnp no)
+		(property "Reference" "#PWR089"
+			(at 361.315 187.325 0)
+			(hide yes)
+			(show_name no)
+			(do_not_autoplace no)
+			(effects
+				(font
+					(size 1.27 1.27)
+				)
+			)
+		)
+		(property "Value" "VCC-3V3-P"
+			(at 361.315 183.515 0)
+			(show_name no)
+			(do_not_autoplace no)
+			(effects
+				(font
+					(size 1.27 1.27)
+				)
+			)
+		)
+		(property "Footprint" ""
+			(at 361.315 187.325 0)
+			(show_name no)
+			(do_not_autoplace no)
+			(effects
+				(font
+					(size 1.27 1.27)
+				)
+			)
+		)
+		(property "Datasheet" ""
+			(at 361.315 187.325 0)
+			(show_name no)
+			(do_not_autoplace no)
+			(effects
+				(font
+					(size 1.27 1.27)
+				)
+			)
+		)
+		(property "Description" ""
+			(at 361.315 187.325 0)
+			(show_name no)
+			(do_not_autoplace no)
+			(effects
+				(font
+					(size 1.27 1.27)
+				)
+			)
+		)
+		(pin ""
+		)
+		(instances
+			(project "oomwoo-kicad"
+				(path "/dbcfb655-8d45-4808-9a74-2a0eb03372e8/7b57c0fa-4a35-4109-8672-3c36267bf8ff"
+					(reference "#PWR089")
+					(unit 1)
+				)
+			)
+		)
 	)
 	(symbol
@@
 	)
 	(symbol
-		(lib_id "oomwoo-kicad-altium-import:VCC3V3_SYS_BAR")
-		(at 361.315 187.325 180)
-		(unit 1)
-		(body_style 1)
-		(exclude_from_sim no)
-		(in_bom yes)
-		(on_board yes)
-		(in_pos_files yes)
-		(dnp no)
-		(property "Reference" "#PWR0691"
-			(at 361.315 187.325 0)
-			(hide yes)
-			(show_name no)
-			(do_not_autoplace no)
-			(effects
-				(font
-					(size 1.27 1.27)
-				)
-			)
-		)
-		(property "Value" "VCC3V3_SYS"
-			(at 361.315 183.515 0)
-			(show_name no)
-			(do_not_autoplace no)
-			(effects
-				(font
-					(size 1.27 1.27)
-				)
-			)
-		)
-		(property "Footprint" ""
-			(at 361.315 187.325 0)
-			(show_name no)
-			(do_not_autoplace no)
-			(effects
-				(font
-					(size 1.27 1.27)
-				)
-			)
-		)
-		(property "Datasheet" ""
-			(at 361.315 187.325 0)
-			(show_name no)
-			(do_not_autoplace no)
-			(effects
-				(font
-					(size 1.27 1.27)
-				)
-			)
-		)
-		(property "Description" ""
-			(at 361.315 187.325 0)
-			(show_name no)
-			(do_not_autoplace no)
-			(effects
-				(font
-					(size 1.27 1.27)
-				)
-			)
-		)
-		(pin ""
-		)
-		(instances
-			(project "oomwoo-kicad"
-				(path "/dbcfb655-8d45-4808-9a74-2a0eb03372e8/7b57c0fa-4a35-4109-8672-3c36267bf8ff"
-					(reference "#PWR0691")
-					(unit 1)
-				)
-			)
-		)
-	)
-	(symbol
 		(lib_id "DesignLibrary:IMU_3_Resistor-1_DesignLibrary.SchLib")
 		(at 241.935 179.705 0)
@@
 	)
 	(symbol
-		(lib_id "oomwoo-kicad-altium-import:VCC3V3_SYS_BAR")
+		(lib_id "oomwoo-kicad-altium-import:VCC-3V3-P_BAR")
 		(at 249.555 167.005 180)
 		(unit 1)
@@
 		(in_pos_files yes)
 		(dnp no)
-		(property "Reference" "#PWR0689"
+		(property "Reference" "#PWR088"
 			(at 249.555 167.005 0)
 			(hide yes)
@@
 			)
 		)
-		(property "Value" "VCC3V3_SYS"
+		(property "Value" "VCC-3V3-P"
 			(at 249.555 163.195 0)
 			(show_name no)
@@
 			(project "oomwoo-kicad"
 				(path "/dbcfb655-8d45-4808-9a74-2a0eb03372e8/7b57c0fa-4a35-4109-8672-3c36267bf8ff"
-					(reference "#PWR0689")
+					(reference "#PWR088")
 					(unit 1)
 				)
