File: kicad/oomwoo-kicad.kicad_pcb (KiCad board)
At the start: 4 copper layers, 116 x 98.7 mm, 236 parts, among them CN1 EV2400, J1 BATTERY, J10 WATER-PUMP, J11 MAIN BRUSH, J12 WHEEL-MOTOR-RIGHT, J13 WHEEL-MOTOR-LEFT, J15 SIDE BRUSH, J17 LiDAR, J18 SPEAKER2, J21 STM-PROGRAM, J23 STM32-PROGRAM, J4 ANTI-FALL-LEFT-DOWN, J5 ANTI-FALL-RIGHT-DOWN, J8 SIDE-PROXI-LEFT, J9 SIDE-PROXI-RIGHT, K2 kEY-4, K3 kEY-4, Q1 AO4407A, Q11 2N3904, Q15 2N3904, Q20 AO3400, Q22 2N3904, Q23 2N3904, Q26 CSD17581Q3A, Q27 CSD17581Q3A, Q28 CSD17581Q3A, Q29 CSD17581Q3A, Q3 PNP-SOT23, Q6 2N3904, Q7 2N3904, Q8 AO3401, Q9 2N3904, U10 BL24131607, U11 MAX98357AETE_T, U13 STM32G473VCT6, U14 DRV8870DDAR, U15 DRV8870DDAR, U18 DRV8870DDAR, U19 ICM-42607-P, U20 DRV8870DDAR, U4 SY8089A, U5 SY8089A, U6 RT9742GGJ5, U7 BQ25792RQMR, U9 ICS-43434_C5656610, X1 ABM3-8_000MHZ-D2Y-T

Commit message: STM32G473VCT6
Parts:
- removed U10: BL24131607, JLCImport:S5B-PH-SM4-TB_LF_SN
- added BOOT1: Conn_01x02_Pin, Connector_PinHeader_2.54mm:PinHeader_1x02_P2.54mm_Vertical, F.Cu at (205.5, 55.7)
- added C10: 100nF/10V, Capacitor_SMD:C_0603_1608Metric, F.Cu at (228.6, 42.4)
- added C101: 0.1uF, Capacitor_SMD:C_0603_1608Metric, F.Cu at (218.6, 42.4)
- added C11: 10uF/10V, Capacitor_SMD:C_0603_1608Metric, F.Cu at (228.6, 44.9)
- added C12: 100nF/10V, Capacitor_SMD:C_0603_1608Metric, F.Cu at (205.3, 22.9)
- added C13: 100nF/10V, Capacitor_SMD:C_0603_1608Metric, F.Cu at (205.3, 25.4)
- added C14: 100nF/10V, Capacitor_SMD:C_0603_1608Metric, F.Cu at (205.3, 27.9)
- added C15: 100nF/10V, Capacitor_SMD:C_0603_1608Metric, F.Cu at (205.3, 30.4)
- added C16: 100nF/10V, Capacitor_SMD:C_0603_1608Metric, F.Cu at (205.3, 32.9)
- added C17: 4.7uF/10V, Capacitor_SMD:C_0603_1608Metric, F.Cu at (205.3, 35.4)
- added C30: 100nF/10V, Capacitor_SMD:C_0603_1608Metric, F.Cu at (205.3, 37.9)
- added C31: 4.7uF/10V, Capacitor_SMD:C_0603_1608Metric, F.Cu at (209.3, 22.9)
- added C32: 100nF/10V, Capacitor_SMD:C_0603_1608Metric, F.Cu at (209.3, 25.4)
- added C33: 4.7uF/10V, Capacitor_SMD:C_0603_1608Metric, F.Cu at (209.3, 27.9)
- added C34: 22pF/10V, Capacitor_SMD:C_0603_1608Metric, F.Cu at (209.3, 30.4)
- added C35: 22pF/10V, Capacitor_SMD:C_0603_1608Metric, F.Cu at (209.3, 32.9)
- added C36: 10uF/50V, Capacitor_SMD:C_0603_1608Metric, F.Cu at (215.9, 54.6)
- added C37: 100nF/10V, Capacitor_SMD:C_0603_1608Metric, F.Cu at (209.3, 35.4)
- added C5: 100nF/10V, Capacitor_SMD:C_0603_1608Metric, F.Cu at (224.6, 42.4)
- added C6: 33nF/10V, Capacitor_SMD:C_0603_1608Metric, F.Cu at (224.6, 44.9)
- added C60: 0.1uF/50V, Capacitor_SMD:C_0603_1608Metric, F.Cu at (229.4, 22.9)
- added C69: 0.1uF/50V, Capacitor_SMD:C_0603_1608Metric, F.Cu at (229.4, 25.4)
- added C7: 10uF/10V, Capacitor_SMD:C_0603_1608Metric, F.Cu at (224.6, 47.5)
- added C75: 47nF/50V, Capacitor_SMD:C_0603_1608Metric, F.Cu at (229.4, 27.9)
- added C77: 1nF/50V, Capacitor_SMD:C_0603_1608Metric, F.Cu at (229.4, 30.4)
- added C78: 0.1uF/50V, Capacitor_SMD:C_0603_1608Metric, F.Cu at (229.4, 32.9)
- added C79: 47nF/50V, Capacitor_SMD:C_0603_1608Metric, F.Cu at (233.4, 22.9)
- added C8: 33nF/10V, Capacitor_SMD:C_0603_1608Metric, F.Cu at (224.6, 50.0)
- added C83: 0.1uF/50V, Capacitor_SMD:C_0603_1608Metric, F.Cu at (233.4, 25.4)
- added C9: 10uF/10V, Capacitor_SMD:C_0603_1608Metric, F.Cu at (224.6, 52.5)
- added D5: SS34, Diode_SMD:D_SMA, F.Cu at (219.4, 32.7)
- added J14: MAIN-FAN, oomwoo_altium:CONN-SMD_4P-P2.00_XUNPU_WAFER-PH2.0-4PWB, F.Cu at (209.9, 46.3)
- added JTAG1: STLINK-V3MINIE, JLCImport:FTSH-107-01-L-DV-K-A, F.Cu at (220.4, 25.9)
- added R1: 10, Resistor_SMD:R_0603_1608Metric, F.Cu at (209.8, 54.6)
- added R100: 100, Resistor_SMD:R_0603_1608Metric, F.Cu at (237.4, 22.9)
- added R118: 1K, Resistor_SMD:R_0603_1608Metric, F.Cu at (218.6, 44.9)
- added R119: 10K, Resistor_SMD:R_0603_1608Metric, F.Cu at (218.6, 47.5)
- added R12: 0, Resistor_SMD:R_0603_1608Metric, F.Cu at (232.6, 47.5)
- added R127: 5.24k, Resistor_SMD:R_0603_1608Metric, F.Cu at (237.4, 25.4)
- added R13: 100k, Resistor_SMD:R_0603_1608Metric, F.Cu at (232.6, 50.0)
- added R132: 100, Resistor_SMD:R_0603_1608Metric, F.Cu at (237.4, 27.9)
- added R15: 2.2k, Resistor_SMD:R_0603_1608Metric, F.Cu at (215.9, 59.1)
- added R16: 0.01, Resistor_SMD:R_0603_1608Metric, F.Cu at (209.3, 37.9)
- added R19: 0, Resistor_SMD:R_0603_1608Metric, F.Cu at (213.3, 22.9)
- added R21: 10k, Resistor_SMD:R_0603_1608Metric, F.Cu at (213.3, 25.4)
- added R22: 10k, Resistor_SMD:R_0603_1608Metric, F.Cu at (213.3, 27.9)
- added R33: 10, Resistor_SMD:R_0603_1608Metric, F.Cu at (213.3, 30.4)
- added R5: 150, Resistor_SMD:R_0603_1608Metric, F.Cu at (228.6, 47.5)
- added R58: 100, Resistor_SMD:R_0603_1608Metric, F.Cu at (233.4, 27.9)
- added R59: 100, Resistor_SMD:R_0603_1608Metric, F.Cu at (233.4, 30.4)
- added R6: 270, Resistor_SMD:R_0603_1608Metric, F.Cu at (228.6, 50.0)
- added R60: 30.31k, Resistor_SMD:R_0603_1608Metric, F.Cu at (233.4, 32.9)
- added R7: 150, Resistor_SMD:R_0603_1608Metric, F.Cu at (228.6, 52.5)
- added R8: 100k, Resistor_SMD:R_0603_1608Metric, F.Cu at (232.6, 42.4)
- added R9: 0, Resistor_SMD:R_0603_1608Metric, F.Cu at (232.6, 44.9)
- C103, C105, C109, C110, C21, C25, C26, C86, C87, C88, C90, C91, C92: footprint oomwoo_altium:CAP-0402 -> Capacitor_SMD:C_0603_1608Metric
- C108, C22, C24, C27: footprint oomwoo_altium:CAP-0603 -> Capacitor_SMD:C_0603_1608Metric
- C19: value 22uF -> 22uF/10V; footprint oomwoo_altium:CAP-0603 -> Capacitor_SMD:C_0603_1608Metric
- C20: value 100nF -> 100nF/10V; footprint oomwoo_altium:CAP-0402 -> Capacitor_SMD:C_0603_1608Metric
- C62, C63, C70: footprint JLCImport:CL05A475MP5NRNC -> Capacitor_SMD:C_0603_1608Metric
- C80: footprint Capacitor_SMD:C_0603_1608Metric -> Capacitor_SMD:C_0805_2012Metric
- C84: value 0.22uF -> 0.22uF/25V; footprint oomwoo_altium:CAP-0402 -> Capacitor_SMD:C_0603_1608Metric
- CN2: value ~ -> S16B-PHDSS_LF_SN; footprint JLCImport:FTSH-107-01-L-DV-K-A -> JLCImport:S16B-PHDSS_LF_SN
- J21: footprint oomwoo_altium:HDR1X5 -> Connector_PinHeader_2.54mm:PinHeader_1x05_P2.54mm_Vertical
- R10, R101, R102, R103, R104, R105, R106, R107, R108, R109, R11, R110, R111, R113, R114, R116, R120, R121, R122, R123, R124, R125, R126, R14, R17, R18, R20, R23, R24, R25, R26, R27, R28, R29, R31, R32, R34, R37, R40, R45, R67, R68, R69, R70, R71, R72, R73, R74, R75, R76, R77, R78, R79, R80, R81, R89, R90, R91, R92, R93, R94, R95, R97, R98: footprint oomwoo_altium:RES-0402 -> Resistor_SMD:R_0603_1608Metric
- R112, R83, R84, R87, R88, R96: footprint oomwoo_altium:RES-0603 -> Resistor_SMD:R_0603_1608Metric
- R115: footprint JLCImport:FRC0402F1003TS -> Resistor_SMD:R_0603_1608Metric
- R2: footprint Resistor_SMD:R_0603_1608Metric_Pad0.98x0.95mm_HandSolder -> Resistor_SMD:R_0603_1608Metric
- moved CN2 25.5 mm to (108.0, 44.1), turned to 180 degrees
Connections:
- net /CM5-GPIO/UART2_RX renamed /MCU-STM32/STM32-TX
- net /CM5-GPIO/UART2_TX renamed /MCU-STM32/STM32-RX
- D22 pad 1: /SIDE-BRUSH/SIDE-BRUSH-CURRENT-ADC -> /MCU-STM32/SIDE-BRUSH-CURRENT-ADC
- Module1 pad 37: /CM5-GPIO/GPIO07 -> /MCU-STM32/STM32-RST
- R105 pad 1: /SIDE-BRUSH/SIDE-BRUSH-IN1 -> /MCU-STM32/SIDE-BRUSH-IN1
- R110 pad 1: /SIDE-BRUSH/SIDE-BRUSH-CURRENT-ADC -> /MCU-STM32/SIDE-BRUSH-CURRENT-ADC
- R91 pad 1: /SIDE-BRUSH/SIDE-BRUSH-IN2 -> /MCU-STM32/SIDE-BRUSH-IN2
- U13 pad 18: /MCU-STM32/BUMPER-SW1 -> unconnected-(U13A-PC3-Pad18)
- U13 pad 26: /MCU-STM32/MAIN-BRUSH-CURRENT-ADC -> /MAIN-BRUSH MOTOR/MAIN-BRUSH-CURRENT-ADC
- U13 pad 37: Net-(U13C-VDDA) -> VCC-3V3-P
- U13 pad 61: /MCU-STM32/MAIN-BRUSH-IN1 -> /MAIN-BRUSH MOTOR/MAIN-BRUSH-IN1
- U13 pad 62: /MCU-STM32/MAIN-BRUSH-IN2 -> /MAIN-BRUSH MOTOR/MAIN-BRUSH-IN2
- U13 pad 67: /MCU-STM32/I2C3_SCL -> /BATTERY-CHARGER/SCL
- U13 pad 68: /BUTTON-LED/LED-HOME -> /BATTERY-CHARGER/SDA
- U13 pad 80: /MCU-STM32/I2C3_SDA -> /BUTTON-LED/LED-HOME
- U13 pad 81: /MCU-STM32/MAIN-FAN-FG -> /MAIN-FAN/MAIN-FAN-S-SENSE
- U13 pad 83: /MCU-STM32/MAIN-FAN-SP -> /MAIN-FAN/MAIN-FAN-S-CTRL
Routing:
- net GND: track 757.8 -> 944.1 mm, vias 797 -> 816
- net /MCU-STM32/SIDE-BRUSH-L-F-ADC: track 122.1 -> 0.00 mm, vias 2 -> 0
- net /MCU-STM32/STM32-TX: track 95.3 -> 0.00 mm, vias 4 -> 0
- net /MCU-STM32/STM32-RX: track 93.6 -> 0.00 mm, vias 4 -> 0
- net (no net): track 8301.3 -> 8387.5 mm, vias 516 -> 518
- net VCC3V3_SYS: track 316.4 -> 354.1 mm, vias 30 -> 32
- net Net-(U18-OUT2): track 0.00 -> 8.84 mm
- net Net-(D9-A): track 8.50 -> 0.00 mm
- net unconnected-(CN2-Pad8): track 0.00 -> 0.57 mm, vias 0 -> 1
- net unconnected-(CN2-Pad13): vias 1 -> 0
- net unconnected-(CN2-Pad11): vias 1 -> 0
- net unconnected-(CN2-9-Pad09): vias 1 -> 0
- net unconnected-(CN2-7-Pad07): vias 2 -> 0
- net unconnected-(CN2-6-Pad06): vias 1 -> 0
- net unconnected-(CN2-5-Pad05): vias 4 -> 0
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