File: kicad/CM5-Highspeed.kicad_sch (KiCad schematic)
At the start: 1 part

Commit message: STM32G473VCT6
Connections:
- net PCIE_CLK_nREQ: now reaches Module1.102 (PCIe_nCLKREQ)
- net PCIE_nWAKE: now reaches Module1.104 (PCIE_nWAKE)
- net PCIE_nRST: now reaches Module1.109 (PCIe_nRST)
- net PCIE_CLK_P: now reaches Module1.110 (PCIe_CLK_P)
- net PCIE_CLK_N: now reaches Module1.112 (PCIe_CLK_N)
- net PCIE_RX_P: now reaches Module1.116 (PCIe_RX_P)
- net PCIE_RX_N: now reaches Module1.118 (PCIe_RX_N)
- net PCIE_TX_P: now reaches Module1.122 (PCIe_TX_P)
- net PCIE_TX_N: now reaches Module1.124 (PCIe_TX_N)
- no-connect marks 50 -> 41
Changed lines of the file:
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@@
-	)
-	(no_connect
-		(at 299.085 109.22)
 	)
 	(no_connect
@@
 	)
 	(no_connect
-		(at 299.085 99.06)
-	)
-	(no_connect
-		(at 299.085 93.98)
-	)
-	(no_connect
 		(at 299.085 198.12)
 	)
@@
 	)
 	(no_connect
-		(at 299.085 81.28)
-	)
-	(no_connect
 		(at 299.085 152.4)
 	)
@@
 	)
 	(no_connect
-		(at 299.085 83.82)
-	)
-	(no_connect
 		(at 360.045 147.32)
 	)
@@
 	)
 	(no_connect
-		(at 299.085 101.6)
-	)
-	(no_connect
 		(at 299.085 154.94)
 	)
@@
 	)
 	(no_connect
-		(at 299.085 106.68)
-	)
-	(no_connect
-		(at 360.045 91.44)
-	)
-	(no_connect
 		(at 299.085 147.32)
 	)
@@
 	)
 	(no_connect
-		(at 299.085 91.44)
-	)
-	(no_connect
 		(at 299.085 182.88)
 	)
@@
 	(wire
 		(pts
+			(xy 286.385 83.82) (xy 299.085 83.82)
+		)
+		(stroke
+			(width 0)
+			(type default)
+		)
+	)
+	(wire
+		(pts
 			(xy 360.045 193.04) (xy 375.92 193.04)
 		)
@@
 	(wire
 		(pts
+			(xy 286.385 91.44) (xy 299.085 91.44)
+		)
+		(stroke
+			(width 0)
+			(type default)
+		)
+	)
+	(wire
+		(pts
 			(xy 360.045 116.84) (xy 375.92 116.84)
 		)
@@
 	(wire
 		(pts
+			(xy 286.385 99.06) (xy 299.085 99.06)
+		)
+		(stroke
+			(width 0)
+			(type default)
+		)
+	)
+	(wire
+		(pts
 			(xy 360.045 180.34) (xy 370.205 180.34)
 		)
@@
 	(wire
 		(pts
+			(xy 286.385 81.28) (xy 299.085 81.28)
+		)
+		(stroke
+			(width 0)
+			(type default)
+		)
+	)
+	(wire
+		(pts
 			(xy 291.465 172.72) (xy 299.085 172.72)
 		)
@@
 	(wire
 		(pts
+			(xy 360.045 91.44) (xy 372.11 91.44)
+		)
+		(stroke
+			(width 0)
+			(type default)
+		)
+	)
+	(wire
+		(pts
 			(xy 360.045 149.86) (xy 370.205 149.86)
 		)
@@
 	(wire
 		(pts
+			(xy 286.385 101.6) (xy 299.085 101.6)
+		)
+		(stroke
+			(width 0)
+			(type default)
+		)
+	)
+	(wire
+		(pts
 			(xy 360.045 119.38) (xy 370.205 119.38)
 		)
@@
 	(wire
 		(pts
+			(xy 286.385 109.22) (xy 299.085 109.22)
+		)
+		(stroke
+			(width 0)
+			(type default)
+		)
+	)
+	(wire
+		(pts
+			(xy 286.385 106.68) (xy 299.085 106.68)
+		)
+		(stroke
+			(width 0)
+			(type default)
+		)
+	)
+	(wire
+		(pts
 			(xy 291.465 165.1) (xy 299.085 165.1)
 		)
@@
 	(wire
 		(pts
+			(xy 286.385 93.98) (xy 299.085 93.98)
+		)
+		(stroke
+			(width 0)
+			(type default)
+		)
+	)
+	(wire
+		(pts
 			(xy 360.045 114.3) (xy 375.92 114.3)
 		)
@@
 		)
 	)
+	(hierarchical_label "PCIE_TX_P"
+		(shape input)
+		(at 286.385 106.68 180)
+		(effects
+			(font
+				(size 1.27 1.27)
+			)
+			(justify right)
+		)
+	)
+	(hierarchical_label "PCIE_nWAKE"
+		(shape output)
+		(at 286.385 83.82 180)
+		(effects
+			(font
+				(size 1.27 1.27)
+			)
+			(justify right)
+		)
+	)
 	(hierarchical_label "USB2_P"
 		(shape bidirectional)
@@
 		)
 	)
+	(hierarchical_label "PCIE_CLK_nREQ"
+		(shape output)
+		(at 286.385 81.28 180)
+		(effects
+			(font
+				(size 1.27 1.27)
+			)
+			(justify right)
+		)
+	)
 	(hierarchical_label "CM4_CAM0_D1_P"
 		(shape bidirectional)
@@
 		)
 	)
+	(hierarchical_label "PCIE_CLK_P"
+		(shape input)
+		(at 286.385 91.44 180)
+		(effects
+			(font
+				(size 1.27 1.27)
+			)
+			(justify right)
+		)
+	)
 	(hierarchical_label "MIPI1_C_P"
 		(shape bidirectional)
@@
 		)
 	)
+	(hierarchical_label "PCIE_RX_P"
+		(shape output)
+		(at 286.385 99.06 180)
+		(effects
+			(font
+				(size 1.27 1.27)
+			)
+			(justify right)
+		)
+	)
 	(hierarchical_label "MIPI1_C_N"
 		(shape bidirectional)
@@
 		)
 	)
+	(hierarchical_label "PCIE_CLK_N"
+		(shape input)
+		(at 286.385 93.98 180)
+		(effects
+			(font
+				(size 1.27 1.27)
+			)
+			(justify right)
+		)
+	)
 	(hierarchical_label "MIPI1_D0_N"
 		(shape bidirectional)
@@
 		(effects
 			(font
+				(size 1.27 1.27)
+			)
+			(justify left)
+		)
+	)
+	(hierarchical_label "PCIE_TX_N"
+		(shape input)
+		(at 286.385 109.22 180)
+		(effects
+			(font
+				(size 1.27 1.27)
+			)
+			(justify right)
+		)
+	)
+	(hierarchical_label "PCIE_RX_N"
+		(shape output)
+		(at 286.385 101.6 180)
+		(effects
+			(font
+				(size 1.27 1.27)
+			)
+			(justify right)
+		)
+	)
+	(hierarchical_label "PCIE_nRST"
+		(shape input)
+		(at 372.11 91.44 0)
+		(effects
+			(font

Commit message: RTC clock, signal integrity
Parts:
- added R101, R96: 10, symbol Device:R_US
Connections:
- net USB2_N: now also R96.2; no longer Module1.103 (USB2_N)
- net USB2_P: now also R101.2; no longer Module1.105 (USB2_P)
- new net: Module1.103 (USB2_N), R96.1
- new net: Module1.105 (USB2_P), R101.1
Changed lines of the file:
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@@
+	(wire
+		(pts
+			(xy 381 86.36) (xy 391.795 86.36)
+		)
+		(stroke
+			(width 0)
+			(type default)
+		)
+	)
 	(wire
 		(pts
@@
 	(wire
 		(pts
+			(xy 381 83.82) (xy 391.795 83.82)
+		)
+		(stroke
+			(width 0)
+			(type default)
+		)
+	)
+	(wire
+		(pts
 			(xy 291.465 142.24) (xy 299.085 142.24)
 		)
@@
 	(wire
 		(pts
-			(xy 360.045 83.82) (xy 370.205 83.82)
+			(xy 360.045 83.82) (xy 373.38 83.82)
 		)
 		(stroke
@@
 	(wire
 		(pts
-			(xy 360.045 86.36) (xy 370.205 86.36)
+			(xy 360.045 86.36) (xy 373.38 86.36)
 		)
 		(stroke
@@
 	(hierarchical_label "USB2_P"
 		(shape bidirectional)
-		(at 370.205 86.36 0)
+		(at 391.795 86.36 0)
 		(effects
 			(font
@@
 	(hierarchical_label "USB2_N"
 		(shape bidirectional)
-		(at 370.205 83.82 0)
+		(at 391.795 83.82 0)
 		(effects
 			(font
@@
 	)
 	(symbol
+		(lib_id "Device:R_US")
+		(at 377.19 83.82 90)
+		(unit 1)
+		(body_style 1)
+		(exclude_from_sim no)
+		(in_bom yes)
+		(on_board yes)
+		(in_pos_files yes)
+		(dnp no)
+		(property "Reference" "R96"
+			(at 384.175 85.09 90)
+			(show_name no)
+			(do_not_autoplace no)
+			(effects
+				(font
+					(size 1.27 1.27)
+				)
+				(justify right)
+			)
+		)
+		(property "Value" "10"
+			(at 380.365 85.09 90)
+			(show_name no)
+			(do_not_autoplace no)
+			(effects
+				(font
+					(size 1.27 1.27)
+				)
+				(justify right)
+			)
+		)
+		(property "Footprint" ""
+			(at 377.444 82.804 90)
+			(hide yes)
+			(show_name no)
+			(do_not_autoplace no)
+			(effects
+				(font
+					(size 1.27 1.27)
+				)
+			)
+		)
+		(property "Datasheet" ""
+			(at 377.19 83.82 0)
+			(hide yes)
+			(show_name no)
+			(do_not_autoplace no)
+			(effects
+				(font
+					(size 1.27 1.27)
+				)
+			)
+		)
+		(property "Description" "Resistor, US symbol"
+			(at 377.19 83.82 0)
+			(hide yes)
+			(show_name no)
+			(do_not_autoplace no)
+			(effects
+				(font
+					(size 1.27 1.27)
+				)
+			)
+		)
+		(pin "2"
+		)
+		(pin "1"
+		)
+		(instances
+			(project "oomwoo-kicad"
+				(path "/dbcfb655-8d45-4808-9a74-2a0eb03372e8/2d8a25d6-58b7-409a-a3b1-0c610bb70760"
+					(reference "R96")
+					(unit 1)
+				)
+			)
+		)
+	)
+	(symbol
 		(lib_id "power:GND")
 		(at 291.465 217.17 0)
@@
 					(unit 1)
 				)
+			)
+		)
+	)
+	(symbol
+		(lib_id "Device:R_US")
+		(at 377.19 86.36 90)
+		(unit 1)
+		(body_style 1)
+		(exclude_from_sim no)
+		(in_bom yes)
+		(on_board yes)
+		(in_pos_files yes)
+		(dnp no)
+		(property "Reference" "R101"
+			(at 384.175 87.63 90)
+			(show_name no)
+			(do_not_autoplace no)
+			(effects
+				(font
+					(size 1.27 1.27)
+				)
+				(justify right)
+			)
+		)
+		(property "Value" "10"
+			(at 380.365 87.63 90)
+			(show_name no)
+			(do_not_autoplace no)
+			(effects
+				(font
+					(size 1.27 1.27)
+				)
+				(justify right)
+			)
+		)
+		(property "Footprint" ""
+			(at 377.444 85.344 90)
+			(hide yes)
+			(show_name no)
+			(do_not_autoplace no)
+			(effects
+				(font
+					(size 1.27 1.27)
+				)
+			)
+		)
+		(property "Datasheet" ""
+			(at 377.19 86.36 0)
+			(hide yes)
+			(show_name no)
+			(do_not_autoplace no)
+			(effects
+				(font
+					(size 1.27 1.27)
+				)
+			)
+		)
+		(property "Description" "Resistor, US symbol"
+			(at 377.19 86.36 0)
+			(hide yes)
+			(show_name no)
+			(do_not_autoplace no)
+			(effects
+				(font
+					(size 1.27 1.27)
+				)
+			)
+		)
+		(pin "2"
+		)
+		(pin "1"
+		)
+		(instances
+			(project "oomwoo-kicad"
+				(path "/dbcfb655-8d45-4808-9a74-2a0eb03372e8/2d8a25d6-58b7-409a-a3b1-0c610bb70760"
+					(reference "R101")
+					(unit 1)
+				)
