File: kicad/WHEEL-MOTORs .kicad_sch (KiCad schematic)
At the start: 32 parts, among them J12 WHEEL-MOTOR-RIGHT, J13 WHEEL-MOTOR-RIGHT, Q12 AO3401, Q13 2N3904, U14 DRV8870DDAR, U15 DRV8870DDAR

Commit message: Battery charging
Other:
- note added: "Isn't Diode reversed?"
Changed lines of the file:
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@@
+		)
+	)
+	(text "Isn't Diode reversed?"
+		(exclude_from_sim no)
+		(at 202.565 273.05 0)
+		(effects
+			(font
+				(size 1.27 1.27)
+			)
 		)
 	)
@@
 		)
 	)
+	(text "Isn't Diode reversed?"
+		(exclude_from_sim no)
+		(at 198.755 186.69 0)
+		(effects
+			(font
+				(size 1.27 1.27)
+			)
+		)
+	)

Commit message: Added Pi CM4/CM5
Parts:
- added U1: WHEEL-MOTOR-RIGHT, JLCImport:S7B-ZR_LF_SN, symbol JLCImport:S7B-ZR_LF_SN
- added U2: WHEEL-MOTOR-LEFT, JLCImport:S7B-ZR_LF_SN, symbol JLCImport:S7B-ZR_LF_SN
Connections:
- net VCC-5V-SYS renamed VCC-5V-REG
- no-connect marks 0 -> 14
Other:
- note added: "Waiting for the pinout"
- note removed: "Isn't Diode reversed?"

Commit message: Changed MCU to STM32G473VCT6
Parts:
- removed Q12: AO3401, oomwoo_altium:SOT23-3D, symbol DesignLibrary:WHEEL MOTOR_1_P-MOS-SOT23_DesignLibrary.SchLib
- removed Q13: 2N3904, oomwoo_altium:SOT23-3D, symbol DesignLibrary:WHEEL MOTOR_0_mirrored_NPN-SOT23_DesignLibrary.SchLib
- removed R88: 20K, oomwoo_altium:RES-0402, symbol DesignLibrary:WHEEL MOTOR_0_Resistor-1_DesignLibrary.SchLib
- removed R91: 1K, oomwoo_altium:RES-0402, symbol DesignLibrary:WHEEL MOTOR_0_Resistor-1_DesignLibrary.SchLib
- removed U1: WHEEL-MOTOR-RIGHT, JLCImport:S7B-ZR_LF_SN, symbol JLCImport:S7B-ZR_LF_SN
- removed U2: WHEEL-MOTOR-LEFT, JLCImport:S7B-ZR_LF_SN, symbol JLCImport:S7B-ZR_LF_SN
- C84: value 0.22uF -> 0.22uF/25V; footprint oomwoo_altium:CAP-0402 -> Capacitor_SMD:C_0603_1608Metric
- C86, C87, C88, C90, C91: footprint oomwoo_altium:CAP-0402 -> Capacitor_SMD:C_0603_1608Metric
- J13: value WHEEL-MOTOR-RIGHT -> WHEEL-MOTOR-LEFT
- R101, R102, R108, R109, R89, R90, R94, R95, R97, R98: footprint oomwoo_altium:RES-0402 -> Resistor_SMD:R_0603_1608Metric
- R83, R84, R87, R96: footprint oomwoo_altium:RES-0603 -> Resistor_SMD:R_0603_1608Metric
Connections:
- net VCC-5V-WHEEL is gone; now on net VCC-5V-REG: R87.2, R96.2
- no-connect marks 14 -> 0
Other:
- note removed: "Waiting for the pinout"

Commit message: STM32G473VCT6
Parts:
- removed C86, C90: 0.1uF, Capacitor_SMD:C_0603_1608Metric, symbol DesignLibrary:WHEEL MOTOR_3_Capacitor-1_DesignLibrary.SchLib
- removed C87, C91: 0.1uF, Capacitor_SMD:C_0603_1608Metric, symbol DesignLibrary:WHEEL MOTOR_2_Capacitor-1_DesignLibrary.SchLib
- removed J12: WHEEL-MOTOR-RIGHT, oomwoo_altium:CONN-SMD_5P-P1.50_ZX-ZH1.5-5PWT, symbol DesignLibrary:WHEEL MOTOR_0_HDRx5_DesignLibrary.SchLib
- removed J13: WHEEL-MOTOR-LEFT, oomwoo_altium:CONN-SMD_5P-P1.50_ZX-ZH1.5-5PWT, symbol DesignLibrary:WHEEL MOTOR_0_HDRx5_DesignLibrary.SchLib
- removed R101, R94: 4K7, Resistor_SMD:R_0603_1608Metric, symbol DesignLibrary:WHEEL MOTOR_0_Resistor-1_DesignLibrary.SchLib
- removed R102, R95: 1K, Resistor_SMD:R_0603_1608Metric, symbol DesignLibrary:WHEEL MOTOR_0_Resistor-1_DesignLibrary.SchLib
- removed R87, R96: 330R, Resistor_SMD:R_0603_1608Metric, symbol DesignLibrary:WHEEL MOTOR_0_Resistor-1_DesignLibrary.SchLib
- added MOT_L1, MOT_R1: S7B-ZR_LF_SN, JLCImport:S7B-ZR_LF_SN, symbol JLCImport:S7B-ZR_LF_SN
- added R49, R50: 10k, symbol Device:R_US
Connections:
- net GND: now also MOT_L1.4, MOT_R1.4, R49.2, R50.2
- net VCC-3V3-P: now also MOT_L1.6, MOT_R1.6
- net VCC-5V-REG: now also MOT_L1.3, MOT_R1.3
- net WHEEL-M-LEFT-ENCODE-A: now also MOT_L1.5
- net WHEEL-M-RIGHT-ENCODE-A: now also MOT_R1.5
- net at U14.6 (OUT1): now also MOT_R1.1
- net at U14.8 (OUT2): now also MOT_R1.2
- net at U15.6 (OUT1): now also MOT_L1.1
- net at U15.8 (OUT2): now also MOT_L1.2
- new net WHEEL-M-LEFT-DROP: MOT_L1.7, R50.1
- new net WHEEL-M-RIGHT-DROP: MOT_R1.7, R49.1
Other:
- note removed: "A"
- note removed: "GND"
- note removed: "M+"
- note removed: "M-"
- note removed: "VCC"

Commit message: RTC clock, signal integrity
Connections:
- net BAT-VCC renamed VM-VBAT
Changed lines of the file:
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@@
 		)
 	)
+	(global_label "VM-VBAT"
+		(shape input)
+		(at 267.97 123.19 90)
+		(fields_autoplaced yes)
+		(effects
+			(font
+				(size 1.27 1.27)
+			)
+			(justify left)
+		)
+		(property "Intersheetrefs" "${INTERSHEET_REFS}"
+			(at 267.97 111.6776 90)
+			(hide yes)
+			(show_name no)
+			(do_not_autoplace no)
+			(effects
+				(font
+					(size 1.27 1.27)
+				)
+				(justify left)
+			)
+		)
+	)
+	(global_label "VM-VBAT"
+		(shape input)
+		(at 267.97 209.55 90)
+		(fields_autoplaced yes)
+		(effects
+			(font
+				(size 1.27 1.27)
+			)
+			(justify left)
+		)
+		(property "Intersheetrefs" "${INTERSHEET_REFS}"
+			(at 267.97 198.0376 90)
+			(hide yes)
+			(show_name no)
+			(do_not_autoplace no)
+			(effects
+				(font
+					(size 1.27 1.27)
+				)
+				(justify left)
+			)
+		)
+	)
 	(hierarchical_label "WHEEL-M-RIGHT-DROP"
 		(shape output)
@@
 	)
 	(symbol
-		(lib_id "oomwoo-kicad-altium-import:BAT-VCC_BAR")
-		(at 267.97 209.55 180)
-		(unit 1)
-		(body_style 1)
-		(exclude_from_sim no)
-		(in_bom yes)
-		(on_board yes)
-		(in_pos_files yes)
-		(dnp no)
-		(property "Reference" "#PWR0566"
-			(at 267.97 209.55 0)
-			(hide yes)
-			(show_name no)
-			(do_not_autoplace no)
-			(effects
-				(font
-					(size 1.27 1.27)
-				)
-			)
-		)
-		(property "Value" "BAT-VCC"
-			(at 267.97 205.74 0)
-			(show_name no)
-			(do_not_autoplace no)
-			(effects
-				(font
-					(size 1.27 1.27)
-				)
-			)
-		)
-		(property "Footprint" ""
-			(at 267.97 209.55 0)
-			(show_name no)
-			(do_not_autoplace no)
-			(effects
-				(font
-					(size 1.27 1.27)
-				)
-			)
-		)
-		(property "Datasheet" ""
-			(at 267.97 209.55 0)
-			(show_name no)
-			(do_not_autoplace no)
-			(effects
-				(font
-					(size 1.27 1.27)
-				)
-			)
-		)
-		(property "Description" ""
-			(at 267.97 209.55 0)
-			(show_name no)
-			(do_not_autoplace no)
-			(effects
-				(font
-					(size 1.27 1.27)
-				)
-			)
-		)
-		(pin ""
-		)
-		(instances
-			(project "oomwoo-kicad"
-				(path "/dbcfb655-8d45-4808-9a74-2a0eb03372e8/dc7554d6-6a04-4f93-8cb8-7c364fc629ef"
-					(reference "#PWR0566")
-					(unit 1)
-				)
-			)
-		)
-	)
-	(symbol
 		(lib_name "WHEEL MOTOR_0_Resistor-1_DesignLibrary.SchLib_6")
 		(lib_id "DesignLibrary:WHEEL MOTOR_0_Resistor-1_DesignLibrary.SchLib")
@@
 					(unit 1)
 				)
-			)
-		)
-	)
-	(symbol
-		(lib_id "oomwoo-kicad-altium-import:BAT-VCC_BAR")
-		(at 267.97 123.19 180)
-		(unit 1)
-		(body_style 1)
-		(exclude_from_sim no)
-		(in_bom yes)
-		(on_board yes)
-		(in_pos_files yes)
-		(dnp no)
-		(property "Reference" "#PWR0565"
-			(at 267.97 123.19 0)
-			(hide yes)
-			(show_name no)
-			(do_not_autoplace no)
-			(effects
-				(font
-					(size 1.27 1.27)
-				)
-			)
-		)
-		(property "Value" "BAT-VCC"
-			(at 267.97 119.38 0)
-			(show_name no)
-			(do_not_autoplace no)
-			(effects
-				(font
-					(size 1.27 1.27)
-				)
-			)
-		)
-		(property "Footprint" ""
-			(at 267.97 123.19 0)
-			(show_name no)
-			(do_not_autoplace no)
-			(effects
-				(font
-					(size 1.27 1.27)
-				)
-			)
-		)
-		(property "Datasheet" ""
-			(at 267.97 123.19 0)
-			(show_name no)
-			(do_not_autoplace no)
-			(effects
-				(font
-					(size 1.27 1.27)
-				)
-			)
-		)
-		(property "Description" ""
-			(at 267.97 123.19 0)
-			(show_name no)
-			(do_not_autoplace no)
-			(effects
-				(font
-					(size 1.27 1.27)
-				)
-			)
-		)
-		(pin ""
-		)
-		(instances
-			(project "oomwoo-kicad"
-				(path "/dbcfb655-8d45-4808-9a74-2a0eb03372e8/dc7554d6-6a04-4f93-8cb8-7c364fc629ef"
-					(reference "#PWR0565")
-					(unit 1)
-				)
