File: kicad/CM5-GPIO.kicad_sch (KiCad schematic)
At the start: 18 parts, among them Q19 RTR030N05HZGTL, U3 74LVC1G07GW_125, U6 RT9742GGJ5

Commit message: Changed MCU to STM32G473VCT6
Parts:
- BOOT1: footprint (none) -> Connector_PinHeader_2.54mm:PinHeader_1x02_P2.54mm_Vertical
- C1, C2: value 100nF / 50V -> 100nF/10V
- C3: value 10u -> 10uf/10V
- C4: value 10uF/16V -> 10uF/10V
- R1: footprint (none) -> Resistor_SMD:R_0603_1608Metric
Changed lines of the file:
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@@
 			)
 		)
-		(property "Value" "100nF / 50V"
+		(property "Value" "100nF/10V"
 			(at 245.11 197.993 0)
 			(show_name no)
@@
 			)
 		)
-		(property "Value" "100nF / 50V"
+		(property "Value" "100nF/10V"
 			(at 231.14 198.755 90)
 			(show_name no)
@@
 			)
 		)
-		(property "Value" "10uF/16V"
+		(property "Value" "10uF/10V"
 			(at 312.928 307.467 90)
 			(show_name no)
@@
 			)
 		)
-		(property "Value" "10u"
+		(property "Value" "10uf/10V"
 			(at 355.346 175.133 0)
 			(show_name no)
@@
 			)
 		)
-		(property "Footprint" ""
+		(property "Footprint" "Resistor_SMD:R_0603_1608Metric"
 			(at 231.394 118.364 90)
 			(hide yes)
@@
 			)
 		)
-		(property "Footprint" ""
+		(property "Footprint" "Connector_PinHeader_2.54mm:PinHeader_1x02_P2.54mm_Vertical"
 			(at 354.33 201.295 0)
 			(hide yes)

Commit message: STM32G473VCT6
Parts:
- removed CONSOLE1: Conn_01x03_Pin, Connector_PinHeader_2.54mm:PinHeader_1x03_P2.54mm_Vertical, symbol Connector:Conn_01x03_Pin
- removed Q19: RTR030N05HZGTL, LIB_RTR030N05HZGTL:SOT95P280X100-3N, symbol SamacSys_Parts:RTR030N05HZGTL
- removed R1: 10, Resistor_SMD:R_0603_1608Metric, symbol Device:R_US
- removed R141: 100k, Resistor_SMD:R_0603_1608Metric, symbol Device:R_US
- added CONSOLE1: Conn_01x05_Pin, symbol Connector:Conn_01x05_Pin
- added Q13: IRLML6344TRPBF, JLCImport:IRLML6344TRPBF, symbol JLCImport:IRLML6344TRPBF
Connections:
- net CONSOLE_RXD: now also CONSOLE1.4 (Pin_4)
- net CONSOLE_TXD: now also CONSOLE1.5 (Pin_5)
- net GND: now also CONSOLE1.1 (Pin_1), Q13.2 (S)
- net PMIC_EN: now also Q13.1 (G)
- net SPI0_SCLK: now also Module1.38 (GPIO11)
- net at Module1.99 (PMIC_ENABLE): now also Q13.3 (D)
- net AUDIO_OUT_L renamed UART4_TX
- net AUDIO_OUT_R renamed UART4_RX
- net UART0_RX renamed SDA1
- net UART0_TX renamed SCL1
- no-connect marks 26 -> 28
Other:
- note added: "Compatible with TTL-234X-3V3 smart cable"
- note added: "UART3_RX on the CM4"
- note added: "UART3_TX on the CM4"
- note added: "UART5_RX on the CM4"
- note added: "UART5_TX on the CM4"

Commit message: External RTC; IR light; side sensors
Parts:
- added Q18: IRLML6344TRPBF, JLCImport:IRLML6344TRPBF, symbol JLCImport:IRLML6344TRPBF
- added R33, R46: 100kOhm, Resistor_SMD:R_0603_1608Metric_Pad0.98x0.95mm_HandSolder, symbol Device:R_US
Connections:
- net GND: now also Q18.2 (S), R33.2, R46.2
- net PMIC_EN: now also R46.1
- net at Module1.99 (PMIC_ENABLE), Q13.3 (D): now also Q18.3 (D)
- new net PMIC_EN2: Q18.1 (G), R33.1
