File: kicad/Front Sensors.kicad_sch (KiCad schematic)
At the start: 14 parts

Commit message: External RTC; IR light; side sensors
Parts:
- removed C7, C8: 4.7uF/10V, symbol Device:C_Small
- removed IR-L1, IR-R1: ZX-ZH1_5-4PWT, JLCImport:ZX-ZH1_5-4PWT, symbol JLCImport:ZX-ZH1_5-4PWT
- added C123: 10uF/50V, Capacitor_SMD:C_0603_1608Metric, symbol JLCImport:CL21A106KBYQNNE
- added C90, C91: 4.7uF/10V, symbol Device:C_Small
- added IR-F1, IR-F2: ZX-ZH1_5-4PWT, JLCImport:ZX-ZH1_5-4PWT, symbol JLCImport:ZX-ZH1_5-4PWT
- added Q19: IRLML6344TRPBF, JLCImport:IRLML6344TRPBF, symbol JLCImport:IRLML6344TRPBF
- added U17: ZX-ZH1_5-2PWT, JLCImport:ZX-ZH1_5-2PWT, symbol JLCImport:ZX-ZH1_5-2PWT
Connections:
- net GND: now also C123.2, C90.2, C91.2, IR-F1.2, IR-F1.3, IR-F1.5, IR-F1.6, IR-F2.2, IR-F2.3, IR-F2.5, IR-F2.6, Q19.2 (S), U17.3, U17.4
- net VCC-3V3-P: now also C90.1, C91.1, IR-F1.1, IR-F2.1, U17.1
- new net: C123.1, Q19.3 (D), U17.2
- new net IR-F-RX1: IR-F1.4
- new net IR-F-RX2: IR-F2.4
- new net LIGHT-ON: Q19.1 (G)
Other:
- note added: "2 IR RECEIVERS"
- note added: "IR LIGHT"
- note added: "https://thepihut.com/products/850nm-ir-led-modules?srsltid=AfmBOorZ0hl4HylQHd5JbNfaA7bqJMbzrmY0bn7Mm12pD_mKEoiRE0nX"
- note removed: "2 CAMERAS"
- note removed: "2 SET IR EMITTERS + IR RECEIVERS"
- note removed: "LED"
- moved on the sheet: C6, R2, R36, R5, R6, R61, R62, R7, VL-L1, VL-R1
