File: kicad/SIDE-PROXIMITY-IR-SENSOR .kicad_sch (KiCad schematic)
At the start: 10 parts, among them J8 SIDE-PROXI-LEFT, J9 SIDE-PROXI-RIGHT, Q6 2N3904, Q7 2N3904

Commit message: Battery charging
Other:
- note added: "What sensor is used for Proxy?"
Changed lines of the file:
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@@
+		)
+	)
+	(text "What sensor is used for Proxy?"
+		(exclude_from_sim no)
+		(at 265.43 188.595 0)
+		(effects
+			(font
+				(size 1.27 1.27)
+			)
 		)
 	)

Commit message: Added Pi CM4/CM5
Connections:
- net VCC-5V-SYS renamed VCC-5V-REG
Changed lines of the file:
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@@
 	)
 	(symbol
-		(lib_id "oomwoo-kicad-altium-import:VCC-5V-SYS_BAR")
+		(lib_id "oomwoo-kicad-altium-import:VCC-5V-REG_BAR")
 		(at 302.26 205.105 180)
 		(unit 1)
@@
 		(in_pos_files yes)
 		(dnp no)
-		(property "Reference" "#PWR0541"
-			(at 302.26 205.105 0)
-			(hide yes)
-			(show_name no)
-			(do_not_autoplace no)
-			(effects
-				(font
-					(size 1.27 1.27)
-				)
-			)
-		)
-		(property "Value" "VCC-5V-SYS"
+		(property "Reference" "#PWR067"
+			(at 302.26 205.105 0)
+			(hide yes)
+			(show_name no)
+			(do_not_autoplace no)
+			(effects
+				(font
+					(size 1.27 1.27)
+				)
+			)
+		)
+		(property "Value" "VCC-5V-REG"
 			(at 302.26 201.295 0)
 			(show_name no)
@@
 			(project "oomwoo-kicad"
 				(path "/dbcfb655-8d45-4808-9a74-2a0eb03372e8/5e1370fc-da76-42ab-8a06-17e0cb799727"
-					(reference "#PWR0541")
+					(reference "#PWR067")
 					(unit 1)
 				)
@@
 	)
 	(symbol
-		(lib_id "oomwoo-kicad-altium-import:VCC-5V-SYS_BAR")
+		(lib_id "oomwoo-kicad-altium-import:VCC-5V-REG_BAR")
 		(at 302.26 128.905 180)
 		(unit 1)
@@
 		(in_pos_files yes)
 		(dnp no)
-		(property "Reference" "#PWR0540"
-			(at 302.26 128.905 0)
-			(hide yes)
-			(show_name no)
-			(do_not_autoplace no)
-			(effects
-				(font
-					(size 1.27 1.27)
-				)
-			)
-		)
-		(property "Value" "VCC-5V-SYS"
+		(property "Reference" "#PWR066"
+			(at 302.26 128.905 0)
+			(hide yes)
+			(show_name no)
+			(do_not_autoplace no)
+			(effects
+				(font
+					(size 1.27 1.27)
+				)
+			)
+		)
+		(property "Value" "VCC-5V-REG"
 			(at 302.26 125.095 0)
 			(show_name no)
@@
 			(project "oomwoo-kicad"
 				(path "/dbcfb655-8d45-4808-9a74-2a0eb03372e8/5e1370fc-da76-42ab-8a06-17e0cb799727"
-					(reference "#PWR0540")
+					(reference "#PWR066")
 					(unit 1)
 				)

Commit message: Changed MCU to STM32G473VCT6
Parts:
- R75, R76, R77, R78, R79, R80: footprint oomwoo_altium:RES-0402 -> Resistor_SMD:R_0603_1608Metric
Changed lines of the file:
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@@
 			)
 		)
-		(property "Footprint" "oomwoo_altium:RES-0402"
+		(property "Footprint" "Resistor_SMD:R_0603_1608Metric"
 			(at 266.7 243.205 0)
 			(hide yes)
@@
 			)
 		)
-		(property "Footprint" "oomwoo_altium:RES-0402"
+		(property "Footprint" "Resistor_SMD:R_0603_1608Metric"
 			(at 287.02 212.725 0)
 			(hide yes)
@@
 			)
 		)
-		(property "Footprint" "oomwoo_altium:RES-0402"
+		(property "Footprint" "Resistor_SMD:R_0603_1608Metric"
 			(at 297.18 149.225 0)
 			(hide yes)
@@
 			)
 		)
-		(property "Footprint" "oomwoo_altium:RES-0402"
+		(property "Footprint" "Resistor_SMD:R_0603_1608Metric"
 			(at 297.18 225.425 0)
 			(hide yes)
@@
 			)
 		)
-		(property "Footprint" "oomwoo_altium:RES-0402"
+		(property "Footprint" "Resistor_SMD:R_0603_1608Metric"
 			(at 287.02 136.525 0)
 			(hide yes)
@@
 			)
 		)
-		(property "Footprint" "oomwoo_altium:RES-0402"
+		(property "Footprint" "Resistor_SMD:R_0603_1608Metric"
 			(at 266.7 167.005 0)
 			(hide yes)

Commit message: STM32G473VCT6
Parts:
- removed Q6, Q7: 2N3904, oomwoo_altium:SOT23-3D, symbol DesignLibrary:SIDE-PROXI_0_NPN-SOT23_DesignLibrary.SchLib
- removed R77, R80: 1K, Resistor_SMD:R_0603_1608Metric, symbol DesignLibrary:SIDE-PROXI_0_Resistor-1_DesignLibrary.SchLib
- added Q30: RTR030N05HZGTL, LIB_RTR030N05HZGTL:SOT95P280X100-3N, symbol SamacSys_Parts:RTR030N05HZGTL
- added Q4: IRLML6344TRPBF, JLCImport:IRLML6344TRPBF, symbol JLCImport:IRLML6344TRPBF
- added R69, R70: 10, Resistor_SMD:R_0603_1608Metric_Pad0.98x0.95mm_HandSolder, symbol Device:R_US
Connections:
- net TOUCHL: now also R69.2
- net TOUCHR: now also R70.2
- net at R76.2: now also Q30.3 (D)
- net at R79.2: now also Q4.3 (D)
- net at J9.5: now also Q4.2 (S)
- net at J8.5: now also Q30.2 (S)
- new net: Q4.1 (G), R70.1
- new net: Q30.1 (G), R69.1

Commit message: External RTC; IR light; side sensors
Parts:
- removed J8: SIDE-PROXI-LEFT, oomwoo_altium:CONN-SMD_5P-P1.50_ZX-ZH1.5-5PWT, symbol DesignLibrary:SIDE-PROXI_0_HDRx5_DesignLibrary.SchLib
- removed J9: SIDE-PROXI-RIGHT, oomwoo_altium:CONN-SMD_5P-P1.50_ZX-ZH1.5-5PWT, symbol DesignLibrary:SIDE-PROXI_0_HDRx5_DesignLibrary.SchLib
- removed Q30: RTR030N05HZGTL, LIB_RTR030N05HZGTL:SOT95P280X100-3N, symbol SamacSys_Parts:RTR030N05HZGTL
- removed Q4: IRLML6344TRPBF, JLCImport:IRLML6344TRPBF, symbol JLCImport:IRLML6344TRPBF
- removed R69, R70: 10, Resistor_SMD:R_0603_1608Metric_Pad0.98x0.95mm_HandSolder, symbol Device:R_US
- removed R75, R78: 1K, Resistor_SMD:R_0603_1608Metric, symbol DesignLibrary:SIDE-PROXI_0_Resistor-1_DesignLibrary.SchLib
- removed R76, R79: 2K, Resistor_SMD:R_0603_1608Metric, symbol DesignLibrary:SIDE-PROXI_2_Resistor-1_DesignLibrary.SchLib
- added C18, C39: 4.7uF/10V, symbol Device:C_Small
- added IR-L1, IR-R1: ZX-ZH1_5-4PWT, JLCImport:ZX-ZH1_5-4PWT, symbol JLCImport:ZX-ZH1_5-4PWT
Connections:
- net GND: now also C18.2, C39.2, IR-L1.2, IR-L1.5, IR-L1.6, IR-R1.2, IR-R1.5, IR-R1.6
- net VCC-3V3-P: now also C18.1, C39.1, IR-L1.1, IR-R1.1
- new net IR-L-RX: IR-L1.4
- new net IR-L-TX: IR-L1.3
- new net IR-R-RX: IR-R1.4
- new net IR-R-TX: IR-R1.3
Other:
- note added: "LED"
- note added: "RECEIVER"
- note added: "VDD"
- note removed: "3V3"
- note removed: "5V"
- note removed: "IRF"
- note removed: "TOUCHL"
- note removed: "TOUCHR"
- note removed: "What sensor is used for Proxy?"
