File: kicad/side-sensors/IR sensor.kicad_sch (KiCad schematic)
At the start: 17 parts, among them Q7 IRLML6344TRPBF, U1 TLC555CDR, U2 SN74LVC2G08DCTR

Commit message: Side sensor VL6180
Parts:
- removed C18: 4.7uF/10V, symbol Device:C_Small
- removed IR-L1: ZX-ZH1_5-4PWT, JLCImport:ZX-ZH1_5-4PWT, symbol JLCImport:ZX-ZH1_5-4PWT
- removed IR1: TSAL6200, JLCImport:TSAL6200, symbol JLCImport:TSAL6200
- removed Q7: IRLML6344TRPBF, JLCImport:IRLML6344TRPBF, symbol JLCImport:IRLML6344TRPBF
- removed U1: TLC555CDR, JLCImport:TLC555CDR, symbol JLCImport:TLC555CDR
- removed U2: SN74LVC2G08DCTR, JLCImport:SN74LVC2G08DCTR, symbol JLCImport:SN74LVC2G08DCTR
- added C6: 1uF/10V, symbol Device:C_Small
- added SIDE-PROXI1: ZX-ZH1_5-7PWT, JLCImport:ZX-ZH1_5-7PWT, symbol JLCImport:ZX-ZH1_5-7PWT
- added U1: VL6180V1NR_1, JLCImport:VL6180V1NR_1, symbol JLCImport:VL6180V1NR_1
- added U2: TLV70028DCKR, JLCImport:TLV70028DCKR, symbol JLCImport:TLV70028DCKR
- C3: value 1nF/10V -> 100nF/10V
- C4: value 10nF/10V -> 4.7/6.3V
- C5: value 100nF/10V -> 4.7/6.3V
- R2: value 18.2k -> 47k
- R3: value 1k -> 47k
- R4: value 100 -> 47k
- R5: value 10 -> 47k
Connections:
- net IR-RX is gone; now on net IR-RX-OUT: RX1.1 (OUT)
- net GND: now also C6.2, SIDE-PROXI1.2, SIDE-PROXI1.8, SIDE-PROXI1.9, U1.12 (GND), U2.2 (GND)
- net IR-RX-OUT: now also SIDE-PROXI1.3
- net VCC-3V3-P: now also R2.2, R5.2, SIDE-PROXI1.1, U2.1 (IN), U2.3 (EN)
- net +2V8: now reaches C3.1
- net +2V8: now also C4.1, C6.1, U1.10 (AVDD), U1.8 (AVDD_VCSEL), U2.5 (OUT); no longer R2.1
- net SDA: now reaches R4.1
- net SDA: now also SIDE-PROXI1.7, U1.6 (SDA)
- net SCL: now reaches R5.1
- net SCL: now also SIDE-PROXI1.6, U1.5 (SCL)
- net CE: now reaches R3.1
- net CE: now also SIDE-PROXI1.5, U1.4 (GPIO0/CE); no longer R2.2
- new net GPIO1: R2.1, SIDE-PROXI1.4, U1.1 (GPIO1)
- no-connect marks 0 -> 6
Other:
- note removed: "GND"
- note removed: "LED"
- note removed: "RECEIVER"
- note removed: "VDD"
- note removed: "~ 20mA"
