File: kicad/main/Main.kicad_pcb (KiCad board)
At the start: 4 copper layers, 116 x 98.7 mm, 290 parts, among them CN1 EV2400, CN2 S16B-PHDSS_LF_SN, J1 BATTERY, J10 WATER-PUMP, J11 MAIN BRUSH, J12 WHEEL-MOTOR-RIGHT, J13 WHEEL-MOTOR-LEFT, J14 MAIN-FAN, J15 SIDE BRUSH, J17 LiDAR, J18 SPEAKER2, J21 STM-PROGRAM, J23 STM32-PROGRAM, J4 ANTI-FALL-LEFT-DOWN, J5 ANTI-FALL-RIGHT-DOWN, J8 SIDE-PROXI-LEFT, J9 SIDE-PROXI-RIGHT, K2 kEY-4, K3 kEY-4, Q1 AO4407A, Q11 2N3904, Q15 2N3904, Q20 AO3400, Q22 2N3904, Q23 2N3904, Q26 CSD17581Q3A, Q27 CSD17581Q3A, Q28 CSD17581Q3A, Q29 CSD17581Q3A, Q3 PNP-SOT23, Q6 2N3904, Q7 2N3904, Q8 AO3401, Q9 2N3904, U11 MAX98357AETE_T, U13 STM32G473VCT6, U14 DRV8870DDAR, U15 DRV8870DDAR, U18 DRV8870DDAR, U19 ICM-42607-P, U20 DRV8870DDAR, U4 SY8089A, U5 SY8089A, U6 RT9742GGJ5, U7 BQ25792RQMR, U9 ICS-43434_C5656610, X1 ABM3-8_000MHZ-D2Y-T

Commit message: Fix edge cut; no-CM STEP
Parts:
- removed C104, C85, C89, C93: 100uF, oomwoo_altium:CAP-SMD_BD6.3-L6.6-W6.6-FD
- removed C40: 100nF/50V, Capacitor_SMD:C_0603_1608Metric
- removed C42: 47pF/10V, Capacitor_SMD:C_0603_1608Metric
- removed C44, C46: 22uF/10V, Capacitor_SMD:C_0805_2012Metric
- removed C7: 10uF/10V, Capacitor_SMD:C_0603_1608Metric
- removed CN1: EV2400, JLCImport:22053041_C5271241
- removed D32, D33: BZT52C12T-7, JLCImport:BZT52C12T-7
- removed D4: SMCJ18A-13-F, JLCImport:SMCJ18A-13-F
- removed J1: BATTERY, oomwoo_altium:CONN-SMD_4P-P2.00_XUNPU_WAFER-PH2.0-4PWB
- removed J10: WATER-PUMP, oomwoo_altium:CONN-SMD_2P-P1.50_ZX-ZH1.5-2PWT
- removed J11: MAIN BRUSH, oomwoo_altium:CONN-SMD_2P-P2.00_XUNPU_WAFER-PH2.0-2PWB
- removed J12: WHEEL-MOTOR-RIGHT, oomwoo_altium:CONN-SMD_5P-P1.50_ZX-ZH1.5-5PWT
- removed J13: WHEEL-MOTOR-LEFT, oomwoo_altium:CONN-SMD_5P-P1.50_ZX-ZH1.5-5PWT
- removed J14: MAIN-FAN, oomwoo_altium:CONN-SMD_4P-P2.00_XUNPU_WAFER-PH2.0-4PWB
- removed J15: SIDE BRUSH, oomwoo_altium:CONN-SMD_2P-P1.50_ZX-ZH1.5-2PWT
- removed J17: LiDAR, oomwoo_altium:CONN-SMD_5P-P1.25_XUNPU_WAFER-GH1.25-5PWB
- removed J18: SPEAKER2, oomwoo_altium:CONN-SMD_2P-P1.00_HX-1.0-2P-WT
- removed J21: STM-PROGRAM, Connector_PinHeader_2.54mm:PinHeader_1x05_P2.54mm_Vertical
- removed J23: STM32-PROGRAM, oomwoo_altium:HDR1X5
- removed J4: ANTI-FALL-LEFT-DOWN, oomwoo_altium:CONN-SMD_8P-P1.50_ZX-ZH1.5-8PWT
- removed J5: ANTI-FALL-RIGHT-DOWN, oomwoo_altium:CONN-SMD_8P-P1.50_ZX-ZH1.5-8PWT
- removed J8: SIDE-PROXI-LEFT, oomwoo_altium:CONN-SMD_5P-P1.50_ZX-ZH1.5-5PWT
- removed J9: SIDE-PROXI-RIGHT, oomwoo_altium:CONN-SMD_5P-P1.50_ZX-ZH1.5-5PWT
- removed L1: 6.8uH, JLCImport:IHLP2525CZER6R8M01
- removed L4: 2.2uH, oomwoo_altium:IND-SMD_L4.4-W4.2
- removed Q15, Q22, Q23: 2N3904, oomwoo_altium:SOT23-3D
- removed Q26, Q27, Q28, Q29: CSD17581Q3A, CSD17581Q3A:TRANS_CSD17581Q3A
- removed R11, R20: 100K, Resistor_SMD:R_0603_1608Metric
- removed R114, R79: 2K, Resistor_SMD:R_0603_1608Metric
- removed R123, R77, R78: 1K, Resistor_SMD:R_0603_1608Metric
- removed R17: 450K, Resistor_SMD:R_0603_1608Metric
- removed R3: 1kOhm, Resistor_SMD:R_0603_1608Metric_Pad0.98x0.95mm_HandSolder
- removed R4: 1k, Resistor_SMD:R_0603_1608Metric_Pad0.98x0.95mm_HandSolder
- removed R42: 158k, Resistor_SMD:R_0603_1608Metric
- removed R43: 30.1k, Resistor_SMD:R_0603_1608Metric
- removed R58, R59: 100, Resistor_SMD:R_0603_1608Metric
- removed R69, R70: 10K, Resistor_SMD:R_0603_1608Metric
- removed R87: 330R, Resistor_SMD:R_0603_1608Metric
- removed U4: SY8089A, oomwoo_altium:SOT5P95B160_300H130
- added C102: 100nF/50V, Capacitor_SMD:C_0603_1608Metric, F.Cu at (109.1, 118.4)
- added C106: 10uF/50V, Capacitor_SMD:C_0603_1608Metric, F.Cu at (107.4, 118.4)
- added C107: 100nF/50V, Capacitor_SMD:C_0603_1608Metric, B.Cu at (111.9, 120.2)
- added C111: 100nF/50V, Capacitor_SMD:C_0603_1608Metric, F.Cu at (112.6, 114.3)
- added C112: 1.2nF/50V, Capacitor_SMD:C_0603_1608Metric, B.Cu at (117.2, 118.8)
- added C113: 10uF/50V, Capacitor_SMD:C_0603_1608Metric, F.Cu at (115.3, 122.1)
- added C114: 10uF/50V, Capacitor_SMD:C_0603_1608Metric, F.Cu at (115.3, 123.7)
- added C115: 10uF/50V, Capacitor_SMD:C_0603_1608Metric, F.Cu at (106.1, 107.0)
- added C116: 10uF/50V, Capacitor_SMD:C_0603_1608Metric, F.Cu at (107.8, 107.0)
- added C117: 100nF/50V, Capacitor_SMD:C_0603_1608Metric, F.Cu at (109.4, 107.0)
- added C118: 100nF/50V, Capacitor_SMD:C_0603_1608Metric, B.Cu at (111.3, 108.8)
- added C119: 100nF/50V, Capacitor_SMD:C_0603_1608Metric, F.Cu at (112.4, 102.8)
- added C120: 1.2nF/50V, Capacitor_SMD:C_0603_1608Metric, B.Cu at (117.1, 107.3)
- added C121: 10uF/50V, Capacitor_SMD:C_0603_1608Metric, F.Cu at (115.2, 110.8)
- added C122: 10uF/50V, Capacitor_SMD:C_0603_1608Metric, F.Cu at (115.2, 112.4)
- added C123: 10uF/50V, Capacitor_SMD:C_0603_1608Metric, B.Cu at (185.5, 69.0)
- added C125: 1nF/50V, Capacitor_SMD:C_0603_1608Metric, F.Cu at (108.6, 87.1)
- added C126: 1nF/50V, Capacitor_SMD:C_0603_1608Metric, B.Cu at (116.9, 96.2)
- added C18: GRM31CR61A107MEA8L, JLCImport:GRM31CR61A107MEA8L, B.Cu at (116.6, 111.6)
- added C39: JBLM2101M025C058RTM_100UF_25V, JLCImport:JBLM2101M025C058RTM_100UF_25V, F.Cu at (103.0, 149.4)
- added C41: 100nF/50V, Capacitor_SMD:C_0603_1608Metric, B.Cu at (180.6, 88.0)
- added C43: 100nF/50V, Capacitor_SMD:C_0603_1608Metric, B.Cu at (179.0, 88.0)
- added C45: 10uF/10V, Capacitor_SMD:C_0603_1608Metric, B.Cu at (174.2, 88.0)
- added C48: 100nF/50V, Capacitor_SMD:C_0603_1608Metric, B.Cu at (177.4, 88.0)
- added C49: 100nF/50V, Capacitor_SMD:C_0603_1608Metric, B.Cu at (175.8, 88.0)
- added C50: 100nF/50V, Capacitor_SMD:C_0603_1608Metric, B.Cu at (186.8, 85.5)
- added C52: 18pF/10V, Capacitor_SMD:C_0603_1608Metric, F.Cu at (153.0, 99.3)
- added C53: 18pF/10V, Capacitor_SMD:C_0603_1608Metric, F.Cu at (153.0, 96.6)
- added C56: 100nF/10V, Capacitor_SMD:C_0603_1608Metric, B.Cu at (142.1, 98.5)
- added C57: 100nF/10V, Capacitor_SMD:C_0603_1608Metric, B.Cu at (151.6, 94.7)
- added C94: 10uF/35V, Capacitor_SMD:C_0603_1608Metric, F.Cu at (105.4, 87.1)
- added C95: 10uF/50V, Capacitor_SMD:C_0603_1608Metric, F.Cu at (105.8, 118.4)
- added CN2: EV2400, JLCImport:A2543WV-4P, F.Cu at (124.4, 96.2)
- added CONTACT_CHGR1: WAFER-PH2_0-4PWB, JLCImport:WAFER-PH2_0-4PWB, F.Cu at (96.4, 80.3)
- added D1: TVS2200DRVR, JLCImport:TVS2200DRVR, F.Cu at (113.1, 83.2)
- added D37: SS34, oomwoo_altium:SMA, B.Cu at (176.1, 99.6)
- added D38: SS34, oomwoo_altium:SMA, B.Cu at (191.3, 100.1)
- added D39: BZT52C12T-7, JLCImport:BZT52C12T-7, F.Cu at (106.9, 87.0)
- added D40: BZT52C12T-7, JLCImport:BZT52C12T-7, B.Cu at (115.2, 96.0)
- added IC5: TPS25730DREFR, LIB_TPS25730DREFR:TPS25730DREFR, B.Cu at (106.3, 113.8)
- added IR-F1: ZX-ZH1_5-4PWT, JLCImport:ZX-ZH1_5-4PWT, F.Cu at (142.2, 150.0)
- added IR-F2: ZX-ZH1_5-4PWT, JLCImport:ZX-ZH1_5-4PWT, F.Cu at (152.5, 150.0)
- added J2: 1-2199119-5, 1-2199119-5:TE_1-2199119-5, F.Cu at (180.8, 87.2)
- added L2: CYA0630-3_3UH, JLCImport:CYA0630-3_3UH, F.Cu at (123.0, 119.2)
- added L3: CYA0630-3_3UH, JLCImport:CYA0630-3_3UH, F.Cu at (123.0, 107.9)
- added LIDAR1: WAFER-GH1_25-6PWB, JLCImport:WAFER-GH1_25-6PWB, F.Cu at (202.8, 99.9)
- added LIGHT1: ZX-ZH1_5-2PWT, JLCImport:ZX-ZH1_5-2PWT, F.Cu at (189.1, 70.2)
- added MAIN_BRUSH1: ZX-ZH1_5-2PWT, JLCImport:ZX-ZH1_5-2PWT, F.Cu at (201.9, 127.0)
- added MAIN_FAN1: WAFER-PH2_0-4PWB, JLCImport:WAFER-PH2_0-4PWB, F.Cu at (96.4, 124.9)
- added MCU_IO1: HC-PM254-8_5H-2X12PS, JLCImport:HC-PM254-8_5H-2X12PS, F.Cu at (174.8, 140.6)
- added MOT_L1: ZX-ZH1_5-7PWT, JLCImport:ZX-ZH1_5-7PWT, F.Cu at (95.7, 138.7)
- added MOT_R1: ZX-ZH1_5-7PWT, JLCImport:ZX-ZH1_5-7PWT, F.Cu at (201.9, 138.6)
- added MP1: M3 x 1.5mm, MountingHole:MountingHole_3.2mm_M3_Pad, F.Cu at (202.4, 70.0)
- added MP2: M3 x 1.5mm, MountingHole:MountingHole_3.2mm_M3_Pad, F.Cu at (202.4, 150.0)
- added MP3: M3 x 1.5mm, MountingHole:MountingHole_3.2mm_M3_Pad, F.Cu at (95.0, 150.0)
- added MP4: M3 x 1.5mm, MountingHole:MountingHole_3.2mm_M3_Pad, F.Cu at (95.0, 70.0)
- added PUMP1: ZX-ZH1_5-2PWT, JLCImport:ZX-ZH1_5-2PWT, F.Cu at (201.9, 111.7)
- added Q10: IRLML6344TRPBF, JLCImport:IRLML6344TRPBF, F.Cu at (194.3, 83.4)
- added Q12: IRLML6344TRPBF, JLCImport:IRLML6344TRPBF, F.Cu at (103.5, 81.7)
- added Q13: IRLML6344TRPBF, JLCImport:IRLML6344TRPBF, F.Cu at (135.5, 120.4)
- added Q14: IRLML6344TRPBF, JLCImport:IRLML6344TRPBF, B.Cu at (112.0, 68.8)
- added Q18: IRLML6344TRPBF, JLCImport:IRLML6344TRPBF, F.Cu at (135.5, 124.2)
- added Q19: IRLML6344TRPBF, JLCImport:IRLML6344TRPBF, B.Cu at (188.4, 68.6)
- added Q21: SQJ844AEP-T1_GE3, JLCImport:SQJ844AEP-T1_GE3, F.Cu at (110.1, 98.7)
- added Q4: SQJ844AEP-T1_GE3, JLCImport:SQJ844AEP-T1_GE3, F.Cu at (110.1, 92.2)
- added Q5: IRLML6344TRPBF, JLCImport:IRLML6344TRPBF, B.Cu at (198.6, 94.7)
- added R117: 10, Resistor_SMD:R_0603_1608Metric, B.Cu at (159.0, 115.6)
- added R134: 10, Resistor_SMD:R_0603_1608Metric, B.Cu at (149.6, 92.1)
- added R135: 100k, Resistor_SMD:R_0603_1608Metric, B.Cu at (145.9, 96.7)
- added R143: 12k, Resistor_SMD:R_0603_1608Metric, B.Cu at (120.5, 118.8)
- added R144: 69.8k, Resistor_SMD:R_0603_1608Metric, B.Cu at (120.5, 120.4)
- added R145: 22.1k, Resistor_SMD:R_0603_1608Metric, B.Cu at (117.2, 120.4)
- added R146: 10, Resistor_SMD:R_0603_1608Metric, F.Cu at (115.8, 102.8)
- added R147: 20k, Resistor_SMD:R_0603_1608Metric, B.Cu at (120.5, 107.3)
- added R148: 12k, Resistor_SMD:R_0603_1608Metric, B.Cu at (120.5, 109.0)
- added R149: 2.2k, Resistor_SMD:R_0603_1608Metric, B.Cu at (117.1, 109.0)
- added R150: 15k, Resistor_SMD:R_0603_1608Metric, B.Cu at (173.1, 106.1)
- added R151: 50k, Resistor_SMD:R_0603_1608Metric, B.Cu at (171.5, 106.1)
- added R152: 15k, Resistor_SMD:R_0603_1608Metric, B.Cu at (188.7, 105.8)
- added R153: 100k, Resistor_SMD:R_0603_1608Metric, B.Cu at (187.1, 105.8)
- added R30: 330, Resistor_SMD:R_0603_1608Metric, B.Cu at (202.4, 90.3)
- added R35: 330, Resistor_SMD:R_0603_1608Metric, B.Cu at (202.4, 76.3)
- added R38: 10k, Resistor_SMD:R_0603_1608Metric, B.Cu at (202.4, 88.2)
- added R39: 10k, Resistor_SMD:R_0603_1608Metric, B.Cu at (202.4, 86.3)
- added R41: 10k, Resistor_SMD:R_0603_1608Metric, B.Cu at (202.4, 84.4)
- added R44: 10k, Resistor_SMD:R_0603_1608Metric, B.Cu at (202.4, 78.3)
- added R46: 100kOhm, Resistor_SMD:R_0603_1608Metric, F.Cu at (138.8, 120.4)
- added R47: 10kOhm, Resistor_SMD:R_0603_1608Metric, F.Cu at (198.6, 100.6)
- added R48: 10, Resistor_SMD:R_0603_1608Metric, B.Cu at (172.3, 87.7)
- added R49: 10k, Resistor_SMD:R_0603_1608Metric, B.Cu at (203.7, 134.4)
- added R50: 10k, Resistor_SMD:R_0603_1608Metric, B.Cu at (94.2, 143.0)
- added R51: 10, Resistor_SMD:R_0603_1608Metric, F.Cu at (135.2, 106.6)
- added R52: 10, Resistor_SMD:R_0603_1608Metric, F.Cu at (135.2, 103.3)
- added R53: 10, Resistor_SMD:R_0603_1608Metric, F.Cu at (135.2, 104.9)
- added R54: 10, Resistor_SMD:R_0603_1608Metric, F.Cu at (135.2, 109.9)
- added R55: 10, Resistor_SMD:R_0603_1608Metric, F.Cu at (135.2, 111.6)
- added R56: 10k, Resistor_SMD:R_0603_1608Metric, B.Cu at (183.7, 88.0)
- added R61: 47k, Resistor_SMD:R_0603_1608Metric, B.Cu at (132.9, 151.2)
- added R62: 47k, Resistor_SMD:R_0603_1608Metric, B.Cu at (134.5, 151.2)
- added R63: 10, Resistor_SMD:R_0603_1608Metric, F.Cu at (135.2, 108.2)
- added R64: 10, Resistor_SMD:R_0603_1608Metric, B.Cu at (159.0, 119.1)
- added R65: 10, Resistor_SMD:R_0603_1608Metric, F.Cu at (135.1, 99.9)
- added R66: 10, Resistor_SMD:R_0603_1608Metric, F.Cu at (135.2, 98.2)
- added SDCARD2: 1040310811, JLCImport:1040310811, B.Cu at (141.2, 82.9)
- added SIDE-L1: ZX-ZH1_5-7PWT, JLCImport:ZX-ZH1_5-7PWT, F.Cu at (114.4, 150.0)
- added SIDE-R1: ZX-ZH1_5-7PWT, JLCImport:ZX-ZH1_5-7PWT, F.Cu at (180.3, 149.9)
- added SIDE_BRUSH1: ZX-ZH1_5-2PWT, JLCImport:ZX-ZH1_5-2PWT, F.Cu at (201.9, 119.3)
- added SPK1: ZX-ZH1_5-2PWT, JLCImport:ZX-ZH1_5-2PWT, F.Cu at (107.6, 69.8)
- added STM_DEBUG1: Conn_01x05_Pin, Connector_PinHeader_2.54mm:PinHeader_1x05_P2.54mm_Vertical, F.Cu at (121.9, 125.6)
- added U1: PCF85063AT_AY_C5151540, JLCImport:PCF85063AT_AY_C5151540, F.Cu at (143.9, 96.6)
- added U10: ICS-43434_C5656610, JLCImport:ICS-43434_C5656610, B.Cu at (195.8, 69.4)
- added U12: 74LVC1G07SE-7, JLCImport:74LVC1G07SE-7, B.Cu at (149.4, 95.0)
- added U16: 74LVC1G07SE-7, JLCImport:74LVC1G07SE-7, B.Cu at (143.3, 96.0)
- added U21: AP64501SP-13, JLCImport:AP64501SP-13, F.Cu at (114.6, 118.3)
- added U22: AP64501SP-13, JLCImport:AP64501SP-13, F.Cu at (114.5, 106.8)
- added U23: BV1HAL45EFJ-E2, JLCImport:BV1HAL45EFJ-E2, B.Cu at (186.6, 100.1)
- added U8: BV1HAL45EFJ-E2, JLCImport:BV1HAL45EFJ-E2, B.Cu at (171.2, 100.1)
- added VL-L1: ZX-ZH1_5-7PWT, JLCImport:ZX-ZH1_5-7PWT, F.Cu at (129.6, 149.9)
- added VL-R1: ZX-ZH1_5-7PWT, JLCImport:ZX-ZH1_5-7PWT, F.Cu at (165.1, 149.9)
- added X2: ABS07-120-32_768KHZ-T, JLCImport:ABS07-120-32_768KHZ-T, F.Cu at (149.8, 98.0)
- added Y1: ASEK-32.768KHZ-LRT, ASEK-32.768KHZ-LRT:XTAL_ASEK-32.768KHZ-LRT, B.Cu at (187.1, 88.2)
- C1, C2, C3: footprint Capacitor_SMD:C_0603_1608Metric_Pad1.08x0.95mm_HandSolder -> Capacitor_SMD:C_0603_1608Metric
- C10, C11, C23, C26, C28, C29, C34, C35, C37, C47, C58, C59, C61, C64, C65, C66, C67, C68, C69, C70, C71, C72, C73, C74, C76, C77, C84, C88, C92, D10, D30, D34, D5, D6, Q1, Q20, Q8, R10, R100, R103, R104, R105, R106, R107, R115, R116, R12, R120, R127, R128, R13, R130, R131, R133, R136, R137, R138, R139, R14, R140, R15, R19, R21, R22, R24, R25, R26, R27, R60, R89, R9, R90, R91, R97, R98, U11, U13, U9, X1: moved to B.Cu
- C19: value 22uF/10V -> 4.7uF/10V; moved to B.Cu
- C20: value 100nF/10V -> JBLM2101M025C058RTM_100UF_25V; footprint Capacitor_SMD:C_0603_1608Metric -> JLCImport:JBLM2101M025C058RTM_100UF_25V
- C21: value 20pF -> JBLM2101M025C058RTM_100UF_25V; footprint Capacitor_SMD:C_0603_1608Metric -> JLCImport:JBLM2101M025C058RTM_100UF_25V
- C22: value 22uF/10V -> JBLM2101M025C058RTM_100UF_25V; footprint Capacitor_SMD:C_0603_1608Metric -> JLCImport:JBLM2101M025C058RTM_100UF_25V
- C36: value 10uF/50V -> JBLM2101M025C058RTM_100UF_25V; footprint Capacitor_SMD:C_0603_1608Metric -> JLCImport:JBLM2101M025C058RTM_100UF_25V
- C38: value 100nF/50V -> GRM31CR61A107MEA8L; footprint Capacitor_SMD:C_0603_1608Metric -> JLCImport:GRM31CR61A107MEA8L
- C4: value 10uF/10V -> 100nF/10V; footprint Capacitor_SMD:C_0603_1608Metric_Pad1.08x0.95mm_HandSolder -> Capacitor_SMD:C_0603_1608Metric
- C6: value 33nF/10V -> 4.7uF/10V; moved to B.Cu
- C60: value 0.1uF/50V -> 10uF/35V
- C62, C63: value 1nF/50V -> 1uF/50V; moved to B.Cu
- C8: value 33nF/10V -> GRM31CR61A107MEA8L; footprint Capacitor_SMD:C_0603_1608Metric -> JLCImport:GRM31CR61A107MEA8L; moved to B.Cu
- C80: footprint Capacitor_SMD:C_0805_2012Metric -> Capacitor_SMD:C_0603_1608Metric
- C86: value 0.1uF -> 100nF/10V; moved to B.Cu
- C87: value 0.1uF -> 100nF/10V; footprint Capacitor_SMD:C_0603_1608Metric -> Capacitor_SMD:C_0603_1608Metric_Pad1.08x0.95mm_HandSolder; moved to B.Cu
- C9: value 10uF/10V -> 100nF/10V
- C90, C91: value 0.1uF -> 4.7uF/10V; moved to B.Cu
- CONSOLE1: value Conn_01x03_Pin -> Conn_01x05_Pin; footprint Connector_PinHeader_2.54mm:PinHeader_1x03_P2.54mm_Vertical -> Connector_PinHeader_2.54mm:PinHeader_1x05_P2.54mm_Vertical
- D2: value LED Green -> TVS2200DRVR; footprint LED_SMD:LED_0603_1608Metric -> JLCImport:TVS2200DRVR; moved to B.Cu
- D3: value SS34 -> SMAJ18A_C148219; footprint Diode_SMD:D_SMA -> JLCImport:SMAJ18A_C148219
- ED3, ED4: moved to F.Cu
- Q6, Q7, Q9: value 2N3904 -> IRLML6344TRPBF; footprint oomwoo_altium:SOT23-3D -> JLCImport:IRLML6344TRPBF; moved to B.Cu
- R101: value 4K7 -> 10
- R102, R126: value 1K -> 510k; moved to B.Cu
- R112: value 0.2R -> 0.2R/10W; footprint Resistor_SMD:R_0603_1608Metric -> Resistor_SMD:R_2512_6332Metric
- R113, R80, R95: value 1K -> 10; moved to B.Cu
- R129: footprint JLCImport:RC0402FR-0717K4L -> Resistor_SMD:R_0603_1608Metric; moved to B.Cu
- R132: value 100 -> 10k; moved to B.Cu
- R141: value 100k -> 10
- R16: footprint Resistor_SMD:R_0603_1608Metric -> Resistor_SMD:R_1206_3216Metric; moved to B.Cu
- R2: value 270 -> 47k; moved to B.Cu
- R33: value 10 -> 100kOhm
- R5: value 150 -> 2.2k; moved to B.Cu
- R6: value 270 -> 2.2k; moved to B.Cu
- R67, R71, R72: value 100R -> 10
- R68: value 100R -> 10; moved to B.Cu
- R7: value 150 -> 47k; moved to B.Cu
- R73, R74: value 10K -> 10; moved to B.Cu
- R75: value 1K -> 100
- R76: value 2K -> 100; moved to B.Cu
- R83, R84, R88: footprint Resistor_SMD:R_0603_1608Metric -> Resistor_SMD:R_2512_6332Metric
- R94: value 4K7 -> 10; moved to B.Cu
- R96: value 330R -> 10
- R99: footprint JLCImport:RC0402FR-07215KL -> Resistor_SMD:R_0603_1608Metric; moved to B.Cu
- U14, U15, U18, U20: footprint oomwoo_altium:HSOP-8_L5.0-W4.0-P1.27-LS6.2-BL-EP -> JLCImport:DRV8870DDAR; moved to B.Cu
- U19: footprint oomwoo_altium:LGA-14_L3.0-W2.5-P0.50-TL_QMI8658A -> JLCImport:ICM-42607-P
- moved D30 248.8 mm to (94.6, 126.4), turned to 90 degrees
- moved U11 247.7 mm to (108.0, 72.1)
- moved D2 244.2 mm to (95.0, 115.0), turned to 180 degrees
- moved C28 231.1 mm to (118.9, 69.3), turned to 90 degrees
- moved MIPI1 216.7 mm to (125.9, 72.3), turned to 180 degrees
- moved R2 216.5 mm to (128.1, 151.2), turned to -90 degrees
- moved CONSOLE1 214.3 mm to (125.6, 125.6)
- moved C23 209.3 mm to (140.7, 69.2), turned to 90 degrees
- moved C1 205.0 mm to (135.2, 113.2)
- moved C2 205.0 mm to (135.2, 114.9)
- moved C3 204.9 mm to (135.2, 116.5)
- moved Module1 203.8 mm to (131.0, 127.5)
- moved C4 196.0 mm to (144.2, 82.7), turned to 180 degrees
- moved MIPI0 193.2 mm to (147.7, 72.3), turned to 180 degrees
- moved CAM0 186.6 mm to (169.5, 72.4), turned to 180 degrees
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- renumbered CN2 to BUMP_CLIFF1
Connections:
- net /CM5-GPIO/I2S_DIN renamed /SPEAKER-MIC/DOUT
- net /LiDAR-M-CTRL renamed /LiDAR/LiDAR-MOTOR-CTRL
- net Net-(Module1A-GPIO11) renamed /CM5-GPIO/SPI0_SCLK
- BUMP_CLIFF1 pad 1: unconnected-(CN2-Pad1) -> /ANTI-FALL/L1-
- BUMP_CLIFF1 pad 10: unconnected-(CN2-Pad10) -> GND
- BUMP_CLIFF1 pad 11: unconnected-(CN2-Pad11) -> VCC-3V3-P
- BUMP_CLIFF1 pad 12: unconnected-(CN2-Pad12) -> VCC-3V3-P
- BUMP_CLIFF1 pad 13: unconnected-(CN2-Pad13) -> /ANTI-FALL/ANTI-FALL-LEFT-DOWN-ADC
- BUMP_CLIFF1 pad 14: unconnected-(CN2-Pad14) -> /ANTI-FALL/ANTI-FALL-RIGHT-DOWN-ADC
- BUMP_CLIFF1 pad 15: unconnected-(CN2-Pad15) -> /ANTI-FALL/LR-
- BUMP_CLIFF1 pad 16: unconnected-(CN2-Pad16) -> /ANTI-FALL/RR+
- BUMP_CLIFF1 pad 2: unconnected-(CN2-Pad2) -> /ANTI-FALL/R2+
- BUMP_CLIFF1 pad 3: unconnected-(CN2-Pad3) -> VCC-3V3-P
- BUMP_CLIFF1 pad 4: unconnected-(CN2-Pad4) -> VCC-3V3-P
- BUMP_CLIFF1 pad 5: unconnected-(CN2-Pad5) -> /ANTI-FALL/ANTI-FALL-LEFT-UP-ADC
- BUMP_CLIFF1 pad 6: unconnected-(CN2-Pad6) -> /ANTI-FALL/ANTI-FALL-RIGHT-UP-ADC
- BUMP_CLIFF1 pad 7: unconnected-(CN2-Pad7) -> GND
- BUMP_CLIFF1 pad 8: unconnected-(CN2-Pad8) -> GND
- BUMP_CLIFF1 pad 9: unconnected-(CN2-Pad9) -> GND
- C103 pad 2: BAT-VCC -> VM-VBAT
- C108 pad 2: VCC3V3_SYS -> VCC-3V3-P
- C109 pad 2: VCC3V3_SYS -> VCC-3V3-P
- C110 pad 2: VCC3V3_SYS -> VCC-3V3-P
- C19 pad 1: GND -> VCC-3V3-P
- C19 pad 2: VCC-3V3-P -> GND
- C20 pad 1: GND -> VM-VBAT
- C20 pad 2: VCC-3V3-P -> GND
- C21 pad 1: VCC-3V3-P -> VM-VBAT
- C21 pad 2: Net-(U4-FB) -> GND
- C22 pad 1: GND -> VM-VBAT
- C22 pad 2: VCC-5V-REG -> GND
- C23 pad 1: VCC3V3_SYS -> VCC-3V3-P
- C24 pad 2: VCC3V3_SYS -> VCC3V3_M2
- C25 pad 2: VCC3V3_SYS -> VCC3V3_M2
- C26 pad 1: VCC3V3_SYS -> VCC3V3_M2
- C27 pad 2: VCC-5V-REG -> BAT-VCC
- C28 pad 1: VCC3V3_SYS -> VCC-3V3-P
- C29 pad 1: VCC3V3_SYS -> VCC-3V3-P
- C36 pad 1: BAT-VCC -> VCC3V3_M2
- C38 pad 1: BAT-VCC -> VCC-3V3-P
- C5 pad 1: VCC3V3_SYS -> VCC-3V3-P
- C59 pad 2: VCC3V3_SYS -> VCC-3V3-P
- C62 pad 1: Net-(D32-K) -> VM-VBAT
- C62 pad 2: Net-(D32-A) -> GND
- C63 pad 1: Net-(D33-K) -> VM-5V
- C63 pad 2: Net-(D33-A) -> GND
- C8 pad 1: Net-(C8-Pad1) -> GND
- C8 pad 2: GND -> VM-5V
- C84 pad 2: BAT-VCC -> VM-VBAT
- C86 pad 1: Net-(C86-Pad1) -> Net-(U16-Y)
- C86 pad 2: GND -> Net-(U12-A)
- C87 pad 1: GND -> VCC-5V-REG
- C87 pad 2: Net-(C87-Pad2) -> GND
- C88 pad 2: BAT-VCC -> VM-VBAT
- C9 pad 1: Net-(C8-Pad1) -> VCC-3V3-P
- C9 pad 2: Net-(C9-Pad2) -> GND
- C90 pad 1: Net-(C90-Pad1) -> VCC-3V3-P
- C91 pad 1: GND -> VCC-3V3-P
- C91 pad 2: Net-(C91-Pad2) -> GND
- C92 pad 2: BAT-VCC -> VM-VBAT
- CAM0 pad 15: VCC3V3_SYS -> VCC-3V3-P
- CONSOLE1 pad 1: /CM5-GPIO/CONSOLE_TXD -> GND
- CONSOLE1 pad 2: /CM5-GPIO/CONSOLE_RXD -> unconnected-(CONSOLE1-Pin_2-Pad2)
- CONSOLE1 pad 3: GND -> unconnected-(CONSOLE1-Pin_3-Pad3)
- D16 pad 1: VCC3V3_SYS -> VCC3V3_M2
- D2 pad 1: Net-(D2-K) -> GND
- D2 pad 2: +3.3VP -> GND
- D3 pad 1: VCC-3V3-P -> BAT-VCC
- D3 pad 2: Net-(D3-A) -> GND
- L5 pad 2: VCC3V3_SYS -> VCC3V3_M2
- MIPI0 pad 15: VCC3V3_SYS -> VCC-3V3-P
- MIPI1 pad 15: VCC3V3_SYS -> VCC-3V3-P
- Module1 pad 102: unconnected-(Module1B-PCIe_nCLKREQ-Pad102) -> /CM5-HIGHSPEED/PCIE_CLK_nREQ
- Module1 pad 103: /BATTERY-CHARGER/D- -> Net-(Module1B-USB2_N)
- Module1 pad 104: unconnected-(Module1B-PCIE_nWAKE-Pad104) -> /CM5-HIGHSPEED/PCIE_nWAKE
- Module1 pad 105: /BATTERY-CHARGER/D+ -> Net-(Module1B-USB2_P)
- Module1 pad 109: unconnected-(Module1B-PCIe_nRST-Pad109) -> /CM5-HIGHSPEED/PCIE_nRST
- Module1 pad 110: unconnected-(Module1B-PCIe_CLK_P-Pad110) -> /CM5-HIGHSPEED/PCIE_CLK_P
- Module1 pad 112: unconnected-(Module1B-PCIe_CLK_N-Pad112) -> /CM5-HIGHSPEED/PCIE_CLK_N
- Module1 pad 116: unconnected-(Module1B-PCIe_RX_P-Pad116) -> /CM5-HIGHSPEED/PCIE_RX_P
- Module1 pad 118: unconnected-(Module1B-PCIe_RX_N-Pad118) -> /CM5-HIGHSPEED/PCIE_RX_N
- Module1 pad 122: unconnected-(Module1B-PCIe_TX_P-Pad122) -> /CM5-HIGHSPEED/PCIE_TX_P
- Module1 pad 124: unconnected-(Module1B-PCIe_TX_N-Pad124) -> /CM5-HIGHSPEED/PCIE_TX_N
- Module1 pad 21: Net-(Module1A-LED_nACT) -> unconnected-(Module1A-LED_nACT-Pad21)
- Module1 pad 28: /CM5-GPIO/AUDIO_OUT_R -> /CM5-GPIO/UART4_RX
- Module1 pad 31: /CM5-GPIO/AUDIO_OUT_L -> /CM5-GPIO/UART4_TX
- Module1 pad 34: /MCU-STM32/STM32-TX -> /CM5-GPIO/UART2_RX
- Module1 pad 37: /MCU-STM32/STM32-RST -> /CM5-GPIO/GPIO07
- Module1 pad 39: /IMU-CS -> /CM5-GPIO/SPI0_CS0
- Module1 pad 40: /IMU-MISO -> /CM5-GPIO/SPI0_MISO
- Module1 pad 44: /IMU-MOSI -> /CM5-GPIO/SPI0_MOSI
- Module1 pad 45: /IMU-INT2 -> /CM5-GPIO/GPIO24
- Module1 pad 46: /IMU-FSYNC -> /CM5-GPIO/GPIO22
- Module1 pad 47: /IMU-INT1 -> /CM5-GPIO/GPIO23
- Module1 pad 54: /MCU-STM32/STM32-RX -> /CM5-GPIO/UART2_TX
- Module1 pad 56: /LiDAR-TXD -> /CM5-GPIO/SCL1
- Module1 pad 58: /CM5-GPIO/UART0_RX -> /CM5-GPIO/SDA1
- Module1 pad 95: Net-(Module1A-LED_nPWR) -> unconnected-(Module1A-LED_nPWR-Pad95)
- Q1 pad 1: BAT-VCC -> VM-VBAT
- Q1 pad 2: BAT-VCC -> VM-VBAT
- Q1 pad 3: BAT-VCC -> VM-VBAT
- Q6 pad 2: Net-(Q6-E) -> GND
- Q6 pad 3: Net-(Q6-C) -> /ANTI-FALL/LR-
- Q7 pad 1: Net-(Q7-B) -> Net-(Q7-G)
- Q7 pad 2: Net-(Q7-E) -> GND
- Q7 pad 3: Net-(Q7-C) -> Net-(Q7-D)
- Q8 pad 1: Net-(Q8-G) -> Net-(Q7-D)
- Q8 pad 2: VCC-5V-REG -> VM-5V
- Q9 pad 1: Net-(Q9-B) -> Net-(Q9-G)
- Q9 pad 3: Net-(Q8-G) -> Net-(Q1-G)
- R101 pad 1: VCC-3V3-P -> Net-(Module1B-USB2_P)
- R101 pad 2: Net-(C91-Pad2) -> /BATTERY-CHARGER/D+
- R102 pad 1: /MCU-STM32/WHEEL-M-LEFT-ENCODE-A -> VCC-5V-REG
- R102 pad 2: Net-(C91-Pad2) -> Net-(U16-Y)
- R103 pad 1: BAT-VCC -> VM-VBAT
- R104 pad 2: Net-(Q15-B) -> Net-(Q9-G)
- R113 pad 1: /CM5-GPIO/UART0_RX -> Net-(U13A-PD2)
- R113 pad 2: Net-(J17-Pad3) -> /LiDAR/LiDAR-RXD
- R126 pad 1: Net-(Q23-B) -> VCC-5V-REG
- R126 pad 2: /BUTTON-LED/LED-PWR -> Net-(U12-A)
- R13 pad 1: VCC3V3_SYS -> +3.3VP
- R141 pad 1: /CM5-GPIO/PMIC_EN -> Net-(C111-Pad1)
- R141 pad 2: GND -> Net-(U21-SW)
- R15 pad 2: VCC3V3_SYS -> VCC-3V3-P
- R18 pad 1: VCC3V3_SYS -> VCC-3V3-P
- R2 pad 1: /CM5-GPIO/AUDIO_OUT_R -> /CM5-GPIO/GPIO17
- R2 pad 2: Net-(C6-Pad1) -> GND
- R23 pad 1: VCC-5V-REG -> BAT-VCC
- R24 pad 1: VCC3V3_SYS -> VCC3V3_M2
- R25 pad 1: Net-(Q8-G) -> Net-(Q7-D)
- R25 pad 2: VCC-5V-REG -> VM-5V
- R27 pad 1: Net-(Q9-B) -> Net-(Q7-G)
- R33 pad 1: Net-(U13A-PB3) -> /CM5-GPIO/PMIC_EN2
- R33 pad 2: /IMU-SCLK -> GND
- R5 pad 1: GND -> VCC-3V3-P
- R5 pad 2: Net-(C6-Pad1) -> /CM5-GPIO/SDA1
- R6 pad 1: /CM5-GPIO/AUDIO_OUT_L -> VCC-3V3-P
- R6 pad 2: Net-(C8-Pad1) -> /CM5-GPIO/SCL1
- R67 pad 1: GND -> /CM5-GPIO/UART4_TX
- R67 pad 2: Net-(J4-Pad2) -> /LiDAR/LiDAR-RXD
- R68 pad 1: GND -> /ANTI-FALL/BUMPER_LED_EN
- R7 pad 1: GND -> VCC-3V3-P
- R7 pad 2: Net-(C8-Pad1) -> /CM5-GPIO/GPIO27
- R71 pad 1: GND -> Net-(Q10-G)
- R71 pad 2: Net-(J4-Pad6) -> /BUTTON-LED/LED-HOME
- R72 pad 1: GND -> Net-(Q12-G)
- R72 pad 2: Net-(J5-Pad6) -> /BUTTON-LED/LED-PWR
- R73 pad 1: GND -> /IMU-MISO
- R73 pad 2: /ANTI-FALL/ANTI-FALL-LEFT-DOWN-ADC -> Net-(U13A-PB4)
- R74 pad 1: GND -> /IMU-MOSI
- R74 pad 2: /ANTI-FALL/ANTI-FALL-RIGHT-DOWN-ADC -> Net-(U13A-PB5)
- R75 pad 1: /MCU-STM32/SIDE-PROXI-LEFT -> Net-(D39-K)
- R75 pad 2: VCC-3V3-P -> Net-(U7-ACDRV2)
- R76 pad 1: VCC-5V-REG -> Net-(D40-K)
- R76 pad 2: Net-(Q6-C) -> Net-(U7-ACDRV1)
- R80 pad 1: /MCU-STM32/TOUCHR -> /FRONT SENSORS/IR-F-RX2
- R80 pad 2: Net-(Q7-B) -> Net-(U13A-PB11)
- R92 pad 1: VCC3V3_SYS -> VCC-3V3-P
- R93 pad 1: VCC3V3_SYS -> VCC-3V3-P
- R94 pad 1: VCC-3V3-P -> /MCU-STM32/STM32-TX
- R94 pad 2: Net-(C87-Pad2) -> /CM5-GPIO/UART2_RX
- R95 pad 1: /MCU-STM32/WHEEL-M-RIGHT-ENCODE-A -> /MCU-STM32/STM32-RX
- R95 pad 2: Net-(C87-Pad2) -> /CM5-GPIO/UART2_TX
- R96 pad 1: Net-(C90-Pad1) -> Net-(Module1B-USB2_N)
- R96 pad 2: VCC-5V-REG -> /BATTERY-CHARGER/D-
- U11 pad 7: unconnected-(U11-VDD-Pad7) -> VCC-5V-REG
- U13 pad 1: unconnected-(U13B-PE2-Pad1) -> /MCU-STM32/SIDE-PROXI-GPIO-R
- U13 pad 10: unconnected-(U13B-PF9-Pad10) -> /MCU-STM32/SIDE-BRUSH-IN1
- U13 pad 11: unconnected-(U13B-PF10-Pad11) -> /MCU-STM32/SIDE-BRUSH-IN2
- U13 pad 16: unconnected-(U13A-PC1-Pad16) -> /ANTI-FALL/CLIFF_LED_EN
- U13 pad 18: unconnected-(U13A-PC3-Pad18) -> /ANTI-FALL/BUMPER_LED_EN
- U13 pad 19: unconnected-(U13B-PF2-Pad19) -> /MCU-STM32/PF2
- U13 pad 2: unconnected-(U13B-PE3-Pad2) -> /MCU-STM32/SIDE-PROXI-CE-R
- U13 pad 3: unconnected-(U13B-PE4-Pad3) -> /MCU-STM32/SIDE-PROXI-GPIO-L
- U13 pad 32: unconnected-(U13A-PB0-Pad32) -> /MCU-STM32/WHEEL-M-RIGHT-DROP
- U13 pad 33: unconnected-(U13A-PB1-Pad33) -> /MCU-STM32/WHEEL-M-LEFT-DROP
- U13 pad 34: unconnected-(U13A-PB2-Pad34) -> /BUTTON-LED/HOME-BTN
- U13 pad 38: unconnected-(U13B-PE7-Pad38) -> /MCU-STM32/PE7
- U13 pad 39: unconnected-(U13B-PE8-Pad39) -> /MCU-STM32/PE8
- U13 pad 4: unconnected-(U13B-PE5-Pad4) -> /MCU-STM32/SIDE-PROXI-CE-L
- U13 pad 40: unconnected-(U13B-PE9-Pad40) -> /MAIN-FAN/MAIN-FAN-S-SENSE
- U13 pad 41: unconnected-(U13B-PE10-Pad41) -> /MCU-STM32/PE10
- U13 pad 42: unconnected-(U13B-PE11-Pad42) -> /MCU-STM32/PE11
- U13 pad 43: unconnected-(U13B-PE12-Pad43) -> /MCU-STM32/PE12
- U13 pad 44: unconnected-(U13B-PE13-Pad44) -> /MCU-STM32/PE13
- U13 pad 45: unconnected-(U13B-PE14-Pad45) -> /MCU-STM32/PE14
- U13 pad 46: unconnected-(U13B-PE15-Pad46) -> /FRONT SENSORS/IR-F-RX1
- U13 pad 47: unconnected-(U13A-PB10-Pad47) -> /MCU-STM32/PB10
- U13 pad 5: unconnected-(U13B-PE6-Pad5) -> /MCU-STM32/PE6
- U13 pad 50: unconnected-(U13A-PB11-Pad50) -> Net-(U13A-PB11)
- U13 pad 51: unconnected-(U13A-PB12-Pad51) -> /BUTTON-LED/LED-HOME
- U13 pad 52: /CM5-GPIO/RUN_PG -> /CM5-GPIO/PMIC_EN
- U13 pad 55: /MCU-STM32/SIDE-PROXI-RIGHT -> /MCU-STM32/PD8
- U13 pad 56: /MCU-STM32/TOUCHR -> /MCU-STM32/PD9
- U13 pad 59: unconnected-(U13A-PD12-Pad59) -> /FRONT SENSORS/LIGHT-ON
- U13 pad 65: /MCU-STM32/SIDE-BRUSH-IN1 -> /MCU-STM32/I2C4_SCL
- U13 pad 66: /MCU-STM32/SIDE-BRUSH-IN2 -> /MCU-STM32/I2C4_SDA
- U13 pad 7: unconnected-(U13A-PC13-Pad7) -> /MCU-STM32/PC13
- U13 pad 73: /CM5-GPIO/PMIC_EN -> /CM5-GPIO/RUN_PG
- U13 pad 79: /BUTTON-LED/HOME-BTN -> /MCU-STM32/PC10
- U13 pad 80: /BUTTON-LED/LED-HOME -> /MCU-STM32/USART4-IR-R-RX
- U13 pad 81: /MAIN-FAN/MAIN-FAN-S-SENSE -> Net-(U13A-PC12)
- U13 pad 84: /IMU-INT2 -> Net-(U13A-PD2)
- U13 pad 87: /MCU-STM32/SIDE-PROXI-LEFT -> /MCU-STM32/PD5
- U13 pad 88: /MCU-STM32/TOUCHL -> /MCU-STM32/USART2-IR-L-RX
- U13 pad 89: unconnected-(U13A-PD7-Pad89) -> /IMU-INT2
- U13 pad 91: /IMU-MISO -> Net-(U13A-PB4)
- U13 pad 92: /IMU-MOSI -> Net-(U13A-PB5)
- U13 pad 97: unconnected-(U13B-PE0-Pad97) -> /MCU-STM32/PE0
- U13 pad 98: unconnected-(U13B-PE1-Pad98) -> /MCU-STM32/PE1
- U14 pad 5: BAT-VCC -> VM-VBAT
- U15 pad 5: BAT-VCC -> VM-VBAT
- U18 pad 5: BAT-VCC -> VM-VBAT
- U19 pad 5: VCC3V3_SYS -> VCC-3V3-P
- U19 pad 8: VCC3V3_SYS -> VCC-3V3-P
- U20 pad 5: BAT-VCC -> VM-VBAT
- U5 pad 4: VCC-5V-REG -> BAT-VCC
- U9 pad 5: VCC3V3_SYS -> VCC-3V3-P
Routing:
- net (no net): track 8387.5 -> 0.00 mm, vias 518 -> 0
- net GND: track 944.1 -> 0.00 mm, vias 816 -> 0
- net VCC-5V-REG: track 513.9 -> 0.00 mm, vias 48 -> 0
- net VCC-3V3-P: track 498.3 -> 0.00 mm, vias 23 -> 0
- net VCC3V3_SYS: track 354.1 -> 0.00 mm, vias 32 -> 0
- net BAT-VCC: track 326.4 -> 0.00 mm, vias 35 -> 0
- net /CM5-GPIO/RUN_PG: track 177.0 -> 0.00 mm, vias 7 -> 0
- net /MCU-STM32/WHEEL-M-LEFT-IN2: track 145.3 -> 0.00 mm, vias 2 -> 0
- net /MCU-STM32/TOUCHL: track 142.2 -> 0.00 mm, vias 4 -> 0
- net /MCU-STM32/WHEEL-M-LEFT-ENCODE-A: track 141.6 -> 0.00 mm, vias 2 -> 0
- net /MCU-STM32/WHEEL-M-L-F-ADC: track 137.9 -> 0.00 mm, vias 2 -> 0
- net /MCU-STM32/WHEEL-M-LEFT-IN1: track 137.4 -> 0.00 mm, vias 2 -> 0
- net /MCU-STM32/SIDE-PROXI-LEFT: track 136.2 -> 0.00 mm, vias 4 -> 0
- net /LiDAR/LiDAR-MOTOR-CTRL: track 133.0 -> 0.00 mm, vias 2 -> 0
- net /IMU-CS: track 130.1 -> 0.00 mm, vias 3 -> 0
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- removed copper zone on In2.Cu, net (none)
- removed copper zone on In2.Cu, net /BATTERY-CHARGER/SDA
- removed copper zone on In2.Cu, net BAT-VCC
- removed copper zone on B.Cu, net GND
- removed copper zone on F.Cu, net GND
- removed copper zone on In1.Cu, net GND
- removed copper zone on In2.Cu, net GND
- removed copper zone on In2.Cu, net VCC-5V-REG
- removed copper zone on In2.Cu, net VCC-CHARG
Other:
- board size 116 x 98.7 mm -> 115.7 x 88.3 mm
