File: kicad/main/Main.kicad_pcb (KiCad board)
At the start: 4 copper layers, 115.7 x 88.3 mm, 356 parts, among them CN2 EV2400, IC5 TPS25730DREFR, J2 1-2199119-5, K2 kEY-4, K3 kEY-4, Q1 AO4407A, Q10 IRLML6344TRPBF, Q11 2N3904, Q12 IRLML6344TRPBF, Q13 IRLML6344TRPBF, Q14 IRLML6344TRPBF, Q18 IRLML6344TRPBF, Q19 IRLML6344TRPBF, Q20 AO3400, Q21 SQJ844AEP-T1_GE3, Q3 PNP-SOT23, Q4 SQJ844AEP-T1_GE3, Q5 IRLML6344TRPBF, Q6 IRLML6344TRPBF, Q7 IRLML6344TRPBF, Q8 AO3401, Q9 IRLML6344TRPBF, U1 PCF85063AT_AY_C5151540, U10 ICS-43434_C5656610, U11 MAX98357AETE_T, U12 74LVC1G07SE-7, U13 STM32G473VCT6, U14 DRV8870DDAR, U15 DRV8870DDAR, U16 74LVC1G07SE-7, U18 DRV8870DDAR, U19 ICM-42607-P, U20 DRV8870DDAR, U21 AP64501SP-13, U22 AP64501SP-13, U23 BV1HAL45EFJ-E2, U5 SY8089A, U6 RT9742GGJ5, U7 BQ25792RQMR, U8 BV1HAL45EFJ-E2, U9 ICS-43434_C5656610, X1 ABM3-8_000MHZ-D2Y-T, X2 ABS07-120-32_768KHZ-T, Y1 ASEK-32.768KHZ-LRT

Commit message: Schematic fixes, 1st round of review
Parts:
- removed C18, C38, C8: GRM31CR61A107MEA8L, JLCImport:GRM31CR61A107MEA8L
- removed C20, C21, C22, C36: JBLM2101M025C058RTM_100UF_25V, JLCImport:JBLM2101M025C058RTM_100UF_25V
- removed C24, C27: 22uF/10V, Capacitor_SMD:C_0603_1608Metric
- removed C25, C57, C86: 100nF/10V, Capacitor_SMD:C_0603_1608Metric
- removed C26: 20pF/10V, Capacitor_SMD:C_0603_1608Metric
- removed C41, C43, C48, C49: 100nF/50V, Capacitor_SMD:C_0603_1608Metric
- removed C52, C53: 18pF/10V, Capacitor_SMD:C_0603_1608Metric
- removed C87: 100nF/10V, Capacitor_SMD:C_0603_1608Metric_Pad1.08x0.95mm_HandSolder
- removed D11, D12: LED-HOME, oomwoo_altium:LED0603-B
- removed D13, D14: LED-PWR, oomwoo_altium:LED0603-B
- removed D16: 3V3-RK, oomwoo_altium:LED0603-B
- removed D17, D19, D20, D31: 1N4007, oomwoo_altium:SOD123
- removed D30: SS34, oomwoo_altium:SMA
- removed K2, K3: kEY-4, oomwoo_altium:KEY-SMD_4P-L6.0-W6.0-P4.50-LS9.0
- removed L5: 2.2uH, oomwoo_altium:IND-SMD_L4.4-W4.2
- removed LIDAR1: WAFER-GH1_25-6PWB, JLCImport:WAFER-GH1_25-6PWB
- removed Q13, Q14, Q18, Q19: IRLML6344TRPBF, JLCImport:IRLML6344TRPBF
- removed Q3: PNP-SOT23, oomwoo_altium:SOT23-3D
- removed R102, R126: 510k, Resistor_SMD:R_0603_1608Metric
- removed R103: 22K, Resistor_SMD:R_0603_1608Metric
- removed R104, R122, R124, R125: 1K, Resistor_SMD:R_0603_1608Metric
- removed R105, R106, R107, R108, R109, R111, R119, R89, R90, R91, R97, R98: 10K, Resistor_SMD:R_0603_1608Metric
- removed R134, R63, R66, R67, R68, R71, R72: 10, Resistor_SMD:R_0603_1608Metric
- removed R24: 450K, Resistor_SMD:R_0603_1608Metric
- removed R26: 100K, Resistor_SMD:R_0603_1608Metric
- removed R33, R46: 100kOhm, Resistor_SMD:R_0603_1608Metric
- removed R56: 10k, Resistor_SMD:R_0603_1608Metric
- removed U12, U16: 74LVC1G07SE-7, JLCImport:74LVC1G07SE-7
- removed U5: SY8089A, oomwoo_altium:SOT5P95B160_300H130
- removed X2: ABS07-120-32_768KHZ-T, JLCImport:ABS07-120-32_768KHZ-T
- added C104: 10uF/25V, Capacitor_SMD:C_0603_1608Metric, B.Cu at (188.4, 76.4)
- added C124: 10uF/25V, Capacitor_SMD:C_0603_1608Metric, B.Cu at (186.8, 76.4)
- added C127: 100nF/50V, Capacitor_SMD:C_0603_1608Metric, F.Cu at (187.4, 76.7)
- added C128: 100nF/50V, Capacitor_SMD:C_0603_1608Metric, B.Cu at (191.0, 79.9)
- added C129: 100nF/50V, Capacitor_SMD:C_0603_1608Metric, F.Cu at (191.4, 73.7)
- added C130: 1.2nF/50V, Capacitor_SMD:C_0603_1608Metric, B.Cu at (195.4, 80.4)
- added C131: 10uF/25V, Capacitor_SMD:C_0603_1608Metric, F.Cu at (197.5, 83.9)
- added C132: 10uF/25V, Capacitor_SMD:C_0603_1608Metric, F.Cu at (195.9, 83.9)
- added C133: 10uF/25V, Capacitor_SMD:C_0603_1608Metric, B.Cu at (195.3, 115.2)
- added C134: 10uF/25V, Capacitor_SMD:C_0603_1608Metric, B.Cu at (203.1, 80.2)
- added C135: 10uF/25V, Capacitor_SMD:C_0603_1608Metric, B.Cu at (203.4, 138.6)
- added C136: 10uF/25V, Capacitor_SMD:C_0603_1608Metric, F.Cu at (103.0, 130.7)
- added C137: 10uF/25V, Capacitor_SMD:C_0603_1608Metric, B.Cu at (111.6, 149.0)
- added C138: 10uF/25V, Capacitor_SMD:C_0603_1608Metric, B.Cu at (195.6, 147.1)
- added C139: 10uF/25V, Capacitor_SMD:C_0603_1608Metric, B.Cu at (153.9, 144.5)
- added C140: 10uF/25V, Capacitor_SMD:C_0603_1608Metric, B.Cu at (153.5, 110.5)
- added C141: 10uF/25V, Capacitor_SMD:C_0603_1608Metric, B.Cu at (153.5, 108.9)
- added C142: 100nF/50V, Capacitor_SMD:C_0603_1608Metric, B.Cu at (203.5, 135.9)
- added C143: 100nF/50V, Capacitor_SMD:C_0603_1608Metric, F.Cu at (101.3, 140.6)
- added C144: 10uF/25V, Capacitor_SMD:C_0603_1608Metric, F.Cu at (194.3, 83.9)
- added C145: 10uF/25V, Capacitor_SMD:C_0603_1608Metric, F.Cu at (192.8, 83.9)
- added C146: 10uF/25V, Capacitor_SMD:C_0603_1608Metric, F.Cu at (115.3, 125.3)
- added C147: 10uF/25V, Capacitor_SMD:C_0603_1608Metric, F.Cu at (112.6, 111.5)
- added C42: 18pF/10V, Capacitor_SMD:C_0603_1608Metric, F.Cu at (148.5, 127.5)
- added C7: 150pF/50V, Capacitor_SMD:C_0603_1608Metric, B.Cu at (105.4, 150.7)
- added CM_ACT1: YLED0603B, JLCImport:YLED0603B, F.Cu at (127.4, 103.3)
- added CM_PWR1: YLED0603B, JLCImport:YLED0603B, F.Cu at (127.4, 116.6)
- added H1: PM254-2-06-S-8_5, JLCImport:PM254-2-06-S-8_5, F.Cu at (137.7, 141.7)
- added HOME1: YLED0603B, JLCImport:YLED0603B, F.Cu at (180.9, 76.0)
- added JP1: ~, Jumper:SolderJumper-2_P1.3mm_Open_RoundedPad1.0x1.5mm, B.Cu at (163.9, 98.0)
- added JP2: ~, Jumper:SolderJumper-2_P1.3mm_Open_RoundedPad1.0x1.5mm, B.Cu at (166.7, 98.2)
- added JP3: ~, Jumper:SolderJumper-2_P1.3mm_Open_RoundedPad1.0x1.5mm, B.Cu at (132.3, 121.2)
- added L4: CYA0630-3_3UH, JLCImport:CYA0630-3_3UH, F.Cu at (201.6, 77.2)
- added M2_ACT1: YLED0603B, JLCImport:YLED0603B, F.Cu at (172.3, 77.9)
- added PWR1: YLED0603B, JLCImport:YLED0603B, F.Cu at (180.9, 78.7)
- added Q2: 2302V, JLCImport:2302V, B.Cu at (188.8, 70.0)
- added R11: 100k, Resistor_SMD:R_0603_1608Metric, B.Cu at (198.0, 142.5)
- added R154: 10, Resistor_SMD:R_0603_1608Metric, F.Cu at (194.5, 73.7)
- added R155: 12k, Resistor_SMD:R_0603_1608Metric, B.Cu at (197.9, 79.6)
- added R156: 69.8k, Resistor_SMD:R_0603_1608Metric, B.Cu at (200.3, 76.9)
- added R157: 22.1k, Resistor_SMD:R_0603_1608Metric, B.Cu at (200.3, 74.4)
- added R158: 100, Resistor_SMD:R_0805_2012Metric, B.Cu at (153.7, 112.3)
- added R17: 100k, Resistor_SMD:R_0603_1608Metric, B.Cu at (198.0, 145.0)
- added R20: 100k, Resistor_SMD:R_0603_1608Metric, B.Cu at (102.7, 145.0)
- added R3: 100k, Resistor_SMD:R_0603_1608Metric, B.Cu at (200.9, 89.9)
- added R36: 10k, Resistor_SMD:R_0603_1608Metric, B.Cu at (107.1, 150.7)
- added R4: 100k, Resistor_SMD:R_0603_1608Metric, B.Cu at (204.3, 89.9)
- added R42: 10k, Resistor_SMD:R_0603_1608Metric, B.Cu at (105.7, 144.7)
- added R43: 100k, Resistor_SMD:R_0603_1608Metric, B.Cu at (202.8, 109.6)
- added R57: 100k, Resistor_SMD:R_0603_1608Metric, F.Cu at (191.6, 144.6)
- added R58: 100k, Resistor_SMD:R_0603_1608Metric, B.Cu at (168.8, 103.9)
- added R59: 100k, Resistor_SMD:R_0603_1608Metric, B.Cu at (184.7, 94.7)
- added R77: 1k, Resistor_SMD:R_0603_1608Metric, F.Cu at (177.5, 75.9)
- added R78: 1k, Resistor_SMD:R_0603_1608Metric, F.Cu at (177.5, 78.4)
- added R79: 1k, Resistor_SMD:R_0603_1608Metric, F.Cu at (172.2, 80.5)
- added R82: 1k, Resistor_SMD:R_0603_1608Metric, F.Cu at (127.2, 113.2)
- added R85: 1k, Resistor_SMD:R_0603_1608Metric, B.Cu at (130.0, 102.4)
- added SW1: TC-6601-5_0-260-8_3, JLCImport:TC-6601-5_0-260-8_3, F.Cu at (159.8, 78.0)
- added SW2: TC-6601-5_0-260-8_3, JLCImport:TC-6601-5_0-260-8_3, F.Cu at (148.9, 78.1)
- added SW3: TC-6601-5_0-260-8_3, JLCImport:TC-6601-5_0-260-8_3, F.Cu at (137.8, 78.2)
- added TP1: TestPoint, TestPoint:TestPoint_Pad_D2.0mm, F.Cu at (124.8, 75.2)
- added TP2: TestPoint, TestPoint:TestPoint_Pad_D2.0mm, F.Cu at (115.0, 73.8)
- added TP3: TestPoint, TestPoint:TestPoint_Pad_D2.0mm, F.Cu at (167.2, 75.7)
- added U2: TPS3828-33DBVR, JLCImport:TPS3828-33DBVR, F.Cu at (138.1, 113.7)
- added U24: AP64501SP-13, JLCImport:AP64501SP-13, F.Cu at (193.3, 78.0)
- added U3: HC-PM254-5_0H-2X4PS-02A, JLCImport:HC-PM254-5_0H-2X4PS-02A, F.Cu at (151.9, 141.6)
- added X3: XKXEL89CII-SUAYLC-32_768K, JLCImport:XKXEL89CII-SUAYLC-32_768K, F.Cu at (149.7, 130.5)
- C1, C10, C12, C13, C14, C15, C16, C2, C30, C32, C37, C4, C5, C56, C9: value 100nF/10V -> 100nF/50V
- C100, C60, C66, C67, C68, C71, C72, C74, C76, C80, C81, C82, C94, C96, C97, C98, C99: value 10uF/35V -> 10uF/25V
- C101: value 0.1uF -> 150pF/50V; moved to B.Cu
- C103: value 0.22uF -> 100nF/50V; moved to B.Cu
- C105: value 100nF -> 150pF/50V; moved to B.Cu
- C106, C113, C114, C115, C116, C121, C122, C123, C95: value 10uF/50V -> 10uF/25V
- C108: value 2.2uF -> 10uF/25V; moved to B.Cu
- C109: value 100nF -> 100nF/50V; moved to B.Cu
- C11, C45: value 10uF/10V -> 10uF/25V
- C110: value 10nF -> 47nF/50V; moved to B.Cu
- C17, C19, C31, C33, C6, C70, C90, C91: value 4.7uF/10V -> 10uF/25V
- C3: value 10uf/10V -> 10uF/25V
- C34, C35: value 22pF/10V -> 22pF/50V
- C39: value JBLM2101M025C058RTM_100UF_25V -> 18pF/10V; footprint JLCImport:JBLM2101M025C058RTM_100UF_25V -> Capacitor_SMD:C_0603_1608Metric
- C47, C58: value 330pF/35V -> 330pF/25V
- C59, C61, C64, C65, C73: value 0.1uF/35V -> 100nF/50V
- C62, C63: value 1uF/50V -> 10uF/25V
- C69, C78, C83: value 0.1uF/50V -> 10uF/25V
- C84: value 0.22uF/25V -> 100nF/50V
- C88: value 0.22uF -> 100nF/50V; moved to F.Cu
- C92: value 0.22uF -> 100nF/50V
- D10, D37, D38, D6: footprint oomwoo_altium:SMA -> Diode_SMD:D_SMA
- D22, R112: moved to B.Cu
- Q1: value AO4407A -> 2302V; footprint JLCImport:AO4407A -> JLCImport:2302V
- Q10: value IRLML6344TRPBF -> 2302V; footprint JLCImport:IRLML6344TRPBF -> JLCImport:2302V; moved to B.Cu
- Q12: value IRLML6344TRPBF -> 2N3906_C49023424; footprint JLCImport:IRLML6344TRPBF -> JLCImport:2N3906_C49023424
- Q5, Q6, Q7, Q9: value IRLML6344TRPBF -> 2302V; footprint JLCImport:IRLML6344TRPBF -> JLCImport:2302V
- R1, R51, R52: value 10 -> 10k; moved to B.Cu
- R10, R27: value 1K -> 100k; moved to F.Cu
- R100, R75, R76: footprint Resistor_SMD:R_0603_1608Metric -> Resistor_SMD:R_0805_2012Metric
- R110, R18, R81, R92, R93: value 10K -> 10k; moved to B.Cu
- R113: value 10 -> 1k
- R116: value 10K -> 100k
- R118: value 1K -> 100k; moved to B.Cu
- R120, R121, R14, R28, R37: value 1K -> 1k
- R130: value 162k -> 100k
- R131: value 38k -> 20k
- R133: value 190k -> 100k
- R136: value 9.5k -> 5.24k
- R137: value 9.4k -> 5.24k
- R138: value 191k -> 100k
- R139: value 198.2k -> 100k
- R140: value 2.28k -> 1k
- R150, R152: value 15k -> 10k
- R151: value 50k -> 47k
- R16: value 0.01 -> 100k; footprint Resistor_SMD:R_1206_3216Metric -> Resistor_SMD:R_0603_1608Metric; moved to F.Cu
- R23: value 100K -> 10k
- R25, R32, R34, R45: value 10K -> 10k
- R29, R40: value 100K -> 100k
- R31: value 1K -> 10k
- R47: value 10kOhm -> 20k; moved to B.Cu
- R48, R55: value 10 -> 100k
- R53, R54: value 10 -> 100k; moved to B.Cu
- R65: value 10 -> 1k; moved to B.Cu
- R83, R84, R88: value 0.2R -> 0.2R/10W; moved to B.Cu
- U1: value PCF85063AT_AY_C5151540 -> NCP1117ST33T3G; footprint JLCImport:PCF85063AT_AY_C5151540 -> NCP1117ST33T3G:SOT230P700X180-4N; moved to B.Cu
- U15: moved to F.Cu
- moved R27 94.3 mm to (110.2, 135.7), turned to -90 degrees
- moved R23 91.1 mm to (187.6, 81.0), turned to 0 degrees
- moved R51 77.7 mm to (203.4, 143.7)
- moved R18 74.5 mm to (146.3, 152.9)
- moved R112 73.4 mm to (195.0, 84.9), turned to -90 degrees
- moved Q10 71.7 mm to (130.9, 117.1), turned to 0 degrees
- moved R10 71.4 mm to (187.6, 79.3)
- moved R92 69.5 mm to (146.4, 151.2)
- moved U19 68.8 mm to (148.4, 151.0), turned to 180 degrees
- moved R93 68.1 mm to (149.9, 151.3)
- moved R55 67.5 mm to (194.1, 144.6), turned to -90 degrees
- moved D10 66.7 mm to (149.2, 140.8), turned to 180 degrees
- moved Q9 66.4 mm to (112.5, 68.8), turned to -90 degrees
- moved R54 64.9 mm to (188.8, 73.4)
- moved R121 64.6 mm to (129.4, 82.9), turned to 0 degrees
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- renumbered MOT_L1 to MOT_WHEEL_L1, MOT_R1 to MOT_WHEEL_R1
Connections:
- C37 pad 1: /MCU-STM32/STM32-RST -> /MCU-STM32/~{STM32_RST}
- C39 pad 1: VM-VBAT -> GND
- C39 pad 2: GND -> Net-(U13A-PC15-OSC32_OUT)
- C67 pad 2: Net-(Q21-D2) -> VCC-CHARG
- C68 pad 2: Net-(Q21-D2) -> VCC-CHARG
- C69 pad 1: Net-(Q21-D2) -> VCC-CHARG
- C94 pad 1: VCC-CHARG -> Net-(Q4-D2)
- CAM0 pad 11: /CAMERA/CAM_IO -> /CAMERA/CAM_GPIO0
- CAM0 pad 12: unconnected-(CAM0-Pad12) -> Net-(CAM0-Pad12)
- CONTACT_CHGR1 pad 3: VCC-CHARG -> Net-(Q4-D2)
- CONTACT_CHGR1 pad 4: VCC-CHARG -> Net-(Q4-D2)
- D1 pad 4: VCC-CHARG -> Net-(Q4-D2)
- D1 pad 5: VCC-CHARG -> Net-(Q4-D2)
- D1 pad 6: VCC-CHARG -> Net-(Q4-D2)
- J2 pad 10: unconnected-(J2-P10-Pad10) -> Net-(J2-P10)
- J2 pad 41: /CM5-HIGHSPEED/PCIE_RX_N -> /CM5-HIGHSPEED/PCIE_RX_P
- J2 pad 43: /CM5-HIGHSPEED/PCIE_RX_P -> /CM5-HIGHSPEED/PCIE_RX_N
- J2 pad 47: /CM5-HIGHSPEED/PCIE_TX_N -> /CM5-HIGHSPEED/PCIE_TX_P
- J2 pad 49: /CM5-HIGHSPEED/PCIE_TX_P -> /CM5-HIGHSPEED/PCIE_TX_N
- J2 pad 69: GND -> unconnected-(J2-P69-Pad69)
- JTAG1 pad 12: /MCU-STM32/STM32-RST -> /MCU-STM32/~{JTAG_RST}
- MAIN_FAN1 pad 1: Net-(MAIN_FAN1-Pad1) -> /MAIN-FAN/MAIN-FAN-S-SENSE
- MAIN_FAN1 pad 2: Net-(D30-K) -> Net-(Q1-D)
- MAIN_FAN1 pad 4: /MAIN-FAN/MAIN-FAN-S-SENSE -> VM-VBAT
- MCU_IO1 pad 10: /MCU-STM32/PC14 -> unconnected-(MCU_IO1-Pad10)
- MCU_IO1 pad 6: /MCU-STM32/PD9 -> unconnected-(MCU_IO1-Pad6)
- MCU_IO1 pad 7: /MCU-STM32/PD8 -> unconnected-(MCU_IO1-Pad7)
- MCU_IO1 pad 9: /MCU-STM32/PC15 -> unconnected-(MCU_IO1-Pad9)
- MIPI0 pad 11: /CAMERA/CAM_IO -> /CAMERA/CAM_GPIO0
- MIPI0 pad 12: unconnected-(MIPI0-Pad12) -> Net-(JP3-A)
- MIPI1 pad 12: unconnected-(MIPI1-Pad12) -> Net-(MIPI1-Pad12)
- MOT_WHEEL_L1 pad 3: VCC-5V-REG -> GND
- MOT_WHEEL_L1 pad 4: GND -> /MCU-STM32/WHEEL-M-LEFT-ENCODE-A
- MOT_WHEEL_L1 pad 5: /MCU-STM32/WHEEL-M-LEFT-ENCODE-A -> VCC-3V3-P
- MOT_WHEEL_L1 pad 6: VCC-3V3-P -> GND
- MOT_WHEEL_R1 pad 3: VCC-5V-REG -> GND
- MOT_WHEEL_R1 pad 4: GND -> /MCU-STM32/WHEEL-M-RIGHT-ENCODE-A
- MOT_WHEEL_R1 pad 5: /MCU-STM32/WHEEL-M-RIGHT-ENCODE-A -> VCC-3V3-P
- MOT_WHEEL_R1 pad 6: VCC-3V3-P -> GND
- Module1 pad 100: unconnected-(Module1A-CAM_GPIO1-Pad100) -> /CAMERA/CAM_GPIO0
- Module1 pad 104: /CM5-HIGHSPEED/PCIE_nWAKE -> Net-(JP1-B)
- Module1 pad 106: unconnected-(Module1B-PCIE_PWR_EN-Pad106) -> Net-(JP2-B)
- Module1 pad 21: unconnected-(Module1A-LED_nACT-Pad21) -> Net-(CM_ACT1-K)
- Module1 pad 28: /CM5-GPIO/UART4_RX -> /CM5-GPIO/GPIO13
- Module1 pad 31: /CM5-GPIO/UART4_TX -> /CM5-GPIO/GPIO12
- Module1 pad 37: /CM5-GPIO/GPIO07 -> /CM5-GPIO/GPIO7
- Module1 pad 38: /CM5-GPIO/SPI0_SCLK -> /CM5-GPIO/GPIO11
- Module1 pad 39: /CM5-GPIO/SPI0_CS0 -> /CM5-GPIO/GPIO8
- Module1 pad 40: /CM5-GPIO/SPI0_MISO -> /CM5-GPIO/GPIO9
- Module1 pad 44: /CM5-GPIO/SPI0_MOSI -> /CM5-GPIO/GPIO10
- Module1 pad 95: unconnected-(Module1A-LED_nPWR-Pad95) -> Net-(Module1A-LED_nPWR)
- Module1 pad 97: /CAMERA/CAM_IO -> /CAMERA/CAM_GPIO1
- Module1 pad 99: Net-(Module1A-PMIC_ENABLE) -> /CM5-GPIO/PMIC_EN
- Q1 pad 1: VM-VBAT -> VCC-3V3-P
- Q1 pad 2: VM-VBAT -> /MAIN-FAN/MAIN-FAN-S-CTRL
- Q1 pad 3: VM-VBAT -> Net-(Q1-D)
- Q10 pad 1: Net-(Q10-G) -> Net-(Module1A-LED_nPWR)
- Q10 pad 3: Net-(Q10-D) -> Net-(CM_PWR1-K)
- Q12 pad 1: Net-(Q12-G) -> Net-(Q12-B)
- Q12 pad 2: GND -> Net-(D26-K)
- Q12 pad 3: Net-(Q12-D) -> Net-(D28-A)
- Q21 pad 5: Net-(Q21-D2) -> VCC-CHARG
- Q4 pad 5: VCC-CHARG -> Net-(Q4-D2)
- Q4 pad 6: Net-(Q21-D2) -> VCC-CHARG
- Q5 pad 1: Net-(Q5-G) -> /ANTI-FALL/BUMPER_LED_EN
- Q6 pad 1: Net-(Q6-G) -> /ANTI-FALL/CLIFF_LED_EN
- Q7 pad 1: Net-(Q7-G) -> /MCU-STM32/WATER-PUMPU-CTRL
- Q9 pad 1: Net-(Q9-G) -> /CM5-GPIO/GPIO06
- Q9 pad 3: Net-(Q1-G) -> Net-(Q9-D)
- R1 pad 1: /IMU-SCLK -> VCC-3V3-P
- R1 pad 2: /CM5-GPIO/SPI0_SCLK -> /MAIN-FAN/MAIN-FAN-S-SENSE
- R10 pad 1: GND -> /CM5-HIGHSPEED/PCIE_PWR_EN
- R10 pad 2: Net-(D16-Pad2) -> GND
- R112 pad 2: Net-(U20-ISEN) -> /MAIN-BRUSH MOTOR/MAIN-BRUSH-CURRENT-ADC
- R118 pad 1: Net-(MAIN_FAN1-Pad1) -> GND
- R118 pad 2: /MAIN-FAN/MAIN-FAN-S-CTRL -> /LiDAR/LIDAR_EN
- R121 pad 1: Net-(Q10-D) -> /BUTTON-LED/CLEAN-BTN
- R121 pad 2: Net-(D11-Pad2) -> VCC-3V3-P
- R135 pad 2: /POWER/V-MOTORS-EN -> /MCU-STM32/~{JTAG_RST}
- R16 pad 1: VCC-3V3-P -> +3.3VP
- R16 pad 2: Net-(U13C-VBAT) -> GND
- R21 pad 1: /MCU-STM32/STM32-RST -> /MCU-STM32/~{STM32_RST}
- R23 pad 1: BAT-VCC -> +3.3VP
- R23 pad 2: Net-(U5-EN) -> /CM5-HIGHSPEED/PCIE_PWR_EN
- R27 pad 1: Net-(Q7-G) -> /MCU-STM32/WHEEL-M-LEFT-IN2
- R27 pad 2: /MCU-STM32/WATER-PUMPU-CTRL -> GND
- R32 pad 1: Net-(Q3-B) -> Net-(Q12-B)
- R45 pad 2: Net-(Q3-B) -> Net-(Q12-B)
- R47 pad 1: /LiDAR/LiDAR-RXD -> /MCU-STM32/WATER-PUMP-SENSE-ADC
- R47 pad 2: Net-(LIDAR1-Pad3) -> GND
- R48 pad 2: Net-(Q6-G) -> GND
- R49 pad 1: /MCU-STM32/WHEEL-M-RIGHT-DROP -> VCC-3V3-P
- R49 pad 2: GND -> /MCU-STM32/WHEEL-M-RIGHT-DROP
- R50 pad 1: /MCU-STM32/WHEEL-M-LEFT-DROP -> VCC-3V3-P
- R50 pad 2: GND -> /MCU-STM32/WHEEL-M-LEFT-DROP
- R51 pad 1: /IMU-MOSI -> VCC-3V3-P
- R51 pad 2: /CM5-GPIO/SPI0_MOSI -> /MCU-STM32/WHEEL-M-RIGHT-ENCODE-A
- R52 pad 1: /IMU-MISO -> VCC-3V3-P
- R52 pad 2: /CM5-GPIO/SPI0_MISO -> /MCU-STM32/WHEEL-M-LEFT-ENCODE-A
- R53 pad 1: /IMU-CS -> /ANTI-FALL/BUMPER_LED_EN
- R53 pad 2: /CM5-GPIO/SPI0_CS0 -> GND
- R54 pad 1: /IMU-INT2 -> /FRONT SENSORS/LIGHT-ON
- R54 pad 2: /CM5-GPIO/GPIO24 -> GND
- R55 pad 1: /IMU-INT1 -> /MCU-STM32/SIDE-BRUSH-IN1
- R55 pad 2: /CM5-GPIO/GPIO23 -> GND
- R65 pad 1: /CM5-GPIO/GPIO07 -> /LiDAR/LiDAR-RXD
- R65 pad 2: /LiDAR/LiDAR-MOTOR-CTRL -> Net-(R65-Pad2)
- R83 pad 2: Net-(U14-ISEN) -> /MCU-STM32/WHEEL-M-R-F-ADC
- R84 pad 2: Net-(U15-ISEN) -> /MCU-STM32/WHEEL-M-L-F-ADC
- R9 pad 1: Net-(Q14-D) -> Net-(Q9-D)
- U1 pad 1: Net-(U1-OSCI) -> GND
- U1 pad 2: Net-(U1-OSCO) -> 3.3VBAT
- U1 pad 3: /POWER/V-MOTORS-EN -> Net-(U1-IN)
- U1 pad 4: GND -> 3.3VBAT
- U13 pad 14: /MCU-STM32/STM32-RST -> /MCU-STM32/~{STM32_RST}
- U13 pad 55: /MCU-STM32/PD8 -> /MCU-STM32/WDO
- U13 pad 56: /MCU-STM32/PD9 -> /LiDAR/LIDAR_EN
- U13 pad 6: Net-(U13C-VBAT) -> 3.3VBAT
- U13 pad 8: /MCU-STM32/PC14 -> Net-(U13A-PC14-OSC32_IN)
- U13 pad 82: /MAIN-FAN/MAIN-FAN-V-CTRL -> /BUTTON-LED/CLEAN-BTN
- U13 pad 9: /MCU-STM32/PC15 -> Net-(U13A-PC15-OSC32_OUT)
- U14 pad 2: Net-(U14-IN2) -> /MCU-STM32/WHEEL-M-RIGHT-IN2
- U14 pad 3: Net-(U14-IN1) -> /MCU-STM32/WHEEL-M-RIGHT-IN1
- U14 pad 7: Net-(U14-ISEN) -> /MCU-STM32/WHEEL-M-R-F-ADC
- U15 pad 2: Net-(U15-IN2) -> /MCU-STM32/WHEEL-M-LEFT-IN2
- U15 pad 3: Net-(U15-IN1) -> /MCU-STM32/WHEEL-M-LEFT-IN1
- U15 pad 7: Net-(U15-ISEN) -> /MCU-STM32/WHEEL-M-L-F-ADC
- U18 pad 2: Net-(U18-IN2) -> /MCU-STM32/SIDE-BRUSH-IN2
- U18 pad 3: Net-(U18-IN1) -> /MCU-STM32/SIDE-BRUSH-IN1
- U20 pad 2: Net-(U20-IN2) -> /MAIN-BRUSH MOTOR/MAIN-BRUSH-IN2
- U20 pad 3: Net-(U20-IN1) -> /MAIN-BRUSH MOTOR/MAIN-BRUSH-IN1
- U20 pad 7: Net-(U20-ISEN) -> /MAIN-BRUSH MOTOR/MAIN-BRUSH-CURRENT-ADC
- U21 pad 3: BAT-VCC -> +3.3VP
- U22 pad 3: BAT-VCC -> /POWER/POWER-EN
- U23 pad 5: /POWER/V-MOTORS-EN -> /MCU-STM32/~{STM32_RST}
- U7 pad 2: Net-(Q21-D2) -> VCC-CHARG
- U7 pad 3: Net-(Q21-D2) -> VCC-CHARG
- U7 pad 8: VCC-CHARG -> Net-(Q4-D2)
- U8 pad 5: /POWER/V-MOTORS-EN -> /MCU-STM32/~{STM32_RST}
