File: kicad/main/BUTTON-LEDs .kicad_sch (KiCad schematic)
At the start: 15 parts, among them K2 kEY-4, K3 kEY-4, Q10 IRLML6344TRPBF, Q12 IRLML6344TRPBF

Commit message: Fix edge cut; no-CM STEP
Parts:
- R71, R72: footprint Resistor_SMD:R_0603_1608Metric_Pad0.98x0.95mm_HandSolder -> Resistor_SMD:R_0603_1608Metric
Changed lines of the file:
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@@
 		)
 		(instances
-			(project "oomwoo-kicad"
+			(project "Main"
 				(path "/dbcfb655-8d45-4808-9a74-2a0eb03372e8/ee620ee5-1d77-4392-93b6-4acdc78b883b"
 					(reference "K2")
@@
 		)
 		(instances
-			(project "oomwoo-kicad"
+			(project "Main"
 				(path "/dbcfb655-8d45-4808-9a74-2a0eb03372e8/ee620ee5-1d77-4392-93b6-4acdc78b883b"
 					(reference "R120")
@@
 		)
 		(instances
-			(project "oomwoo-kicad"
+			(project "Main"
 				(path "/dbcfb655-8d45-4808-9a74-2a0eb03372e8/ee620ee5-1d77-4392-93b6-4acdc78b883b"
 					(reference "#PWR0622")
@@
 		)
 		(instances
-			(project "oomwoo-kicad"
+			(project "Main"
 				(path "/dbcfb655-8d45-4808-9a74-2a0eb03372e8/ee620ee5-1d77-4392-93b6-4acdc78b883b"
 					(reference "D13")
@@
 		)
 		(instances
-			(project "oomwoo-kicad"
+			(project "Main"
 				(path "/dbcfb655-8d45-4808-9a74-2a0eb03372e8/ee620ee5-1d77-4392-93b6-4acdc78b883b"
 					(reference "D11")
@@
 		)
 		(instances
-			(project "oomwoo-kicad"
+			(project "Main"
 				(path "/dbcfb655-8d45-4808-9a74-2a0eb03372e8/ee620ee5-1d77-4392-93b6-4acdc78b883b"
 					(reference "R124")
@@
 		)
 		(instances
-			(project "oomwoo-kicad"
+			(project "Main"
 				(path "/dbcfb655-8d45-4808-9a74-2a0eb03372e8/ee620ee5-1d77-4392-93b6-4acdc78b883b"
 					(reference "Q10")
@@
 		)
 		(instances
-			(project "oomwoo-kicad"
+			(project "Main"
 				(path "/dbcfb655-8d45-4808-9a74-2a0eb03372e8/ee620ee5-1d77-4392-93b6-4acdc78b883b"
 					(reference "#PWR0619")
@@
 		)
 		(instances
-			(project "oomwoo-kicad"
+			(project "Main"
 				(path "/dbcfb655-8d45-4808-9a74-2a0eb03372e8/ee620ee5-1d77-4392-93b6-4acdc78b883b"
 					(reference "R122")
@@
 		)
 		(instances
-			(project "oomwoo-kicad"
+			(project "Main"
 				(path "/dbcfb655-8d45-4808-9a74-2a0eb03372e8/ee620ee5-1d77-4392-93b6-4acdc78b883b"
 					(reference "#PWR0624")
@@
 		)
 		(instances
-			(project "oomwoo-kicad"
+			(project "Main"
 				(path "/dbcfb655-8d45-4808-9a74-2a0eb03372e8/ee620ee5-1d77-4392-93b6-4acdc78b883b"
 					(reference "#PWR0623")
@@
 			)
 		)
-		(property "Footprint" "Resistor_SMD:R_0603_1608Metric_Pad0.98x0.95mm_HandSolder"
+		(property "Footprint" "Resistor_SMD:R_0603_1608Metric"
 			(at 226.441 268.224 90)
 			(hide yes)
@@
 		)
 		(instances
-			(project "oomwoo-kicad"
+			(project "Main"
 				(path "/dbcfb655-8d45-4808-9a74-2a0eb03372e8/ee620ee5-1d77-4392-93b6-4acdc78b883b"
 					(reference "R72")
@@
 		)
 		(instances
-			(project "oomwoo-kicad"
+			(project "Main"
 				(path "/dbcfb655-8d45-4808-9a74-2a0eb03372e8/ee620ee5-1d77-4392-93b6-4acdc78b883b"
 					(reference "R125")
@@
 		)
 		(instances
-			(project "oomwoo-kicad"
+			(project "Main"
 				(path "/dbcfb655-8d45-4808-9a74-2a0eb03372e8/ee620ee5-1d77-4392-93b6-4acdc78b883b"
 					(reference "#PWR0625")
@@
 		)
 		(instances
-			(project "oomwoo-kicad"
+			(project "Main"
 				(path "/dbcfb655-8d45-4808-9a74-2a0eb03372e8/ee620ee5-1d77-4392-93b6-4acdc78b883b"
 					(reference "D14")
@@
 		)
 		(instances
-			(project "oomwoo-kicad"
+			(project "Main"
 				(path "/dbcfb655-8d45-4808-9a74-2a0eb03372e8/ee620ee5-1d77-4392-93b6-4acdc78b883b"
 					(reference "#PWR0620")
@@
 		)
 		(instances
-			(project "oomwoo-kicad"
+			(project "Main"
 				(path "/dbcfb655-8d45-4808-9a74-2a0eb03372e8/ee620ee5-1d77-4392-93b6-4acdc78b883b"
 					(reference "K3")
@@
 			)
 		)
-		(property "Footprint" "Resistor_SMD:R_0603_1608Metric_Pad0.98x0.95mm_HandSolder"
+		(property "Footprint" "Resistor_SMD:R_0603_1608Metric"
 			(at 226.441 189.484 90)
 			(hide yes)
@@
 		)
 		(instances
-			(project "oomwoo-kicad"
+			(project "Main"
 				(path "/dbcfb655-8d45-4808-9a74-2a0eb03372e8/ee620ee5-1d77-4392-93b6-4acdc78b883b"
 					(reference "R71")
@@
 		)
 		(instances
-			(project "oomwoo-kicad"
+			(project "Main"
 				(path "/dbcfb655-8d45-4808-9a74-2a0eb03372e8/ee620ee5-1d77-4392-93b6-4acdc78b883b"
 					(reference "Q12")
@@
 		)
 		(instances
-			(project "oomwoo-kicad"
+			(project "Main"
 				(path "/dbcfb655-8d45-4808-9a74-2a0eb03372e8/ee620ee5-1d77-4392-93b6-4acdc78b883b"
 					(reference "D12")
@@
 		)
 		(instances
-			(project "oomwoo-kicad"
+			(project "Main"
 				(path "/dbcfb655-8d45-4808-9a74-2a0eb03372e8/ee620ee5-1d77-4392-93b6-4acdc78b883b"
 					(reference "R121")
@@
 		)
 		(instances
-			(project "oomwoo-kicad"
+			(project "Main"
 				(path "/dbcfb655-8d45-4808-9a74-2a0eb03372e8/ee620ee5-1d77-4392-93b6-4acdc78b883b"
 					(reference "#PWR0621")

Commit message: Schematic fixes, 1st round of review
Parts:
- removed D11, D12: LED-HOME, oomwoo_altium:LED0603-B, symbol DesignLibrary:BUTTON-LED_3_LED-SMD_DesignLibrary.SchLib
- removed D13, D14: LED-PWR, oomwoo_altium:LED0603-B, symbol DesignLibrary:BUTTON-LED_3_LED-SMD_DesignLibrary.SchLib
- removed K2, K3: kEY-4, oomwoo_altium:KEY-SMD_4P-L6.0-W6.0-P4.50-LS9.0, symbol DesignLibrary:BUTTON-LED_0_kEY-4_DesignLibrary.SchLib
- removed Q10, Q12: IRLML6344TRPBF, JLCImport:IRLML6344TRPBF, symbol JLCImport:IRLML6344TRPBF
- removed R122, R124, R125: 1K, Resistor_SMD:R_0603_1608Metric, symbol DesignLibrary:BUTTON-LED_1_Resistor-1_DesignLibrary.SchLib
- removed R71, R72: 10, Resistor_SMD:R_0603_1608Metric, symbol Device:R_US
- added HOME1, PWR1: YLED0603B, JLCImport:YLED0603B, symbol JLCImport:YLED0603B
- added R77, R78: 1k, Resistor_SMD:R_0603_1608Metric, symbol Device:R_US
- added SW1, SW2, SW3: TC-6601-5_0-260-8_3, JLCImport:TC-6601-5_0-260-8_3, symbol JLCImport:TC-6601-5_0-260-8_3
- R120, R121: value 1K -> 1k; MANUFACTURER * -> (none); Manufacturer (none) -> *
Connections:
- net GND: now also HOME1.2 (K), PWR1.2 (K), SW1.1, SW1.2, SW2.1, SW2.2, SW3.1, SW3.2
- net HOME-BTN: now also SW2.3, SW2.4
- net LED-HOME: now also R77.1
- net LED-PWR: now also R78.1
- net POWER-BTN: now also SW1.3, SW1.4
- net VCC-3V3-P: now also R121.2
- net CLEAN-BTN: now reaches R121.1
- net CLEAN-BTN: now also SW3.3, SW3.4
- new net: PWR1.1 (A), R78.2
- new net: HOME1.1 (A), R77.2
