File: kicad/main/Battery-Charger.kicad_sch (KiCad schematic)
At the start: 69 parts, among them CN1 EV2400, IC5 TPS25730DREFR, IC6 TVS2200DRVR, IC7 TVS2200DRVR, J1 BATTERY, Q26 CSD17581Q3A, Q27 CSD17581Q3A, Q28 CSD17581Q3A, Q29 CSD17581Q3A, U7 BQ25792RQMR

Commit message: Fix edge cut; no-CM STEP
Parts:
- removed C62, C63: 1nF/50V, Capacitor_SMD:C_0603_1608Metric, symbol Device:C
- removed CN1: EV2400, JLCImport:22053041_C5271241, symbol JLCImport:22053041_C5271241
- removed D32, D33: BZT52C12T-7, JLCImport:BZT52C12T-7, symbol JLCImport:BZT52C12T-7
- removed D4: SMCJ18A-13-F, JLCImport:SMCJ18A-13-F, symbol JLCImport:SMCJ18A-13-F
- removed IC6, IC7: TVS2200DRVR, TLV76733DRVR:SON65P200X200X80-7N, symbol SamacSys_Parts:TVS2200DRVR
- removed J1: BATTERY, oomwoo_altium:CONN-SMD_4P-P2.00_XUNPU_WAFER-PH2.0-4PWB, symbol DesignLibrary:POWER_2_HDRx4_DesignLibrary.SchLib
- removed Q26, Q27, Q28, Q29: CSD17581Q3A, CSD17581Q3A:TRANS_CSD17581Q3A, symbol CSD17581Q3A:CSD17581Q3A
- removed R58, R59: 100, Resistor_SMD:R_0603_1608Metric, symbol Device:R_US
- added C125, C126: 1nF/50V, Capacitor_SMD:C_0603_1608Metric, symbol Device:C
- added C94: 10uF/35V, Capacitor_SMD:C_0603_1608Metric, symbol Device:C
- added CN2: EV2400, JLCImport:A2543WV-4P, symbol JLCImport:A2543WV-4P
- added CONTACT_CHGR1: WAFER-PH2_0-4PWB, JLCImport:WAFER-PH2_0-4PWB, symbol JLCImport:WAFER-PH2_0-4PWB
- added D1, D2: TVS2200DRVR, JLCImport:TVS2200DRVR, symbol JLCImport:TVS2200DRVR
- added D3: SMAJ18A_C148219, JLCImport:SMAJ18A_C148219, symbol JLCImport:SMAJ18A_C148219
- added D39, D40: BZT52C12T-7, JLCImport:BZT52C12T-7, symbol JLCImport:BZT52C12T-7
- added Q21, Q4: SQJ844AEP-T1_GE3, JLCImport:SQJ844AEP-T1_GE3, symbol JLCImport:SQJ844AEP-T1_GE3
- added R75, R76: 100, Resistor_SMD:R_0603_1608Metric, symbol Device:R_US
- C60: value 0.1uF/50V -> 10uF/35V
- C80: footprint Capacitor_SMD:C_0805_2012Metric -> Capacitor_SMD:C_0603_1608Metric
- IC5: footprint SamacSys_Parts:TPS25730DREFR -> LIB_TPS25730DREFR:TPS25730DREFR
- R129: footprint JLCImport:RC0402FR-0717K4L -> Resistor_SMD:R_0603_1608Metric
- R132: value 100 -> 10k
- R99: footprint JLCImport:RC0402FR-07215KL -> Resistor_SMD:R_0603_1608Metric
Connections:
- net BAT-VCC: now also D3.1
- net GND: now also C94.2, CN2.1, CONTACT_CHGR1.1, CONTACT_CHGR1.2, CONTACT_CHGR1.5, CONTACT_CHGR1.6, D1.1 (GND), D1.2 (GND), D1.3 (GND), D1.7 (GND), D2.1 (GND), D2.2 (GND), D2.3 (GND), D2.7 (GND), D3.2
- net SCL: now also CN2.2
- net SDA: now also CN2.3
- net VBUS: now also D2.4 (IN), D2.5 (IN), D2.6 (IN)
- net VCC-CHARG: now also C94.1, CONTACT_CHGR1.3, CONTACT_CHGR1.4, D1.4 (IN), D1.5 (IN), D1.6 (IN), Q4.5 (D2)
- net VOUT_PD: now also Q21.6 (D1)
- net at C67.2, C68.2, C69.1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: now also Q21.5 (D2), Q4.6 (D1)
- net at U7.10 (ACDRV2): now also R75.2
- net at U7.11 (ACDRV1): now also R76.2
- new net: C125.1, D39.2 (A), Q4.1 (S1), Q4.3 (S2)
- new net: C125.2, D39.1 (K), Q4.2 (G1), Q4.4 (G2), R75.1
- new net: C126.2, D40.1 (K), Q21.2 (G1), Q21.4 (G2), R76.1
- new net: C126.1, D40.2 (A), Q21.1 (S1), Q21.3 (S2)

Commit message: Schematic fixes, 1st round of review
Parts:
- C100, C60, C66, C67, C68, C71, C72, C74, C76, C80, C81, C82, C94, C96, C97, C98, C99: value 10uF/35V -> 10uF/25V; LCSC (none) -> C96446
- C125, C126: LCSC C23733 -> (none); Manufacturer Part CL05A475MP5NRNC -> (none)
- C47, C58: value 330pF/35V -> 330pF/25V
- C59, C61, C64, C65, C73: value 0.1uF/35V -> 100nF/50V; LCSC (none) -> C1591
- C69, C78, C83: value 0.1uF/50V -> 10uF/25V; LCSC (none) -> C96446
- C70: value 4.7uF/10V -> 10uF/25V; LCSC C23733 -> C96446; Manufacturer Part CL05A475MP5NRNC -> (none)
- D29: LCSC (none) -> C19171394; MANUFACTURER * -> (none); Manufacturer (none) -> *
- D34: LCSC (none) -> C97502
- IC5: LCSC (none) -> C22438973
- R100, R75, R76: footprint Resistor_SMD:R_0603_1608Metric -> Resistor_SMD:R_0805_2012Metric
- R115: LCSC C2906859 -> (none); Manufacturer Part FRC0402F1003TS -> (none)
- R130: value 162k -> 100k
- R131: value 38k -> 20k
- R133: value 190k -> 100k
- R136: value 9.5k -> 5.24k
- R137: value 9.4k -> 5.24k
- R138: value 191k -> 100k
- R139: value 198.2k -> 100k
- R140: value 2.28k -> 1k
- R37: value 1K -> 1k; MANUFACTURER * -> (none); Manufacturer (none) -> *
- USB2: LCSC (none) -> C37616412
Connections:
- net VCC-CHARG: now also C67.2, C68.2, C69.1, Q21.5 (D2), Q4.6 (D1), U7.2 (VBUS), U7.3 (VBUS); no longer C94.1, CONTACT_CHGR1.3, CONTACT_CHGR1.4, D1.4 (IN), D1.5 (IN), D1.6 (IN), Q4.5 (D2), U7.8 (VAC2)
- new net: C94.1, CONTACT_CHGR1.3, CONTACT_CHGR1.4, D1.4 (IN), D1.5 (IN), D1.6 (IN), Q4.5 (D2), U7.8 (VAC2)
