File: kicad/main/CM5-Highspeed.kicad_sch (KiCad schematic)
At the start: 3 parts

Commit message: Fix edge cut; no-CM STEP
Parts:
- R101, R96: footprint (none) -> Resistor_SMD:R_0603_1608Metric
Changed lines of the file:
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@@
 		)
 		(instances
-			(project "oomwoo-kicad"
+			(project "Main"
 				(path "/dbcfb655-8d45-4808-9a74-2a0eb03372e8/2d8a25d6-58b7-409a-a3b1-0c610bb70760"
 					(reference "#PWR032")
@@
 			)
 		)
-		(property "Footprint" ""
+		(property "Footprint" "Resistor_SMD:R_0603_1608Metric"
 			(at 377.444 82.804 90)
 			(hide yes)
@@
 		)
 		(instances
-			(project "oomwoo-kicad"
+			(project "Main"
 				(path "/dbcfb655-8d45-4808-9a74-2a0eb03372e8/2d8a25d6-58b7-409a-a3b1-0c610bb70760"
 					(reference "R96")
@@
 		)
 		(instances
-			(project "oomwoo-kicad"
+			(project "Main"
 				(path "/dbcfb655-8d45-4808-9a74-2a0eb03372e8/2d8a25d6-58b7-409a-a3b1-0c610bb70760"
 					(reference "#PWR017")
@@
 			)
 		)
-		(property "Footprint" ""
+		(property "Footprint" "Resistor_SMD:R_0603_1608Metric"
 			(at 377.444 85.344 90)
 			(hide yes)
@@
 		)
 		(instances
-			(project "oomwoo-kicad"
+			(project "Main"
 				(path "/dbcfb655-8d45-4808-9a74-2a0eb03372e8/2d8a25d6-58b7-409a-a3b1-0c610bb70760"
 					(reference "R101")
@@
 		)
 		(instances
-			(project "oomwoo-kicad"
+			(project "Main"
 				(path "/dbcfb655-8d45-4808-9a74-2a0eb03372e8/2d8a25d6-58b7-409a-a3b1-0c610bb70760"
 					(reference "Module1")

Commit message: Schematic fixes, 1st round of review
Parts:
- added JP1, JP2: (no value), Jumper:SolderJumper-2_P1.3mm_Open_RoundedPad1.0x1.5mm, symbol Jumper:SolderJumper_2_Open
- Module1: LCSC (none) -> 2X C6932320
Connections:
- net PCIE_nWAKE: now also JP1.1 (A); no longer Module1.104 (PCIE_nWAKE)
- net at Module1.106 (PCIE_PWR_EN): now also JP2.2 (B)
- new net: JP1.2 (B), Module1.104 (PCIE_nWAKE)
- new net PCIE_PWR_EN: JP2.1 (A)
- no-connect marks 41 -> 40
