File: kicad/main/Front Sensors.kicad_sch (KiCad schematic)
At the start: 17 parts, among them Q19 IRLML6344TRPBF, U17 ZX-ZH1_5-2PWT

Commit message: Fix edge cut; no-CM STEP
Parts:
- removed R36: 47k, symbol Device:R_US
- added C19: 4.7uF/10V, Capacitor_SMD:C_0603_1608Metric, symbol Device:C_Small
- C6, C90, C91: footprint (none) -> Capacitor_SMD:C_0603_1608Metric
- R2, R5, R6, R61, R62, R7: footprint (none) -> Resistor_SMD:R_0603_1608Metric
- renumbered U17 to LIGHT1
Connections:
- net GND: now also C19.2
- net VCC-3V3-P: now also C19.1; no longer C6.1, VL-L1.1
- new net: C6.1, VL-L1.1

Commit message: Schematic fixes, 1st round of review
Parts:
- removed Q19: IRLML6344TRPBF, JLCImport:IRLML6344TRPBF, symbol JLCImport:IRLML6344TRPBF
- added Q2: 2302V, JLCImport:2302V, symbol JLCImport:2302V
- added R54: 100k, Resistor_SMD:R_0603_1608Metric, symbol Device:R_US
- C123: value 10uF/50V -> 10uF/25V; LCSC C2932476 -> C96446; MPN CL21A106KBYQNNE -> (none); Manufacturer Part CL21A106KBYQNNE -> (none)
- C19, C6, C90, C91: value 4.7uF/10V -> 10uF/25V; LCSC (none) -> C96446
Connections:
- net GND: now also Q2.2 (S), R54.2
- net LIGHT-ON: now also Q2.1 (G), R54.1
- net at C123.1, LIGHT1.2: now also Q2.3 (D)
