File: kicad/main/IMU-ICM-4267-P .kicad_sch (KiCad schematic)
At the start: 7 parts, among them U19 ICM-42607-P

Commit message: Fix edge cut; no-CM STEP
Parts:
- U19: footprint oomwoo_altium:LGA-14_L3.0-W2.5-P0.50-TL_QMI8658A -> JLCImport:ICM-42607-P
Changed lines of the file:
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@@
 		)
 		(instances
-			(project "oomwoo-kicad"
+			(project "Main"
 				(path "/dbcfb655-8d45-4808-9a74-2a0eb03372e8/7b57c0fa-4a35-4109-8672-3c36267bf8ff"
 					(reference "#PWR089")
@@
 		)
 		(instances
-			(project "oomwoo-kicad"
+			(project "Main"
 				(path "/dbcfb655-8d45-4808-9a74-2a0eb03372e8/7b57c0fa-4a35-4109-8672-3c36267bf8ff"
 					(reference "R93")
@@
 		)
 		(instances
-			(project "oomwoo-kicad"
+			(project "Main"
 				(path "/dbcfb655-8d45-4808-9a74-2a0eb03372e8/7b57c0fa-4a35-4109-8672-3c36267bf8ff"
 					(reference "#PWR0692")
@@
 		)
 		(instances
-			(project "oomwoo-kicad"
+			(project "Main"
 				(path "/dbcfb655-8d45-4808-9a74-2a0eb03372e8/7b57c0fa-4a35-4109-8672-3c36267bf8ff"
 					(reference "C110")
@@
 		)
 		(instances
-			(project "oomwoo-kicad"
+			(project "Main"
 				(path "/dbcfb655-8d45-4808-9a74-2a0eb03372e8/7b57c0fa-4a35-4109-8672-3c36267bf8ff"
 					(reference "C108")
@@
 		)
 		(instances
-			(project "oomwoo-kicad"
+			(project "Main"
 				(path "/dbcfb655-8d45-4808-9a74-2a0eb03372e8/7b57c0fa-4a35-4109-8672-3c36267bf8ff"
 					(reference "R18")
@@
 		)
 		(instances
-			(project "oomwoo-kicad"
+			(project "Main"
 				(path "/dbcfb655-8d45-4808-9a74-2a0eb03372e8/7b57c0fa-4a35-4109-8672-3c36267bf8ff"
 					(reference "#PWR0690")
@@
 			)
 		)
-		(property "Footprint" "oomwoo_altium:LGA-14_L3.0-W2.5-P0.50-TL_QMI8658A"
+		(property "Footprint" "JLCImport:ICM-42607-P"
 			(at 290.195 192.405 0)
 			(hide yes)
@@
 		)
 		(instances
-			(project "oomwoo-kicad"
+			(project "Main"
 				(path "/dbcfb655-8d45-4808-9a74-2a0eb03372e8/7b57c0fa-4a35-4109-8672-3c36267bf8ff"
 					(reference "U19")
@@
 		)
 		(instances
-			(project "oomwoo-kicad"
+			(project "Main"
 				(path "/dbcfb655-8d45-4808-9a74-2a0eb03372e8/7b57c0fa-4a35-4109-8672-3c36267bf8ff"
 					(reference "R92")
@@
 		)
 		(instances
-			(project "oomwoo-kicad"
+			(project "Main"
 				(path "/dbcfb655-8d45-4808-9a74-2a0eb03372e8/7b57c0fa-4a35-4109-8672-3c36267bf8ff"
 					(reference "C109")
@@
 		)
 		(instances
-			(project "oomwoo-kicad"
+			(project "Main"
 				(path "/dbcfb655-8d45-4808-9a74-2a0eb03372e8/7b57c0fa-4a35-4109-8672-3c36267bf8ff"
 					(reference "#PWR088")

Commit message: Schematic fixes, 1st round of review
Parts:
- C108: value 2.2uF -> 10uF/25V; LCSC (none) -> C96446; MANUFACTURER * -> (none); Manufacturer (none) -> *
- C109: value 100nF -> 100nF/50V; LCSC (none) -> C1591; MANUFACTURER * -> (none); Manufacturer (none) -> *
- C110: value 10nF -> 47nF/50V; MANUFACTURER * -> (none); Manufacturer (none) -> *
- R18, R92, R93: value 10K -> 10k; MANUFACTURER * -> (none); Manufacturer (none) -> *
- U19: LCSC (none) -> C5129967; MANUFACTURER * -> (none); Manufacturer (none) -> *
