File: kicad/main/M.2.kicad_sch (KiCad schematic)
At the start: 15 parts, among them J2 1-2199119-5, Y1 ASEK-32.768KHZ-LRT

Commit message: Fix edge cut; no-CM STEP
Parts:
- removed C51: 875105242010, LIB_875105242010:CAPAE530X550N, symbol 875105242010:875105242010
- removed D3: (no value), LED_SMD:LED_0603_1608Metric, symbol Library:LED
- removed R57: (no value), Resistor_SMD:R_0603_1608Metric, symbol Library:R
- added C36: JBLM2101M025C058RTM_100UF_25V, JLCImport:JBLM2101M025C058RTM_100UF_25V, symbol JLCImport:JBLM2101M025C058RTM_100UF_25V
- added MP4: M3 x 1.5mm, MountingHole:MountingHole_3.2mm_M3_Pad, symbol WA-SMSI_9774XXX360:WA-SMSI_9774XXX360
- C41, C43, C48, C49: value (none) -> 100nF/50V
- C45: value (none) -> 10uF/10V; footprint Capacitor_SMD:C_0805_2012Metric -> Capacitor_SMD:C_0603_1608Metric; Field4 Digikey -> (none); Field5 490-14381-1-ND -> (none); Field6 GRM21BR71A106KA73L -> (none); Field7 Murata -> (none); Part Description 10uF 10% 10V Ceramic Capacitor X7R 0805 (2012 Metric) -> (none)
- C50: value (none) -> 100nF/50V; Field4 Farnell -> (none); Field5 2611911 -> (none); Field6 RM EMK105 B7104KV-F -> (none); Field7 TAIYO YUDEN EUROPE GMBH -> (none); Part Description 0.1uF 10% 16V Ceramic Capacitor X7R 0402 (1005 Metric) -> (none)
- MP1, MP2, MP3: footprint WA-SMSI_9774XXX360:WA-SMSI_9774015360 -> MountingHole:MountingHole_3.2mm_M3_Pad
- R56: value (none) -> 10k
Connections:
- net GND: now also C36.2, MP4.1
- net VCC3V3_M2: now also C36.1
- net PCIE_LED: no longer names the net of J2.10 (P10)
- no-connect marks 32 -> 33

Commit message: Schematic fixes, 1st round of review
Parts:
- removed C36: JBLM2101M025C058RTM_100UF_25V, JLCImport:JBLM2101M025C058RTM_100UF_25V, symbol JLCImport:JBLM2101M025C058RTM_100UF_25V
- removed C41, C43, C48, C49: 100nF/50V, Capacitor_SMD:C_0603_1608Metric, symbol Library:C
- removed R56: 10k, Resistor_SMD:R_0603_1608Metric, symbol Library:R_US
- added M2_ACT1: YLED0603B, JLCImport:YLED0603B, symbol JLCImport:YLED0603B
- added R79: 1k, Resistor_SMD:R_0603_1608Metric, symbol Device:R_US
- C45: value 10uF/10V -> 10uF/25V; LCSC (none) -> C96446
- C50: LCSC (none) -> C1591
- J2: LCSC (none) -> C574849; PACKAGE None -> (none); PRICE None -> (none)
- MP1, MP2, MP3, MP4: MP 9774015360R -> (none)
- Y1: LCSC (none) -> C2650753; MANUFACTURER Abracon -> (none); Manufacturer (none) -> Abracon
Connections:
- net GND: no longer J2.69 (P69)
- net PCIE_RX_N: now also J2.43 (P43); no longer J2.41 (P41)
- net PCIE_RX_P: now also J2.41 (P41); no longer J2.43 (P43)
- net PCIE_TX_N: now also J2.49 (P49); no longer J2.47 (P47)
- net PCIE_TX_P: now also J2.47 (P47); no longer J2.49 (P49)
- net VCC3V3_M2: now also R79.1
- net at J2.10 (P10): now also M2_ACT1.2 (K)
- new net: M2_ACT1.1 (A), R79.2
