File: kicad/main/MAIN-BRUSH-MOTOR .kicad_sch (KiCad schematic)
At the start: 9 parts, among them J11 MAIN BRUSH, U20 DRV8870DDAR

Commit message: Fix edge cut; no-CM STEP
Parts:
- removed C104: 100uF, oomwoo_altium:CAP-SMD_BD6.3-L6.6-W6.6-FD, symbol DesignLibrary:WHEEL MOTOR_3_Capacitor-2_DesignLibrary.SchLib
- removed J11: MAIN BRUSH, oomwoo_altium:CONN-SMD_2P-P2.00_XUNPU_WAFER-PH2.0-2PWB, symbol DesignLibrary:MAIN-BRUSH MOTOR_0_HDRx2_DesignLibrary.SchLib
- added C21: JBLM2101M025C058RTM_100UF_25V, JLCImport:JBLM2101M025C058RTM_100UF_25V, symbol JLCImport:JBLM2101M025C058RTM_100UF_25V
- added MAIN_BRUSH1: ZX-ZH1_5-2PWT, JLCImport:ZX-ZH1_5-2PWT, symbol JLCImport:ZX-ZH1_5-2PWT
- R112: value 0.2R -> 0.2R/10W; footprint Resistor_SMD:R_0603_1608Metric -> Resistor_SMD:R_2512_6332Metric
- U20: footprint oomwoo_altium:HSOP-8_L5.0-W4.0-P1.27-LS6.2-BL-EP -> JLCImport:DRV8870DDAR
Connections:
- net GND: now also C21.2, MAIN_BRUSH1.3, MAIN_BRUSH1.4
- net VM-VBAT: now also C21.1
- net at U20.6 (OUT1): now also MAIN_BRUSH1.1
- net at U20.8 (OUT2): now also MAIN_BRUSH1.2
Other:
- moved on the sheet: C103

Commit message: Schematic fixes, 1st round of review
Parts:
- removed C21: JBLM2101M025C058RTM_100UF_25V, JLCImport:JBLM2101M025C058RTM_100UF_25V, symbol JLCImport:JBLM2101M025C058RTM_100UF_25V
- removed D31: 1N4007, oomwoo_altium:SOD123, symbol DesignLibrary:WHEEL MOTOR_3_DIODE-1_DesignLibrary.SchLib
- removed R106, R107, R111: 10K, Resistor_SMD:R_0603_1608Metric, symbol DesignLibrary:WHEEL MOTOR_0_Resistor-1_DesignLibrary.SchLib
- added C134: 10uF/25V, Capacitor_SMD:C_0603_1608Metric, symbol JLCImport:CL21A106KBYQNNE
- added R3, R4: 100k, Resistor_SMD:R_0603_1608Metric, symbol Device:R_US
- C103: value 0.22uF -> 100nF/50V; LCSC (none) -> C1591; MANUFACTURER * -> (none); Manufacturer (none) -> *
- R112: LCSC (none) -> C5375488; MANUFACTURER * -> (none); Manufacturer (none) -> *
- U20: LCSC (none) -> C86590; MANUFACTURER * -> (none); Manufacturer (none) -> *
Connections:
- net GND: now also C134.2, R3.2, R4.2
- net MAIN-BRUSH-CURRENT-ADC: now also R112.2, U20.7 (ISEN)
- net MAIN-BRUSH-IN1: now also U20.3 (IN1), R3.1
- net MAIN-BRUSH-IN2: now also U20.2 (IN2), R4.1
- net VM-VBAT: now also C134.1
