File: kicad/main/MIPI-CAMERA.kicad_sch (KiCad schematic)
At the start: 7 parts

Commit message: Schematic fixes, 1st round of review
Parts:
- added JP3: (no value), Jumper:SolderJumper-2_P1.3mm_Open_RoundedPad1.0x1.5mm, symbol Jumper:SolderJumper_2_Open
- added TP1, TP2, TP3: TestPoint, TestPoint:TestPoint_Pad_D2.0mm, symbol Connector:TestPoint
- C23, C28, C29: LCSC (none) -> C1591
- CAM0, MIPI0, MIPI1: LCSC (none) -> C3168538; MANUFACTURER Amphoenol FCI -> (none); Manufacturer (none) -> Amphoenol FCI
Connections:
- net at CAM0.12: now also TP3.1
- net at MIPI0.12: now also JP3.1 (A), TP1.1
- net at MIPI1.12: now also TP2.1
- net CAM_IO renamed CAM_GPIO0
- new net CAM_GPIO1: JP3.2 (B)
- no-connect marks 3 -> 0
Other:
- moved on the sheet: C23
