File: kicad/main/Main.kicad_sch (KiCad schematic)
At the start: 10 parts

Commit message: Side sensor VL6180
Other:
- sheet MCU-STM32 ports: added I2C4_SCL, I2C4_SDA, SIDE-PROXI-CE-L, SIDE-PROXI-CE-R, SIDE-PROXI-GPIO-L, SIDE-PROXI-GPIO-R; removed USART2-IR-L-TX, USART4-IR-R-TX
- sheet SIDE-PROXI ports: added CE-L, CE-R, GPIO1-L, GPIO1-R, SCL, SDA; removed IR-L-TX, IR-R-TX
- note added: "RTC_WD"
Changed lines of the file:
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@@
 		)
 	)
+	(text "RTC_WD"
+		(exclude_from_sim no)
+		(at 480.695 86.995 0)
+		(effects
+			(font
+				(size 3.048 3.048)
+				(thickness 0.6096)
+				(bold yes)
+				(italic yes)
+			)
+			(justify left bottom)
+		)
+	)
 	(text "ANTI-FALL IR"
 		(exclude_from_sim no)
@@
 	(text "SIDE PROXI SENSOR"
 		(exclude_from_sim no)
-		(at 250.19 33.02 0)
+		(at 263.525 29.21 0)
 		(effects
 			(font
@@
 	(wire
 		(pts
-			(xy 224.155 114.3) (xy 224.155 41.275)
+			(xy 213.995 114.3) (xy 213.995 26.67)
 		)
 		(stroke
@@
 	(wire
 		(pts
-			(xy 224.155 41.275) (xy 245.11 41.275)
+			(xy 213.995 26.67) (xy 245.11 26.67)
 		)
 		(stroke
@@
 	(wire
 		(pts
+			(xy 236.855 51.435) (xy 245.11 51.435)
+		)
+		(stroke
+			(width 0)
+			(type default)
+		)
+	)
+	(wire
+		(pts
+			(xy 216.535 114.3) (xy 216.535 28.575)
+		)
+		(stroke
+			(width 0)
+			(type default)
+		)
+	)
+	(wire
+		(pts
 			(xy 394.97 261.62) (xy 443.865 261.62)
 		)
@@
 	(wire
 		(pts
-			(xy 234.95 48.895) (xy 245.11 48.895)
+			(xy 228.6 44.45) (xy 245.11 44.45)
 		)
 		(stroke
@@
 	(wire
 		(pts
+			(xy 236.855 114.3) (xy 236.855 51.435)
+		)
+		(stroke
+			(width 0)
+			(type default)
+		)
+	)
+	(wire
+		(pts
+			(xy 219.075 30.48) (xy 219.075 114.3)
+		)
+		(stroke
+			(width 0)
+			(type default)
+		)
+	)
+	(wire
+		(pts
 			(xy 394.97 349.885) (xy 443.865 349.885)
 		)
@@
 	(wire
 		(pts
+			(xy 239.395 53.34) (xy 239.395 114.3)
+		)
+		(stroke
+			(width 0)
+			(type default)
+		)
+	)
+	(wire
+		(pts
 			(xy 351.155 140.97) (xy 351.155 123.825)
 		)
@@
 	(wire
 		(pts
+			(xy 245.11 46.355) (xy 231.14 46.355)
+		)
+		(stroke
+			(width 0)
+			(type default)
+		)
+	)
+	(wire
+		(pts
 			(xy 100.33 147.701) (xy 148.59 147.701)
 		)
@@
 	(wire
 		(pts
-			(xy 233.045 46.99) (xy 233.045 114.3)
+			(xy 226.06 42.545) (xy 226.06 114.3)
 		)
 		(stroke
@@
 	(wire
 		(pts
+			(xy 228.6 114.3) (xy 228.6 44.45)
+		)
+		(stroke
+			(width 0)
+			(type default)
+		)
+	)
+	(wire
+		(pts
 			(xy 426.72 208.28) (xy 443.865 208.28)
 		)
@@
 	(wire
 		(pts
-			(xy 234.95 114.3) (xy 234.95 48.895)
+			(xy 194.31 234.315) (xy 194.31 259.715)
 		)
 		(stroke
@@
 	(wire
 		(pts
-			(xy 194.31 234.315) (xy 194.31 259.715)
+			(xy 231.14 46.355) (xy 231.14 114.3)
 		)
 		(stroke
@@
 	(wire
 		(pts
+			(xy 245.11 30.48) (xy 219.075 30.48)
+		)
+		(stroke
+			(width 0)
+			(type default)
+		)
+	)
+	(wire
+		(pts
+			(xy 245.11 53.34) (xy 239.395 53.34)
+		)
+		(stroke
+			(width 0)
+			(type default)
+		)
+	)
+	(wire
+		(pts
 			(xy 394.97 278.765) (xy 443.865 278.765)
 		)
@@
 	(wire
 		(pts
-			(xy 226.06 43.18) (xy 226.06 114.3)
-		)
-		(stroke
-			(width 0)
-			(type default)
-		)
-	)
-	(wire
-		(pts
 			(xy 429.26 85.09) (xy 429.26 210.185)
 		)
@@
 	(wire
 		(pts
+			(xy 216.535 28.575) (xy 245.11 28.575)
+		)
+		(stroke
+			(width 0)
+			(type default)
+		)
+	)
+	(wire
+		(pts
 			(xy 262.89 228.6) (xy 306.07 228.6)
 		)
@@
 	(wire
 		(pts
-			(xy 245.11 46.99) (xy 233.045 46.99)
+			(xy 245.11 42.545) (xy 226.06 42.545)
 		)
 		(stroke
@@
 	(wire
 		(pts
-			(xy 245.11 43.18) (xy 226.06 43.18)
-		)
-		(stroke
-			(width 0)
-			(type default)
-		)
-	)
-	(wire
-		(pts
 			(xy 100.33 168.021) (xy 148.59 168.021)
 		)
@@
 		)
 		(pin "IR-L-RX" output
-			(at 245.11 41.275 180)
+			(at 245.11 26.67 180)
 			(effects
 				(font
@@
 			)
 		)
-		(pin "IR-L-TX" input
-			(at 245.11 43.18 180)
+		(pin "IR-R-RX" output
+			(at 245.11 42.545 180)
 			(effects
 				(font
@@
 			)
 		)
-		(pin "IR-R-RX" output
-			(at 245.11 46.99 180)
+		(pin "CE-L" input
+			(at 245.11 28.575 180)
+			(effects
+				(font
+					(size 1.27 1.27)
+				)
+				(justify left)
+			)
+		)
+		(pin "CE-R" input
+			(at 245.11 44.45 180)
+			(effects
+				(font
+					(size 1.27 1.27)
+				)
+				(justify left)
+			)
+		)
+		(pin "GPIO1-L" input
+			(at 245.11 30.48 180)
+			(effects
+				(font
+					(size 1.27 1.27)
+				)
+				(justify left)
+			)
+		)
+		(pin "GPIO1-R" input
+			(at 245.11 46.355 180)
 			(effects
 				(font
@@
 			)
 		)
-		(pin "IR-R-TX" input
-			(at 245.11 48.895 180)
+		(pin "SCL" input
+			(at 245.11 53.34 180)
+			(effects
+				(font
+					(size 1.27 1.27)
+				)
+				(justify left)
+			)
+		)
+		(pin "SDA" bidirectional
+			(at 245.11 51.435 180)
 			(effects
 				(font
@@
 			)
 		)
-		(pin "MAIN-BRUSH-IN1" input
+		(pin "MAIN-BRUSH-IN1" output
 			(at 148.59 129.54 180)
 			(effects
@@
 			)
 		)
-		(pin "MAIN-BRUSH-IN2" input
+		(pin "MAIN-BRUSH-IN2" output
 			(at 148.59 131.445 180)
 			(effects
@@
 			)
 		)
-		(pin "SIDE-BRUSH-IN1" input
+		(pin "SIDE-BRUSH-IN1" output
 			(at 148.59 205.74 180)
 			(effects
@@
 			)
 		)
-		(pin "SIDE-BRUSH-IN2" input
+		(pin "SIDE-BRUSH-IN2" output
 			(at 148.59 207.645 180)
 			(effects
@@
 		)
 		(pin "USART2-IR-L-RX" input
-			(at 233.045 114.3 90)
+			(at 226.06 114.3 90)
 			(effects
 				(font
@@
 			)
 		)
-		(pin "USART4-IR-R-TX" output
-			(at 234.95 114.3 90)
+		(pin "USART4-IR-R-RX" input
+			(at 213.995 114.3 90)
 			(effects
 				(font
@@
 			)
 		)
-		(pin "USART2-IR-L-TX" output
-			(at 226.06 114.3 90)
+		(pin "I2C4_SCL" input
+			(at 239.395 114.3 90)
 			(effects
 				(font
@@
 			)
 		)
-		(pin "USART4-IR-R-RX" input
-			(at 224.155 114.3 90)
+		(pin "I2C4_SDA" input
+			(at 236.855 114.3 90)
+			(effects
+				(font
+					(size 1.27 1.27)
+				)
+				(justify right)
+			)
+		)
+		(pin "SIDE-PROXI-CE-L" output
+			(at 216.535 114.3 90)
+			(effects
+				(font
+					(size 1.27 1.27)
+				)
+				(justify right)
+			)
+		)
+		(pin "SIDE-PROXI-CE-R" output
+			(at 228.6 114.3 90)
+			(effects
+				(font
+					(size 1.27 1.27)
+				)
+				(justify right)
+			)
+		)
+		(pin "SIDE-PROXI-GPIO-L" input
+			(at 219.075 114.3 90)
+			(effects
+				(font
+					(size 1.27 1.27)
+				)
+				(justify right)
+			)
+		)
+		(pin "SIDE-PROXI-GPIO-R" input
+			(at 231.14 114.3 90)
 			(effects
 				(font
@@
 		)
 		(fill
-			(color 0 0 0 0)
+			(color 128 255 128 1)
 		)
 		(property "Sheetname" "RTC_WATCHDOG"

Commit message: Fix edge cut; no-CM STEP
Parts:
- R1, R51, R52, R53, R54, R55, R63, R65, R66, R67: footprint (none) -> Resistor_SMD:R_0603_1608Metric
Changed lines of the file:
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@@
 			)
 		)
-		(property "Footprint" ""
+		(property "Footprint" "Resistor_SMD:R_0603_1608Metric"
 			(at 268.224 253.619 90)
 			(hide yes)
@@
 		)
 		(instances
-			(project "oomwoo-kicad"
+			(project "Main"
 				(path "/dbcfb655-8d45-4808-9a74-2a0eb03372e8"
 					(reference "R53")
@@
 			)
 		)
-		(property "Footprint" ""
+		(property "Footprint" "Resistor_SMD:R_0603_1608Metric"
 			(at 294.259 261.239 90)
 			(hide yes)
@@
 		)
 		(instances
-			(project "oomwoo-kicad"
+			(project "Main"
 				(path "/dbcfb655-8d45-4808-9a74-2a0eb03372e8"
 					(reference "R63")
@@
 			)
 		)
-		(property "Footprint" ""
+		(property "Footprint" "Resistor_SMD:R_0603_1608Metric"
 			(at 285.369 258.699 90)
 			(hide yes)
@@
 		)
 		(instances
-			(project "oomwoo-kicad"
+			(project "Main"
 				(path "/dbcfb655-8d45-4808-9a74-2a0eb03372e8"
 					(reference "R55")
@@
 			)
 		)
-		(property "Footprint" ""
+		(property "Footprint" "Resistor_SMD:R_0603_1608Metric"
 			(at 277.114 256.159 90)
 			(hide yes)
@@
 		)
 		(instances
-			(project "oomwoo-kicad"
+			(project "Main"
 				(path "/dbcfb655-8d45-4808-9a74-2a0eb03372e8"
 					(reference "R54")
@@
 			)
 		)
-		(property "Footprint" ""
+		(property "Footprint" "Resistor_SMD:R_0603_1608Metric"
 			(at 347.599 135.001 90)
 			(hide yes)
@@
 		)
 		(instances
-			(project "oomwoo-kicad"
+			(project "Main"
 				(path "/dbcfb655-8d45-4808-9a74-2a0eb03372e8"
 					(reference "R65")
@@
 			)
 		)
-		(property "Footprint" ""
+		(property "Footprint" "Resistor_SMD:R_0603_1608Metric"
 			(at 249.809 248.539 90)
 			(hide yes)
@@
 		)
 		(instances
-			(project "oomwoo-kicad"
+			(project "Main"
 				(path "/dbcfb655-8d45-4808-9a74-2a0eb03372e8"
 					(reference "R51")
@@
 			)
 		)
-		(property "Footprint" ""
+		(property "Footprint" "Resistor_SMD:R_0603_1608Metric"
 			(at 240.919 245.999 90)
 			(hide yes)
@@
 		)
 		(instances
-			(project "oomwoo-kicad"
+			(project "Main"
 				(path "/dbcfb655-8d45-4808-9a74-2a0eb03372e8"
 					(reference "R1")
@@
 			)
 		)
-		(property "Footprint" ""
+		(property "Footprint" "Resistor_SMD:R_0603_1608Metric"
 			(at 350.139 144.526 90)
 			(hide yes)
@@
 		)
 		(instances
-			(project "oomwoo-kicad"
+			(project "Main"
 				(path "/dbcfb655-8d45-4808-9a74-2a0eb03372e8"
 					(reference "R66")
@@
 			)
 		)
-		(property "Footprint" ""
+		(property "Footprint" "Resistor_SMD:R_0603_1608Metric"
 			(at 258.699 251.079 90)
 			(hide yes)
@@
 		)
 		(instances
-			(project "oomwoo-kicad"
+			(project "Main"
 				(path "/dbcfb655-8d45-4808-9a74-2a0eb03372e8"
 					(reference "R52")
@@
 			)
 		)
-		(property "Footprint" ""
+		(property "Footprint" "Resistor_SMD:R_0603_1608Metric"
 			(at 352.679 155.956 90)
 			(hide yes)
@@
 		)
 		(instances
-			(project "oomwoo-kicad"
+			(project "Main"
 				(path "/dbcfb655-8d45-4808-9a74-2a0eb03372e8"
 					(reference "R67")
@@
 		)
 		(instances
-			(project "oomwoo-kicad"
+			(project "Main"
 				(path "/dbcfb655-8d45-4808-9a74-2a0eb03372e8"
 					(page "35")
@@
 		)
 		(instances
-			(project "oomwoo-kicad"
+			(project "Main"
 				(path "/dbcfb655-8d45-4808-9a74-2a0eb03372e8"
 					(page "2")
@@
 		)
 		(instances
-			(project "oomwoo-kicad"
+			(project "Main"
 				(path "/dbcfb655-8d45-4808-9a74-2a0eb03372e8"
 					(page "24")
@@
 		)
 		(instances
-			(project "oomwoo-kicad"
+			(project "Main"
 				(path "/dbcfb655-8d45-4808-9a74-2a0eb03372e8"
 					(page "29")
@@
 		)
 		(instances
-			(project "oomwoo-kicad"
+			(project "Main"
 				(path "/dbcfb655-8d45-4808-9a74-2a0eb03372e8"
 					(page "20")
@@
 		)
 		(instances
-			(project "oomwoo-kicad"
+			(project "Main"
 				(path "/dbcfb655-8d45-4808-9a74-2a0eb03372e8"
 					(page "30")
@@
 		)
 		(instances
-			(project "oomwoo-kicad"
+			(project "Main"
 				(path "/dbcfb655-8d45-4808-9a74-2a0eb03372e8"
 					(page "32")
@@
 		)
 		(instances
-			(project "oomwoo-kicad"
+			(project "Main"
 				(path "/dbcfb655-8d45-4808-9a74-2a0eb03372e8"
 					(page "27")
@@
 		)
 		(instances
-			(project "oomwoo-kicad"
+			(project "Main"
 				(path "/dbcfb655-8d45-4808-9a74-2a0eb03372e8"
 					(page "5")
@@
 		)
 		(instances
-			(project "oomwoo-kicad"
+			(project "Main"
 				(path "/dbcfb655-8d45-4808-9a74-2a0eb03372e8"
 					(page "25")
@@
 		)
 		(instances
-			(project "oomwoo-kicad"
+			(project "Main"
 				(path "/dbcfb655-8d45-4808-9a74-2a0eb03372e8"
 					(page "26")
@@
 		)
 		(instances
-			(project "oomwoo-kicad"
+			(project "Main"
 				(path "/dbcfb655-8d45-4808-9a74-2a0eb03372e8"
 					(page "4")
@@
 		)
 		(instances
-			(project "oomwoo-kicad"
+			(project "Main"
 				(path "/dbcfb655-8d45-4808-9a74-2a0eb03372e8"
 					(page "3")
@@
 		)
 		(instances
-			(project "oomwoo-kicad"
+			(project "Main"
 				(path "/dbcfb655-8d45-4808-9a74-2a0eb03372e8"
 					(page "22")
@@
 		)
 		(instances
-			(project "oomwoo-kicad"
+			(project "Main"
 				(path "/dbcfb655-8d45-4808-9a74-2a0eb03372e8"
 					(page "23")
@@
 		)
 		(instances
-			(project "oomwoo-kicad"
+			(project "Main"
 				(path "/dbcfb655-8d45-4808-9a74-2a0eb03372e8"
 					(page "34")
@@
 		)
 		(instances
-			(project "oomwoo-kicad"
+			(project "Main"
 				(path "/dbcfb655-8d45-4808-9a74-2a0eb03372e8"
 					(page "19")
@@
 		)
 		(instances
-			(project "oomwoo-kicad"
+			(project "Main"
 				(path "/dbcfb655-8d45-4808-9a74-2a0eb03372e8"
 					(page "28")
@@
 		)
 		(instances
-			(project "oomwoo-kicad"
+			(project "Main"
 				(path "/dbcfb655-8d45-4808-9a74-2a0eb03372e8"
 					(page "33")
@@
 		)
 		(instances
-			(project "oomwoo-kicad"
+			(project "Main"
 				(path "/dbcfb655-8d45-4808-9a74-2a0eb03372e8"
 					(page "21")

Commit message: Schematic fixes, 1st round of review
Parts:
- removed R1, R51, R52, R53, R54, R55, R63, R65, R66, R67: 10, Resistor_SMD:R_0603_1608Metric, symbol Device:R_US
Other:
- sheet RTC_WATCHDOG renamed WATCHDOG
- sheet BUTTON-LED ports: added CLEAN-BTN; removed none
- sheet CAMERA ports: added CAM_GPIO0, CAM_GPIO1; removed CAM_IO
- sheet CM5-GPIO ports: added CAM_GPIO1; removed GPIO07, GPIO22, GPIO23, GPIO24, PMIC_EN2, SPI0_CS0, SPI0_MISO, SPI0_MOSI, SPI0_SCLK, UART4_RX, UART4_TX
- sheet CM5-HIGHSPEED ports: added PCIE_PWR_EN; removed none
- sheet LiDAR ports: added LIDAR_EN; removed none
- sheet MAIN-FAN ports: added none; removed MAIN-FAN-V-CTRL
- sheet MCU-STM32 ports: added CLEAN-BTN, LIDAR_EN, WDO, ~{JTAG_RST}, ~{STM32_RST}; removed MAIN-FAN-V-CTRL
- sheet POWER ports: added M2_PWR_EN; removed none
- sheet WATCHDOG: file RTC_WATCHDOG.kicad_sch -> WATCHDOG.kicad_sch
- sheet WATCHDOG ports: added WDI, ~{MR}, ~{PULSE_OUT}; removed LATCH_OUT, PULSE_OUT, SCL, SDA
- note added: "SIDE BRUSH MOTORs"
- note added: "WD"
- note removed: "RTC_WD"
- note removed: "SIDE BURSH MOTORs"
