File: kicad/main/SPEAKER-MIC.kicad_sch (KiCad schematic)
At the start: 15 parts, among them J18 SPEAKER2, Q14 IRLML6344TRPBF, U10 ICS-43434_C5656610, U11 MAX98357AETE_T, U9 ICS-43434_C5656610

Commit message: Fix edge cut; no-CM STEP
Parts:
- removed J18: SPEAKER2, oomwoo_altium:CONN-SMD_2P-P1.00_HX-1.0-2P-WT, symbol DesignLibrary:SPEAKER-MIC_0_HDRx2_DesignLibrary.SchLib
- added SPK1: ZX-ZH1_5-2PWT, JLCImport:ZX-ZH1_5-2PWT, symbol JLCImport:ZX-ZH1_5-2PWT
Connections:
- net GND: now also SPK1.3, SPK1.4
- net at ED4.1, U11.9 (OUTP): now also SPK1.1
- net at ED3.1, U11.10 (OUTN): now also SPK1.2

Commit message: Schematic fixes, 1st round of review
Parts:
- removed Q14: IRLML6344TRPBF, JLCImport:IRLML6344TRPBF, symbol JLCImport:IRLML6344TRPBF
- added Q9: 2302V, JLCImport:2302V, symbol JLCImport:2302V
- C10, C5, C9: value 100nF/10V -> 100nF/50V; LCSC (none) -> C1591
- C11: value 10uF/10V -> 10uF/25V; LCSC (none) -> C96446
- ED3, ED4: LCSC (none) -> C5261080; MANUFACTURER WillSemi(韦尔半导体) -> (none); Manufacturer (none) -> WillSemi(韦尔半导体)
Connections:
- net GND: now also Q9.2 (S)
- net SP_SHUTDOWN: now also Q9.1 (G)
- net at R9.1: now also Q9.3 (D)
