File: kicad/main/WHEEL-MOTORs .kicad_sch (KiCad schematic)
At the start: 20 parts, among them U14 DRV8870DDAR, U15 DRV8870DDAR

Commit message: Fix edge cut; no-CM STEP
Parts:
- removed C85, C89: 100uF, oomwoo_altium:CAP-SMD_BD6.3-L6.6-W6.6-FD, symbol DesignLibrary:WHEEL MOTOR_3_Capacitor-2_DesignLibrary.SchLib
- removed MOT_L1, MOT_R1: S7B-ZR_LF_SN, JLCImport:S7B-ZR_LF_SN, symbol JLCImport:S7B-ZR_LF_SN
- added C20, C39: JBLM2101M025C058RTM_100UF_25V, JLCImport:JBLM2101M025C058RTM_100UF_25V, symbol JLCImport:JBLM2101M025C058RTM_100UF_25V
- added MOT_L1, MOT_R1: ZX-ZH1_5-7PWT, JLCImport:ZX-ZH1_5-7PWT, symbol JLCImport:ZX-ZH1_5-7PWT
- R49, R50: footprint (none) -> Resistor_SMD:R_0603_1608Metric
- R83, R84: footprint Resistor_SMD:R_0603_1608Metric -> Resistor_SMD:R_2512_6332Metric
- U14, U15: footprint oomwoo_altium:HSOP-8_L5.0-W4.0-P1.27-LS6.2-BL-EP -> JLCImport:DRV8870DDAR
Connections:
- net GND: now also C20.2, C39.2, MOT_L1.4, MOT_L1.8, MOT_L1.9, MOT_R1.4, MOT_R1.8, MOT_R1.9
- net VCC-3V3-P: now also MOT_L1.6, MOT_R1.6
- net VCC-5V-REG: now also MOT_L1.3, MOT_R1.3
- net VM-VBAT: now also C20.1, C39.1
- net WHEEL-M-LEFT-DROP: now also MOT_L1.7
- net WHEEL-M-LEFT-ENCODE-A: now also MOT_L1.5
- net WHEEL-M-RIGHT-DROP: now also MOT_R1.7
- net WHEEL-M-RIGHT-ENCODE-A: now also MOT_R1.5
- net at U14.6 (OUT1): now also MOT_R1.1
- net at U14.8 (OUT2): now also MOT_R1.2
- net at U15.6 (OUT1): now also MOT_L1.1
- net at U15.8 (OUT2): now also MOT_L1.2

Commit message: Schematic fixes, 1st round of review
Parts:
- removed C20, C39: JBLM2101M025C058RTM_100UF_25V, JLCImport:JBLM2101M025C058RTM_100UF_25V, symbol JLCImport:JBLM2101M025C058RTM_100UF_25V
- removed D19, D20: 1N4007, oomwoo_altium:SOD123, symbol DesignLibrary:WHEEL MOTOR_3_DIODE-1_DesignLibrary.SchLib
- removed R108, R109, R89, R90, R97, R98: 10K, Resistor_SMD:R_0603_1608Metric, symbol DesignLibrary:WHEEL MOTOR_0_Resistor-1_DesignLibrary.SchLib
- added C135, C136: 10uF/25V, Capacitor_SMD:C_0603_1608Metric, symbol JLCImport:CL21A106KBYQNNE
- added C142, C143: 100nF/50V, Capacitor_SMD:C_0603_1608Metric, symbol Library:C_0603
- added R11, R17, R20, R27: 100k, Resistor_SMD:R_0603_1608Metric, symbol Device:R_US
- added R51, R52: 10k, Resistor_SMD:R_0603_1608Metric, symbol Device:R_US
- C84: value 0.22uF/25V -> 100nF/50V; LCSC (none) -> C1591; MANUFACTURER * -> (none); Manufacturer (none) -> *
- C88: value 0.22uF -> 100nF/50V; LCSC (none) -> C1591; MANUFACTURER * -> (none); Manufacturer (none) -> *
- R83, R84: value 0.2R -> 0.2R/10W; LCSC (none) -> C5375488; MANUFACTURER * -> (none); Manufacturer (none) -> *
- U14, U15: LCSC (none) -> C86590; MANUFACTURER * -> (none); Manufacturer (none) -> *
- renumbered MOT_L1 to MOT_WHEEL_L1, MOT_R1 to MOT_WHEEL_R1
Connections:
- net VCC-5V-REG is gone; now on net GND: MOT_WHEEL_L1.3, MOT_WHEEL_R1.3
- net GND: now also MOT_WHEEL_L1.6, MOT_WHEEL_R1.6, C135.2, C136.2, C142.2, C143.2, R11.2, R17.2, R20.2, R27.2; no longer MOT_WHEEL_L1.4, MOT_WHEEL_R1.4, R49.2, R50.2
- net VCC-3V3-P: now also MOT_WHEEL_L1.5, MOT_WHEEL_R1.5, R49.1, R50.1, C142.1, C143.1, R51.1, R52.1; no longer MOT_WHEEL_L1.6, MOT_WHEEL_R1.6
- net VM-VBAT: now also C135.1, C136.1
- net WHEEL-M-L-F-ADC: now also R84.2, U15.7 (ISEN)
- net WHEEL-M-LEFT-DROP: now also R50.2; no longer R50.1
- net WHEEL-M-LEFT-ENCODE-A: now also MOT_WHEEL_L1.4, R52.2; no longer MOT_WHEEL_L1.5
- net WHEEL-M-LEFT-IN1: now also U15.3 (IN1), R20.1
- net WHEEL-M-LEFT-IN2: now also U15.2 (IN2), R27.1
- net WHEEL-M-R-F-ADC: now also R83.2, U14.7 (ISEN)
- net WHEEL-M-RIGHT-DROP: now also R49.2; no longer R49.1
- net WHEEL-M-RIGHT-ENCODE-A: now also MOT_WHEEL_R1.4, R51.2; no longer MOT_WHEEL_R1.5
- net WHEEL-M-RIGHT-IN1: now also U14.3 (IN1), R11.1
- net WHEEL-M-RIGHT-IN2: now also U14.2 (IN2), R17.1
Other:
- moved on the sheet: R49, R50
